File: RetPCSchematics/RetPCSchematics.sch (KiCad schematic (older format))
At the start: 13 parts

Commit message: Update with Demux
Found a demux for the Graphics Unit
Parts:
- removed U? (x2): 74LS154, symbol 74xx:74LS154
- added U? (x6): 74HC237, symbol 74xx_IEEE:74HC237
Connections:
- wire segments 65 -> 94
Changed lines of the file:
@@
 EESchema Schematic File Version 4
+LIBS:RetPCSchematics-cache
 EELAYER 26 0
 EELAYER END
@@
 L Memory_RAM:628128 U?
 U 1 1 5BB7F65C
-P 13450 6650
-F 0 "U?" H 13450 7966 50  0000 C CNN
-F 1 "628128" H 13450 7875 50  0000 C CNN
-F 2 "" H 13450 6650 50  0001 C CNN
-F 3 "" H 13450 6650 50  0001 C CNN
-	1    13450 6650
-	1    0    0    -1
-$EndComp
-$Comp
-L 74xx:74LS154 U?
-U 1 1 5BB812D7
-P 15350 7950
-F 0 "U?" H 15350 9128 50  0000 C CNN
-F 1 "74LS154" H 15350 9037 50  0000 C CNN
-F 2 "" H 15350 7950 50  0001 C CNN
-F 3 "http://www.ti.com/lit/gpn/sn74LS154" H 15350 7950 50  0001 C CNN
-	1    15350 7950
-	1    0    0    -1
-$EndComp
-$Comp
-L 74xx:74LS154 U?
-U 1 1 5BB814D7
-P 15350 5700
-F 0 "U?" H 15350 6878 50  0000 C CNN
-F 1 "74LS154" H 15350 6787 50  0000 C CNN
-F 2 "" H 15350 5700 50  0001 C CNN
-F 3 "http://www.ti.com/lit/gpn/sn74LS154" H 15350 5700 50  0001 C CNN
-	1    15350 5700
+P 11950 6500
+F 0 "U?" H 11950 7816 50  0000 C CNN
+F 1 "628128" H 11950 7725 50  0000 C CNN
+F 2 "" H 11950 6500 50  0001 C CNN
+F 3 "" H 11950 6500 50  0001 C CNN
+	1    11950 6500
 	1    0    0    -1
 $EndComp
@@
 L 74xx:74HC590 U?
 U 1 1 5BB84844
-P 11900 4350
-F 0 "U?" V 11854 5091 50  0000 L CNN
-F 1 "74HC590" V 11945 5091 50  0000 L CNN
-F 2 "" H 11900 4400 50  0001 C CNN
-F 3 "https://assets.nexperia.com/documents/data-sheet/74HC590.pdf" H 11900 4400 50  0001 C CNN
-	1    11900 4350
+P 10400 4200
+F 0 "U?" V 10354 4941 50  0000 L CNN
+F 1 "74HC590" V 10445 4941 50  0000 L CNN
+F 2 "" H 10400 4250 50  0001 C CNN
+F 3 "https://assets.nexperia.com/documents/data-sheet/74HC590.pdf" H 10400 4250 50  0001 C CNN
+	1    10400 4200
 	0    1    1    0
 $EndComp
 Wire Wire Line
-	12400 4750 12400 4950
-Wire Wire Line
-	12400 5600 12750 5600
-Wire Wire Line
-	12300 5700 12750 5700
-Wire Wire Line
-	12300 4750 12300 5050
-Wire Wire Line
-	12200 5800 12750 5800
-Wire Wire Line
-	12200 4750 12200 5150
-Wire Wire Line
-	12100 4750 12100 5250
-Wire Wire Line
-	12100 5900 12750 5900
-Wire Wire Line
-	12000 4750 12000 5350
-Wire Wire Line
-	12000 6000 12750 6000
-Wire Wire Line
-	11900 4750 11900 5450
-Wire Wire Line
-	11900 6100 12750 6100
-Wire Wire Line
-	11800 4750 11800 5550
-Wire Wire Line
-	11800 6200 12750 6200
-Wire Wire Line
-	11700 4750 11700 5650
-Wire Wire Line
-	11700 6300 12750 6300
-Text Notes 11800 5800 0    50   ~ 0
+	10900 4600 10900 4800
+Wire Wire Line
+	10900 5450 11250 5450
+Wire Wire Line
+	10800 5550 11250 5550
+Wire Wire Line
+	10800 4600 10800 4900
+Wire Wire Line
+	10700 5650 11250 5650
+Wire Wire Line
+	10700 4600 10700 5000
+Wire Wire Line
+	10600 4600 10600 5100
+Wire Wire Line
+	10600 5750 11250 5750
+Wire Wire Line
+	10500 4600 10500 5200
+Wire Wire Line
+	10500 5850 11250 5850
+Wire Wire Line
+	10400 4600 10400 5300
+Wire Wire Line
+	10400 5950 11250 5950
+Wire Wire Line
+	10300 4600 10300 5400
+Wire Wire Line
+	10300 6050 11250 6050
+Wire Wire Line
+	10200 4600 10200 5500
+Wire Wire Line
+	10200 6150 11250 6150
+Text Notes 10300 5650 0    50   ~ 0
 MUX\n
 $Comp
 L MCU_Microchip_PIC16:PIC16F716-IP U?
 U 1 1 5BB94BE8
-P 9800 6400
-F 0 "U?" H 9800 7478 50  0000 C CNN
-F 1 "PIC16F716-IP" H 9800 7387 50  0000 C CNN
-F 2 "" H 9800 6400 50  0001 C CIN
-F 3 "http://ww1.microchip.com/downloads/en/DeviceDoc/41206B.pdf" H 9800 6400 50  0001 C CNN
-	1    9800 6400
-	1    0    0    -1
-$EndComp
+P 8300 6250
+F 0 "U?" H 8300 7328 50  0000 C CNN
+F 1 "PIC16F716-IP" H 8300 7237 50  0000 C CNN
+F 2 "" H 8300 6250 50  0001 C CIN
+F 3 "http://ww1.microchip.com/downloads/en/DeviceDoc/41206B.pdf" H 8300 6250 50  0001 C CNN
+	1    8300 6250
+	1    0    0    -1
+$EndComp
+$Comp
+L 74xx_IEEE:74HC237 U?
+U 1 1 5BB88565
+P 13600 5000
+F 0 "U?" H 13600 5516 50  0000 C CNN
+F 1 "74HC237" H 13600 5425 50  0000 C CNN
+F 2 "" H 13600 5000 50  0001 C CNN
+F 3 "" H 13600 5000 50  0001 C CNN
+	1    13600 5000
+	1    0    0    -1
+$EndComp
+$Comp
+L 74xx_IEEE:74HC237 U?
+U 1 1 5BB8DEB5
+P 13600 6300
+F 0 "U?" H 13600 6816 50  0000 C CNN
+F 1 "74HC237" H 13600 6725 50  0000 C CNN
+F 2 "" H 13600 6300 50  0001 C CNN
+F 3 "" H 13600 6300 50  0001 C CNN
+	1    13600 6300
+	1    0    0    -1
+$EndComp
+$Comp
+L 74xx_IEEE:74HC237 U?
+U 1 1 5BB90A7D
+P 15600 6350
+F 0 "U?" H 15600 6866 50  0000 C CNN
+F 1 "74HC237" H 15600 6775 50  0000 C CNN
+F 2 "" H 15600 6350 50  0001 C CNN
+F 3 "" H 15600 6350 50  0001 C CNN
+	1    15600 6350
+	1    0    0    -1
+$EndComp
+$Comp
+L 74xx_IEEE:74HC237 U?
+U 1 1 5BB92045
+P 13600 7650
+F 0 "U?" H 13600 8166 50  0000 C CNN
+F 1 "74HC237" H 13600 8075 50  0000 C CNN
+F 2 "" H 13600 7650 50  0001 C CNN
+F 3 "" H 13600 7650 50  0001 C CNN
+	1    13600 7650
+	1    0    0    -1
+$EndComp
+$Comp
+L 74xx_IEEE:74HC237 U?
+U 1 1 5BB9360A
+P 15600 7700
+F 0 "U?" H 15600 8216 50  0000 C CNN
+F 1 "74HC237" H 15600 8125 50  0000 C CNN
+F 2 "" H 15600 7700 50  0001 C CNN
+F 3 "" H 15600 7700 50  0001 C CNN
+	1    15600 7700
+	1    0    0    -1
+$EndComp
+Wire Wire Line
+	16050 4250 17150 4250
+Wire Wire Line
+	14150 4800 14150 3750
+Wire Wire Line
+	14150 3750 17150 3750
+Wire Wire Line
+	14150 6100 14300 6100
+Wire Wire Line
+	14300 6100 14300 3850
+Wire Wire Line
+	14300 3850 17150 3850
+Wire Wire Line
+	14500 7450 14500 3950
+Wire Wire Line
+	14500 3950 17150 3950
+Wire Wire Line
+	14150 7450 14500 7450
+Wire Wire Line
+	14150 6200 14600 6200
+Wire Wire Line
+	14600 6200 14600 5750
+Wire Wire Line
+	14600 5750 17150 5750
+Wire Wire Line
+	17150 4750 17350 4750
+$Comp
+L 74xx_IEEE:74HC237 U?
+U 1 1 5BBCD7DF
+P 15500 4850
+F 0 "U?" H 15500 5366 50  0000 C CNN
+F 1 "74HC237" H 15500 5275 50  0000 C CNN
+F 2 "" H 15500 4850 50  0001 C CNN
+F 3 "" H 15500 4850 50  0001 C CNN
+	1    15500 4850
+	1    0    0    -1
+$EndComp
+Wire Wire Line
+	14150 4900 14600 4900
+Wire Wire Line
+	14600 4900 14600 5650
+Wire Wire Line
+	14600 5650 17150 5650
+Wire Wire Line
+	14150 7550 14700 7550
+Wire Wire Line
+	14700 7550 14700 5850
+Wire Wire Line
+	14700 5850 17150 5850
+Wire Wire Line
+	14150 7650 14800 7650
+Wire Wire Line
+	14800 7650 14800 7300
+Wire Wire Line
+	14800 7300 16800 7300
+Wire Wire Line
+	16800 7300 16800 7700
+Wire Wire Line
+	16800 7700 17150 7700
+Wire Wire Line
+	14150 6300 14800 6300
+Wire Wire Line
+	14800 6300 14800 7250
+Wire Wire Line
+	14800 7250 16900 7250
+Wire Wire Line
+	16900 7250 16900 7600
+Wire Wire Line
+	16900 7600 17150 7600
 $EndSCHEMATC

Commit message: test
Parts:
- removed U? (x6): 74HC237, symbol 74xx_IEEE:74HC237
- added J?: Bus_ISA_8bit, symbol Bus_ISA_8bit
- added U? (x12): 74LVC1G18, symbol 74LVC1G18
Connections:
- net labels added: Binarycounter
- wire segments 94 -> 143
Other:
- note removed: "MUX\n"
