File: RetPCSchematics/VGA-GraphicsAdapter.sch (KiCad schematic (older format))
At the start: 30 parts

Commit message: Added labels
Added labels for information
Connections:
- net labels added: BinaryCounter, BlueLatch, BlueSignal, Clock, GND, GreenLatch, GreenSignal, ISA8BitBus, RedLatch, RedSignal, VGAChipProcessor, VRAM, VideoDataPlexingUnit, VideoTransferControl
- net labels removed: Blue, Green, Red
- wire segments 188 -> 213
Other:
- moved on the sheet: J?, X?
Changed lines of the file:
@@
 EESchema Schematic File Version 4
-LIBS:RetPCSchematics-cache
+LIBS:VGA-GraphicsAdapter-cache
 EELAYER 26 0
 EELAYER END
@@
 	10300 4100 10900 4100
 Wire Wire Line
-	9800 4900 10400 4900
-Wire Wire Line
 	10400 4900 10400 4200
 Wire Wire Line
@@
 Wire Wire Line
 	10850 6050 10900 6050
-Text Label 11900 1750 0    50   ~ 0
-Red
-Text Label 11800 3700 0    50   ~ 0
-Green
-Text Label 11950 5550 0    50   ~ 0
-Blue
 $Comp
 L Connector:DB15_Female_HighDensity J?
@@
 L Graphic:Logo_Open_Hardware_Large #LOGO?
 U 1 1 5BB7E327
-P 9450 8300
-F 0 "#LOGO?" H 9450 8800 50  0001 C CNN
-F 1 "Logo_Open_Hardware_Large" H 9450 7900 50  0001 C CNN
-F 2 "" H 9450 8300 50  0001 C CNN
-F 3 "~" H 9450 8300 50  0001 C CNN
-	1    9450 8300
+P 8000 2950
+F 0 "#LOGO?" H 8000 3450 50  0001 C CNN
+F 1 "Logo_Open_Hardware_Large" H 8000 2550 50  0001 C CNN
+F 2 "" H 8000 2950 50  0001 C CNN
+F 3 "~" H 8000 2950 50  0001 C CNN
+	1    8000 2950
 	1    0    0    -1
 $EndComp
@@
 L Oscillator:DGOF5S3 X?
 U 1 1 5BB7E889
-P 6850 -100
-F 0 "X?" H 6509 -54 50  0000 R CNN
-F 1 "DGOF5S3" H 6509 -145 50  0000 R CNN
-F 2 "Oscillator:Oscillator_DIP-14" H 7300 -450 50  0001 C CNN
-F 3 "http://www.conwin.com/datasheets/cx/cx030.pdf" H 6750 -100 50  0001 C CNN
-	1    6850 -100
+P 3350 1700
+F 0 "X?" H 3009 1746 50  0000 R CNN
+F 1 "DGOF5S3" H 3009 1655 50  0000 R CNN
+F 2 "Oscillator:Oscillator_DIP-14" H 3800 1350 50  0001 C CNN
+F 3 "http://www.conwin.com/datasheets/cx/cx030.pdf" H 3250 1700 50  0001 C CNN
+	1    3350 1700
 	1    0    0    -1
 $EndComp
@@
 L Connector:Bus_ISA_8bit J?
 U 1 1 5BD7DCB9
-P 5750 10150
-F 0 "J?" V 5796 11780 50  0000 L CNN
-F 1 "Bus_ISA_8bit" V 5705 11780 50  0000 L CNN
-F 2 "" H 5750 10150 50  0001 C CNN
-F 3 "https://en.wikipedia.org/wiki/Industry_Standard_Architecture" H 5750 10150 50  0001 C CNN
-	1    5750 10150
+P 7200 10050
+F 0 "J?" V 7246 11680 50  0000 L CNN
+F 1 "Bus_ISA_8bit" V 7155 11680 50  0000 L CNN
+F 2 "" H 7200 10050 50  0001 C CNN
+F 3 "https://en.wikipedia.org/wiki/Industry_Standard_Architecture" H 7200 10050 50  0001 C CNN
+	1    7200 10050
 	0    1    -1   0
 $EndComp
@@
 Wire Wire Line
 	5950 1700 9300 1700
-Connection ~ 7250 3250
-Wire Wire Line
-	7250 3250 7300 3250
 Connection ~ 5450 3750
 Wire Wire Line
@@
 $EndComp
 Wire Wire Line
-	3500 6050 3900 6050
-Wire Wire Line
 	4250 6050 4650 6050
 Wire Wire Line
@@
 	1    0    0    -1
 $EndComp
+Wire Wire Line
+	1900 9150 1900 9350
+Wire Wire Line
+	1900 9350 1750 9350
+Wire Wire Line
+	1750 9350 1750 6050
+Wire Wire Line
+	1750 6050 3500 6050
+Connection ~ 3500 6050
+Wire Wire Line
+	3500 6050 3900 6050
+Text Label 1550 4200 0    67   ~ 0
+BinaryCounter
+Text Label 4400 4700 0    67   ~ 0
+VRAM
+Text Label 9150 3000 0    67   ~ 0
+RedLatch
+Text Label 9150 4900 0    67   ~ 0
+GreenLatch
+Text Label 9150 6700 0    67   ~ 0
+BlueLatch
+Text Label 11950 1800 0    67   ~ 0
+RedSignal
+Text Label 11950 3650 0    67   ~ 0
+GreenSignal
+Text Label 12050 5850 0    67   ~ 0
+BlueSignal
+Text Label 2750 1450 0    67   ~ 0
+Clock
+Text Label 9000 9150 0    67   ~ 0
+ISA8BitBus
+Text Label 2550 5900 0    67   ~ 0
+VideoTransferControl
+Text Label 6650 6500 0    67   ~ 0
+VideoDataPlexingUnit
+$Comp
+L power:GND #PWR?
+U 1 1 5BD056E0
+P 2600 4300
+F 0 "#PWR?" H 2600 4050 50  0001 C CNN
+F 1 "GND" H 2605 4127 50  0000 C CNN
+F 2 "" H 2600 4300 50  0001 C CNN
+F 3 "" H 2600 4300 50  0001 C CNN
+	1    2600 4300
+	1    0    0    -1
+$EndComp
+$Comp
+L power:GND #PWR?
+U 1 1 5BD05A0E
+P 10350 3050
+F 0 "#PWR?" H 10350 2800 50  0001 C CNN
+F 1 "GND" H 10355 2877 50  0000 C CNN
+F 2 "" H 10350 3050 50  0001 C CNN
+F 3 "" H 10350 3050 50  0001 C CNN
+	1    10350 3050
+	1    0    0    -1
+$EndComp
+Wire Wire Line
+	10350 3000 10350 3050
+Connection ~ 10350 3000
+Wire Wire Line
+	10350 3000 11400 3000
+Wire Wire Line
+	9800 3000 9050 3000
+Wire Wire Line
+	9050 3000 9050 2300
+Wire Wire Line
+	9050 2300 9200 2300
+Connection ~ 9800 3000
+Wire Wire Line
+	9200 2300 9200 2400
+Wire Wire Line
+	9200 2400 9300 2400
+Connection ~ 9200 2300
+Wire Wire Line
+	9200 2300 9300 2300
+$Comp
+L power:GND #PWR?
+U 1 1 5BD3750D
+P 10400 4950
+F 0 "#PWR?" H 10400 4700 50  0001 C CNN
+F 1 "GND" H 10405 4777 50  0000 C CNN
+F 2 "" H 10400 4950 50  0001 C CNN
+F 3 "" H 10400 4950 50  0001 C CNN
+	1    10400 4950
+	1    0    0    -1
+$EndComp
+Wire Wire Line
+	10400 4900 10400 4950
+$Comp
+L power:GND #PWR?
+U 1 1 5BD5124D
+P 10400 6800
+F 0 "#PWR?" H 10400 6550 50  0001 C CNN
+F 1 "GND" H 10405 6627 50  0000 C CNN
+F 2 "" H 10400 6800 50  0001 C CNN
+F 3 "" H 10400 6800 50  0001 C CNN
+	1    10400 6800
+	1    0    0    -1
+$EndComp
+Wire Wire Line
+	10400 6750 10400 6800
+Wire Wire Line
+	10450 6750 11400 6750
+Wire Wire Line
+	9800 6750 9000 6750
+Wire Wire Line
+	9000 6750 9000 6050
+Wire Wire Line
+	9000 6050 9200 6050
+Connection ~ 9800 6750
+Wire Wire Line
+	9200 6050 9200 6150
+Wire Wire Line
+	9200 6150 9300 6150
+Connection ~ 9200 6050
+Wire Wire Line
+	9200 6050 9300 6050
+Wire Wire Line
+	9150 4900 9150 4300
+Wire Wire Line
+	9150 4200 9300 4200
+Wire Wire Line
+	9150 4900 9800 4900
+Connection ~ 9800 4900
+Wire Wire Line
+	9800 4900 10400 4900
+Wire Wire Line
+	9150 4300 9300 4300
+Connection ~ 9150 4300
+Wire Wire Line
+	9150 4300 9150 4200
+Text Label 3800 8700 0    67   ~ 0
+VGAChipProcessor
 $EndSCHEMATC

Commit message: Updated wiring
Made wiring for clock logic for RGB latches. Changed wiring for ISA bus
Parts:
- added U15: 74AUC2G00, symbol 74xGxx:74AUC2G00
- added U4: 74AHC1G08, symbol 74xGxx:74AHC1G08
- added U6: 74LS161, symbol 74xx:74LS161
- gave numbers to parts that had none: 27
Connections:
- wire segments 213 -> 284
Other:
- moved on the sheet: J1, X1

Commit message: Continued wiring
Parts:
- added C? (x3): C, symbol Device:C
- U1: symbol RetPC:PIC16F707QFP -> VGA-GraphicsAdapter-rescue:PIC16F707QFP-RetPC
Connections:
- wire segments 284 -> 296
Changed lines of the file:
@@
 	3700 5500 3700 5800
 $Comp
-L RetPC:PIC16F707QFP U1
+L VGA-GraphicsAdapter-rescue:PIC16F707QFP-RetPC U1
 U 1 1 5BF67D1E
 P 2450 6500
@@
 Connection ~ 10350 3000
 Wire Wire Line
-	10350 3000 11400 3000
+	10350 3000 10900 3000
 Wire Wire Line
 	9200 2300 9200 2400
@@
 	6450 1400 8850 1400
 Wire Wire Line
-	10400 6750 11400 6750
+	10400 6750 10900 6750
 Connection ~ 10400 6750
 Wire Wire Line
-	11400 4900 10400 4900
+	11400 4900 10900 4900
 Connection ~ 10400 4900
 Wire Wire Line
@@
 Wire Wire Line
 	2200 9150 2200 9500
+Wire Wire Line
+	10900 4900 10900 4600
+Connection ~ 10900 4900
+Wire Wire Line
+	10900 4900 10400 4900
+Wire Wire Line
+	10900 3000 10900 2700
+Connection ~ 10900 3000
+Wire Wire Line
+	10900 3000 11400 3000
+Wire Wire Line
+	10900 6750 10900 6450
+Connection ~ 10900 6750
+Wire Wire Line
+	10900 6750 11400 6750
+$Comp
+L Device:C C?
+U 1 1 5BF2BB2F
+P 12000 2850
+F 0 "C?" H 12115 2896 50  0000 L CNN
+F 1 "C" H 12115 2805 50  0000 L CNN
+F 2 "" H 12038 2700 50  0001 C CNN
+F 3 "~" H 12000 2850 50  0001 C CNN
+	1    12000 2850
+	1    0    0    -1
+$EndComp
+Wire Wire Line
+	11900 2700 12000 2700
+Wire Wire Line
+	11400 3000 12000 3000
+Connection ~ 11400 3000
+$Comp
+L Device:C C?
+U 1 1 5BF61837
+P 12000 4750
+F 0 "C?" H 12115 4796 50  0000 L CNN
+F 1 "C" H 12115 4705 50  0000 L CNN
+F 2 "" H 12038 4600 50  0001 C CNN
+F 3 "~" H 12000 4750 50  0001 C CNN
+	1    12000 4750
+	1    0    0    -1
+$EndComp
+$Comp
+L Device:C C?
+U 1 1 5BF7C75D
+P 12000 6600
+F 0 "C?" H 12115 6646 50  0000 L CNN
+F 1 "C" H 12115 6555 50  0000 L CNN
+F 2 "" H 12038 6450 50  0001 C CNN
+F 3 "~" H 12000 6600 50  0001 C CNN
+	1    12000 6600
+	1    0    0    -1
+$EndComp
+Wire Wire Line
+	12000 6450 11900 6450
+Wire Wire Line
+	11400 6750 12000 6750
+Connection ~ 11400 6750
+Wire Wire Line
+	11900 4600 12000 4600
+Wire Wire Line
+	11400 4900 12000 4900
+Connection ~ 11400 4900
 $EndSCHEMATC

Commit message: minor fixes
Parts:
- gave numbers to parts that had none: 3
Changed lines of the file:
@@
 	10900 6750 11400 6750
 $Comp
-L Device:C C?
+L Device:C C1
 U 1 1 5BF2BB2F
 P 12000 2850
-F 0 "C?" H 12115 2896 50  0000 L CNN
+F 0 "C1" H 12115 2896 50  0000 L CNN
 F 1 "C" H 12115 2805 50  0000 L CNN
 F 2 "" H 12038 2700 50  0001 C CNN
@@
 Connection ~ 11400 3000
 $Comp
-L Device:C C?
+L Device:C C2
 U 1 1 5BF61837
 P 12000 4750
-F 0 "C?" H 12115 4796 50  0000 L CNN
+F 0 "C2" H 12115 4796 50  0000 L CNN
 F 1 "C" H 12115 4705 50  0000 L CNN
 F 2 "" H 12038 4600 50  0001 C CNN
@@
 $EndComp
 $Comp
-L Device:C C?
+L Device:C C3
 U 1 1 5BF7C75D
 P 12000 6600
-F 0 "C?" H 12115 6646 50  0000 L CNN
+F 0 "C3" H 12115 6646 50  0000 L CNN
 F 1 "C" H 12115 6555 50  0000 L CNN
 F 2 "" H 12038 6450 50  0001 C CNN

Commit message: updated schematics and pcblayout for Graphics adapter
Parts:
- removed C1, C2, C3: C, symbol Device:C
- removed U22, U23, U24: 74LS573, symbol 74xx:74LS573
- removed U25, U26, U27: AD558JN, symbol Analog_DAC:AD558JN
- added U?: TDA8772, symbol Video:TDA8772
Connections:
- net labels removed: BlueLatch, BlueSignal, GreenLatch, GreenSignal, PWR-5V, RedLatch, RedSignal
- wire segments 296 -> 234
Other:
- moved on the sheet: J2

Commit message: sync
Parts:
- removed J2: DB15_Female_HighDensity, symbol Connector:DB15_Female_HighDensity
Changed lines of the file:
@@
 $EndDescr
-$Comp
-L Connector:DB15_Female_HighDensity J2
-U 1 1 5BB7315E
-P 14100 4500
-F 0 "J2" H 14100 5367 50  0000 C CNN
-F 1 "DB15_Female_HighDensity" H 14100 5276 50  0000 C CNN
-F 2 "" H 13150 4900 50  0001 C CNN
-F 3 " ~" H 13150 4900 50  0001 C CNN
-	1    14100 4500
-	1    0    0    -1
-$EndComp
-Text Label 14450 4650 0    50   ~ 0
-H-SYNC
-Text Label 14450 4450 0    50   ~ 0
-V-SYNC
-Wire Wire Line
-	14400 4500 14850 4500
-Wire Wire Line
-	14400 4700 14850 4700
 $Comp
 L Graphic:Logo_Open_Hardware_Large #LOGO1
@@
 Wire Wire Line
 	6450 1400 12950 1400
-Wire Wire Line
-	12700 3300 13550 3300
-Wire Wire Line
-	13550 3300 13550 4100
-Wire Wire Line
-	13550 4100 13800 4100
-Wire Wire Line
-	12700 3500 13450 3500
-Wire Wire Line
-	13450 3500 13450 4300
-Wire Wire Line
-	13450 4300 13800 4300
-Wire Wire Line
-	12700 3700 13350 3700
-Wire Wire Line
-	13350 3700 13350 4500
-Wire Wire Line
-	13350 4500 13800 4500
 $EndSCHEMATC

Commit message: Made Revision 2.0.1 for the grahpics card and added external libraries
Better adress handling and data loading. Changed GPU to Atmega 640. Added external libraries for footprints and schematic symbols. Changed to DVI-D output format
Parts:
- removed U1: PIC16F707QFP, symbol VGA-GraphicsAdapter-rescue:PIC16F707QFP-RetPC
- removed U15: 74AUC2G00, symbol 74xGxx:74AUC2G00
- removed U2: 74HC590, symbol 74xx:74HC590
- removed U3, U7, U8: 74LVC2G125, symbol 74xGxx:74LVC2G125
- removed U4: 74AHC1G08, symbol 74xGxx:74AHC1G08
- removed U6: 74LS161, symbol 74xx:74LS161
- removed U?: TDA8772, symbol Video:TDA8772
- added U15, U22, U23, U3, U33, U34, U35, U36, U37, U38, U39, U40, U41, U42, U43, U44, U45, U46, U47, U48, U49: 74LVC1G18, symbol 74xGxx:74LVC1G18
- added U2: 628128, symbol Memory_RAM:628128
- added U24, U7: 74LS245, symbol 74xx:74LS245
- added U25, U26, U27, U52, U? (x2): 74LS573, symbol 74xx:74LS573
- added U28: TFP410, symbol ti:TFP410
- added U29, U30, U31, U32, U50, U6: 4520, symbol 4xxx:4520
- added U4: 74LVC2G157, symbol 74xGxx:74LVC2G157
- added U53: 74LVC2G240, symbol 74xGxx:74LVC2G240
- added U54: 74LS21, symbol 74xx:74LS21
- added U8: SN74LVC245AN, digikey-footprints:DIP-20_W7.62mm, symbol dk_Logic-Buffers-Drivers-Receivers-Transceivers:SN74LVC245AN
- added U?: ATmega644P-20PU, Package_DIP:DIP-40_W15.24mm, symbol MCU_Microchip_ATmega:ATmega644P-20PU
- J1: footprint (none) -> RetPC:8Bit_ISA_BUS
Connections:
- net labels added: +3.3V, +5V, A0, A1, A10, A11, A12, A13, A14, A15, A16, A17, A18, A19, A2, A3, A4, A5, A6, A7, A8, A9, ALEN, BusRead, CountReset, D0, D1, D2, D3, D4, D5, D6, D7, LoadEnable, LoadPulse
- net labels removed: BinaryCounter, VGAChipProcessor, VideoTransferControl
- wire segments 223 -> 595
Other:
- moved on the sheet: J1, U10, U11, U12, U13, U14, U16, U17, U18, U19, U20, U21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

Commit message: Added more control singals and started rerouting
Added controlsignals and started rerouting pcb to rev 2.0.1
Parts:
- removed unit 2 of U53
- removed U54: 74LS21, symbol 74xx:74LS21
- added U1, U55, U57: 74LS245, symbol 74xx:74LS245
- added U? (x2): 74LS09, symbol 74xx:74LS09
- added U?: TFP410, symbol ti:TFP410
- added U?: 74LVC2G240, symbol 74xGxx:74LVC2G240
- gave numbers to parts that had none: 3
Connections:
- net labels added: AEN, GClock
- wire segments 595 -> 634
Other:
- moved on the sheet: U58
