File: RetPCSchematics/VGA-GraphicsAdapter.sch (KiCad schematic (older format))
At the start: 40 parts, among them J1 Bus_ISA_8bit, J2 74320-9004, U1 74AUC2G125, U10 ATmega644P-20PU, U11 628128, U12 628128, U13 SN74LVC245AN, U14 74LS245, U15 74LVC2G240, U16 74LVC2G240, U17 74LVC1G18, U18 74LVC1G18, U19 74LVC1G18, U2 74LVC2G240, U20 74LVC1G18, U21 ATF22V10D, U22 74LS245, U23 74LVC1G373, U24 74LVC1G373, U25 74LVC1G373, U26 74LVC1G373, U27 74LVC1G373, U28 74LVC1G373, U29 74LVC1G373, U3 ATF22V10D, U30 74LVC1G373, U31 74LVC1G373, U32 74LVC1G373, U33 74LVC1G373, U34 74LVC1G373, U36 TFP410, U37 ATF750C, U4 ATF22V10D, U5 74LS245, U6 ATF22V10D, U7 74LS245, U8 74LS245, U9 74LS245, X1 DGOF5S3

Commit message: sync
workstation switch sync
Changed lines of the file:
@@
 D7
 Entry Wire Line
-	6650 2600 6750 2700
+	6650 3500 6750 3400
 Entry Wire Line
-	6650 2700 6750 2800
+	6650 3400 6750 3300
 Entry Wire Line
-	6650 2800 6750 2900
+	6650 3300 6750 3200
 Entry Wire Line
-	6650 2900 6750 3000
+	6650 3200 6750 3100
 Entry Wire Line
-	6650 3000 6750 3100
+	6650 3100 6750 3000
 Entry Wire Line
-	6650 3100 6750 3200
+	6650 3000 6750 2900
 Entry Wire Line
-	6650 3200 6750 3300
+	6650 2900 6750 2800
 Entry Wire Line
-	6650 3300 6750 3400
-Text Label 6750 2700 0    50   ~ 0
+	6650 2800 6750 2700
+Text Label 6750 3400 0    50   ~ 0
 D0
-Text Label 6750 2800 0    50   ~ 0
+Text Label 6750 3300 0    50   ~ 0
 D1
-Text Label 6750 2900 0    50   ~ 0
+Text Label 6750 3200 0    50   ~ 0
 D2
-Text Label 6750 3000 0    50   ~ 0
-D3
 Text Label 6750 3100 0    50   ~ 0
+D3
+Text Label 6750 3000 0    50   ~ 0
 D4
-Text Label 6750 3200 0    50   ~ 0
+Text Label 6750 2900 0    50   ~ 0
 D5
-Text Label 6750 3300 0    50   ~ 0
+Text Label 6750 2800 0    50   ~ 0
 D6
-Text Label 6750 3400 0    50   ~ 0
+Text Label 6750 2700 0    50   ~ 0
 D7
 Text GLabel 6450 8150 1    50   BiDi ~ 0
@@
 	7650 6850 7650 6700
 Wire Wire Line
-	6750 2700 6800 2700
-Wire Wire Line
-	6750 2800 6800 2800
+	6750 3400 6800 3400
 Wire Wire Line
-	6750 2900 6800 2900
+	6750 3300 6800 3300
 Wire Wire Line
-	6750 3000 6800 3000
+	6750 3200 6800 3200
 Wire Wire Line
 	6750 3100 6800 3100
 Wire Wire Line
-	6750 3200 6800 3200
+	6750 3000 6800 3000
 Wire Wire Line
-	6750 3300 6800 3300
+	6750 2900 6800 2900
 Wire Wire Line
-	6750 3400 6800 3400
+	6750 2800 6800 2800
+Wire Wire Line
+	6750 2700 6800 2700
 Wire Wire Line
 	6500 3150 6550 3150
@@
 Wire Wire Line
 	9900 8200 9900 8650
-Wire Bus Line
-	4050 4850 4050 6700
 Text Label 4650 8150 1    50   ~ 0
 A16
@@
 Text Label 6850 5700 0    50   ~ 0
 D1
+Wire Bus Line
+	4050 4850 4050 6700
+Wire Bus Line
+	1650 8050 2150 8050
 Wire Wire Line
-	3500 5650 4400 5650
+	2550 6350 4750 6350
 Wire Wire Line
-	2750 6150 4650 6150
+	2650 6250 4700 6250
 Wire Wire Line
-	3450 6050 4600 6050
+	3850 4950 4150 4950
 Wire Wire Line
-	3400 5950 4550 5950
+	3800 5050 4150 5050
 Wire Wire Line
-	3350 5850 4500 5850
+	3750 5150 4150 5150
 Wire Wire Line
-	3300 5750 4450 5750
+	3700 5250 4200 5250
 Wire Wire Line
-	3550 5550 4350 5550
+	3650 5350 4250 5350
 Wire Wire Line
 	3600 5450 4300 5450
 Wire Wire Line
-	3650 5350 4250 5350
+	3550 5550 4350 5550
 Wire Wire Line
-	3700 5250 4200 5250
+	3300 5750 4450 5750
 Wire Wire Line
-	3750 5150 4150 5150
+	3350 5850 4500 5850
 Wire Wire Line
-	3800 5050 4150 5050
+	3400 5950 4550 5950
 Wire Wire Line
-	3850 4950 4150 4950
+	3450 6050 4600 6050
 Wire Wire Line
-	2650 6250 4700 6250
+	2750 6150 4650 6150
 Wire Wire Line
-	2550 6350 4750 6350
-Wire Bus Line
-	1650 8050 2150 8050
+	3500 5650 4400 5650
 Wire Bus Line
 	10350 9800 10350 11000

Commit message: EOD sync
Only control signals left to route
Parts:
- removed unit 1 of U2
Connections:
- wire segments 549 -> 547
Changed lines of the file:
@@
 Wire Wire Line
 	1900 6600 2450 6600
-Text GLabel 1350 6200 0    50   BiDi ~ 0
+Text GLabel 2350 5900 3    50   BiDi ~ 0
 GEnd
 $Comp
@@
 	1    0    0    -1
 $EndComp
-Wire Wire Line
-	2350 5900 2350 6200
-Wire Wire Line
-	2350 6200 1900 6200
 Text GLabel 6800 3600 3    50   BiDi ~ 0
 GEnd
@@
 Text GLabel 6050 8150 1    50   BiDi ~ 0
 Sel
-$Comp
-L power:GND #PWR01
-U 1 1 603E6A1B
-P 1600 6000
-F 0 "#PWR01" H 1600 5750 50  0001 C CNN
-F 1 "GND" H 1605 5827 50  0000 C CNN
-F 2 "" H 1600 6000 50  0001 C CNN
-F 3 "" H 1600 6000 50  0001 C CNN
-	1    1600 6000
-	-1   0    0    1
-$EndComp
-$Comp
-L 74xGxx:74LVC2G240 U2
-U 1 1 603E6A21
-P 1600 6200
-F 0 "U2" V 1529 6070 50  0000 R CNN
-F 1 "74LVC2G240" V 1620 6070 50  0000 R CNN
-F 2 "Package_SO:VSSOP-8_2.3x2mm_P0.5mm" H 1600 6200 50  0001 C CNN
-F 3 "http://www.ti.com/lit/sg/scyt129e/scyt129e.pdf" H 1600 6200 50  0001 C CNN
-	1    1600 6200
-	-1   0    0    -1
-$EndComp
 Wire Wire Line
 	7200 3900 6700 3900

Commit message: sync
Parts:
- added J3: Conn_01x02_Male, Connector_PinHeader_1.00mm:PinHeader_1x02_P1.00mm_Vertical, symbol Connector:Conn_01x02_Male
Changed lines of the file:
@@
 	1    0    0    1
 $EndComp
+Text GLabel 14100 6850 2    50   BiDi ~ 0
+Hsync
 Text GLabel 14100 6750 2    50   BiDi ~ 0
-Hsync
-Text GLabel 14100 6850 2    50   BiDi ~ 0
 Vsync
 Text GLabel 11850 4550 0    50   BiDi ~ 0
@@
 D1
 Wire Bus Line
+	1650 8050 2150 8050
+Wire Bus Line
+	10350 9800 10350 11000
+Wire Wire Line
+	3900 4850 4150 4850
+Wire Wire Line
+	2550 6350 4750 6350
+Wire Wire Line
+	2650 6250 4700 6250
+Wire Wire Line
+	3850 4950 4150 4950
+Wire Wire Line
+	3800 5050 4150 5050
+Wire Wire Line
+	3750 5150 4150 5150
+Wire Wire Line
+	3700 5250 4200 5250
+Wire Wire Line
+	3650 5350 4250 5350
+Wire Wire Line
+	3600 5450 4300 5450
+Wire Wire Line
+	3550 5550 4350 5550
+Wire Wire Line
+	3300 5750 4450 5750
+Wire Wire Line
+	3350 5850 4500 5850
+Wire Wire Line
+	3400 5950 4550 5950
+Wire Wire Line
+	3450 6050 4600 6050
+Wire Wire Line
+	2750 6150 4650 6150
+Wire Wire Line
+	3500 5650 4400 5650
+Wire Bus Line
+	6650 5550 7350 5550
+Wire Bus Line
+	4050 6700 4700 6700
+Wire Bus Line
+	9850 8950 9850 9800
+Wire Bus Line
+	1850 6700 4050 6700
+Wire Bus Line
+	8050 8850 8050 9800
+Wire Bus Line
+	10350 8500 10350 9800
+Wire Bus Line
+	2150 9700 5950 9700
+Wire Bus Line
 	4050 4850 4050 6700
 Wire Bus Line
-	1650 8050 2150 8050
-Wire Wire Line
-	2550 6350 4750 6350
-Wire Wire Line
-	2650 6250 4700 6250
-Wire Wire Line
-	3850 4950 4150 4950
-Wire Wire Line
-	3800 5050 4150 5050
-Wire Wire Line
-	3750 5150 4150 5150
-Wire Wire Line
-	3700 5250 4200 5250
-Wire Wire Line
-	3650 5350 4250 5350
-Wire Wire Line
-	3600 5450 4300 5450
-Wire Wire Line
-	3550 5550 4350 5550
-Wire Wire Line
-	3300 5750 4450 5750
-Wire Wire Line
-	3350 5850 4500 5850
-Wire Wire Line
-	3400 5950 4550 5950
-Wire Wire Line
-	3450 6050 4600 6050
-Wire Wire Line
-	2750 6150 4650 6150
-Wire Wire Line
-	3500 5650 4400 5650
-Wire Bus Line
-	10350 9800 10350 11000
-Wire Wire Line
-	3900 4850 4150 4850
-Wire Bus Line
-	6650 5550 7350 5550
-Wire Bus Line
-	4050 6700 4700 6700
-Wire Bus Line
-	9850 8950 9850 9800
-Wire Bus Line
-	1850 6700 4050 6700
-Wire Bus Line
-	8050 8850 8050 9800
-Wire Bus Line
-	10350 8500 10350 9800
-Wire Bus Line
-	2150 9700 5950 9700
-Wire Bus Line
 	3400 11000 10350 11000
 Wire Bus Line
@@
 Wire Bus Line
 	2150 8000 5850 8000
+$Comp
+L Connector:Conn_01x02_Male J3
+U 1 1 5C554E39
+P 10200 850
+F 0 "J3" V 10260 890 50  0000 L CNN
+F 1 "Conn_01x02_Male" V 10351 890 50  0000 L CNN
+F 2 "Connector_PinHeader_1.00mm:PinHeader_1x02_P1.00mm_Vertical" H 10200 850 50  0001 C CNN
+F 3 "~" H 10200 850 50  0001 C CNN
+	1    10200 850
+	0    1    1    0
+$EndComp
+$Comp
+L power:+3.3V #PWR0102
+U 1 1 5C554FE5
+P 10100 1050
+F 0 "#PWR0102" H 10100 900 50  0001 C CNN
+F 1 "+3.3V" H 10115 1223 50  0000 C CNN
+F 2 "" H 10100 1050 50  0001 C CNN
+F 3 "" H 10100 1050 50  0001 C CNN
+	1    10100 1050
+	-1   0    0    1
+$EndComp
+$Comp
+L power:GND #PWR0103
+U 1 1 5C5550EF
+P 10200 1050
+F 0 "#PWR0103" H 10200 800 50  0001 C CNN
+F 1 "GND" H 10205 877 50  0000 C CNN
+F 2 "" H 10200 1050 50  0001 C CNN
+F 3 "" H 10200 1050 50  0001 C CNN
+	1    10200 1050
+	1    0    0    -1
+$EndComp
 $EndSCHEMATC

Commit message: EOD sync
Changed lines of the file:
@@
 L Graphic:Logo_Open_Hardware_Large #LOGO1
 U 1 1 5BB7E327
-P 8100 5250
-F 0 "#LOGO1" H 8100 5750 50  0001 C CNN
-F 1 "Logo_Open_Hardware_Large" H 8100 4850 50  0001 C CNN
-F 2 "" H 8100 5250 50  0001 C CNN
-F 3 "~" H 8100 5250 50  0001 C CNN
-	1    8100 5250
+P 7950 5150
+F 0 "#LOGO1" H 7950 5650 50  0000 C CNN
+F 1 "Logo_Open_Hardware_Large" H 7950 4750 50  0001 C CNN
+F 2 "" H 7950 5150 50  0001 C CNN
+F 3 "~" H 7950 5150 50  0001 C CNN
+	1    7950 5150
 	1    0    0    -1
 $EndComp
@@
 	0    1    1    0
 $EndComp
-$Comp
-L power:+5V #PWR068
-U 1 1 5F5531AD
-P 14100 7750
-F 0 "#PWR068" H 14100 7600 50  0001 C CNN
-F 1 "+5V" H 14115 7923 50  0000 C CNN
-F 2 "" H 14100 7750 50  0001 C CNN
-F 3 "" H 14100 7750 50  0001 C CNN
-	1    14100 7750
-	0    1    1    0
-$EndComp
 Wire Wire Line
 	9450 5850 9400 5850
@@
 Text Label 6850 5700 0    50   ~ 0
 D1
+$Comp
+L Connector:Conn_01x02_Male J3
+U 1 1 5C554E39
+P 10200 850
+F 0 "J3" V 10260 890 50  0000 L CNN
+F 1 "Conn_01x02_Male" V 10351 890 50  0000 L CNN
+F 2 "Connector_PinHeader_1.00mm:PinHeader_1x02_P1.00mm_Vertical" H 10200 850 50  0001 C CNN
+F 3 "~" H 10200 850 50  0001 C CNN
+	1    10200 850
+	0    1    1    0
+$EndComp
+$Comp
+L power:+3.3V #PWR0102
+U 1 1 5C554FE5
+P 10100 1050
+F 0 "#PWR0102" H 10100 900 50  0001 C CNN
+F 1 "+3.3V" H 10115 1223 50  0000 C CNN
+F 2 "" H 10100 1050 50  0001 C CNN
+F 3 "" H 10100 1050 50  0001 C CNN
+	1    10100 1050
+	-1   0    0    1
+$EndComp
+$Comp
+L power:GND #PWR0103
+U 1 1 5C5550EF
+P 10200 1050
+F 0 "#PWR0103" H 10200 800 50  0001 C CNN
+F 1 "GND" H 10205 877 50  0000 C CNN
+F 2 "" H 10200 1050 50  0001 C CNN
+F 3 "" H 10200 1050 50  0001 C CNN
+	1    10200 1050
+	1    0    0    -1
+$EndComp
 Wire Bus Line
-	1650 8050 2150 8050
+	4050 4850 4050 6700
+$Comp
+L power:GND #PWR0104
+U 1 1 5C5714FE
+P 11900 6900
+F 0 "#PWR0104" H 11900 6650 50  0001 C CNN
+F 1 "GND" V 11905 6772 50  0000 R CNN
+F 2 "" H 11900 6900 50  0001 C CNN
+F 3 "" H 11900 6900 50  0001 C CNN
+	1    11900 6900
+	0    -1   -1   0
+$EndComp
+$Comp
+L power:+5V #PWR0105
+U 1 1 5C571784
+P 11900 9700
+F 0 "#PWR0105" H 11900 9550 50  0001 C CNN
+F 1 "+5V" H 11915 9873 50  0000 C CNN
+F 2 "" H 11900 9700 50  0001 C CNN
+F 3 "" H 11900 9700 50  0001 C CNN
+	1    11900 9700
+	0    1    1    0
+$EndComp
+$Comp
+L power:GND #PWR0106
+U 1 1 5C57216C
+P 11900 9900
+F 0 "#PWR0106" H 11900 9650 50  0001 C CNN
+F 1 "GND" V 11905 9772 50  0000 R CNN
+F 2 "" H 11900 9900 50  0001 C CNN
+F 3 "" H 11900 9900 50  0001 C CNN
+	1    11900 9900
+	0    -1   -1   0
+$EndComp
 Wire Bus Line
-	10350 9800 10350 11000
-Wire Wire Line
-	3900 4850 4150 4850
+	1650 8050 2150 8050
 Wire Wire Line
 	2550 6350 4750 6350
@@
 	3500 5650 4400 5650
 Wire Bus Line
+	10350 9800 10350 11000
+Wire Wire Line
+	3900 4850 4150 4850
+Wire Bus Line
 	6650 5550 7350 5550
 Wire Bus Line
@@
 	2150 9700 5950 9700
 Wire Bus Line
-	4050 4850 4050 6700
-Wire Bus Line
 	3400 11000 10350 11000
 Wire Bus Line
@@
 	2150 8000 5850 8000
 $Comp
-L Connector:Conn_01x02_Male J3
-U 1 1 5C554E39
-P 10200 850
-F 0 "J3" V 10260 890 50  0000 L CNN
-F 1 "Conn_01x02_Male" V 10351 890 50  0000 L CNN
-F 2 "Connector_PinHeader_1.00mm:PinHeader_1x02_P1.00mm_Vertical" H 10200 850 50  0001 C CNN
-F 3 "~" H 10200 850 50  0001 C CNN
-	1    10200 850
+L power:+3.3V #PWR?
+U 1 1 5C5D25E7
+P 14100 7750
+F 0 "#PWR?" H 14100 7600 50  0001 C CNN
+F 1 "+3.3V" V 14115 7878 50  0000 L CNN
+F 2 "" H 14100 7750 50  0001 C CNN
+F 3 "" H 14100 7750 50  0001 C CNN
+	1    14100 7750
 	0    1    1    0
 $EndComp
-$Comp
-L power:+3.3V #PWR0102
-U 1 1 5C554FE5
-P 10100 1050
-F 0 "#PWR0102" H 10100 900 50  0001 C CNN
-F 1 "+3.3V" H 10115 1223 50  0000 C CNN
-F 2 "" H 10100 1050 50  0001 C CNN
-F 3 "" H 10100 1050 50  0001 C CNN
-	1    10100 1050
-	-1   0    0    1
-$EndComp
-$Comp
-L power:GND #PWR0103
-U 1 1 5C5550EF
-P 10200 1050
-F 0 "#PWR0103" H 10200 800 50  0001 C CNN
-F 1 "GND" H 10205 877 50  0000 C CNN
-F 2 "" H 10200 1050 50  0001 C CNN
-F 3 "" H 10200 1050 50  0001 C CNN
-	1    10200 1050
-	1    0    0    -1
-$EndComp
 $EndSCHEMATC

Commit message: Some relabeling and cleanup of CGA-card
Parts:
- J1: symbol Connector:Bus_ISA_8bit -> VGA-GraphicsAdapter-rescue:Bus_ISA_8bit-Connector
- U10: symbol MCU_Microchip_ATmega:ATmega644P-20PU -> VGA-GraphicsAdapter-rescue:ATmega644P-20PU-MCU_Microchip_ATmega
Connections:
- net labels added: VA0, VA1, VA10, VA11, VA12, VA13, VA14, VA15, VA16, VA17, VA2, VA3, VA4, VA5, VA6, VA7, VA8, VA9, XA0, XA1, XA10, XA11, XA12, XA13, XA14, XA15, XA16, XA17, XA2, XA3, XA4, XA5, XA6, XA7, XA8, XA9
- net labels removed: A16, A17, Clock, VRAM
- wire segments 547 -> 546

Commit message: Started on Rev 4.0
started on a +3.3V main circuit. Bigger RAM, can now additionally support EGA and TGA through firmware if memory map doesn't collide in a non compatible way.
Parts:
- removed U11, U12: 628128, SMD_Packages:SOJ-32, symbol Memory_RAM:628128
- removed U14: 74LS245, Package_DIP:DIP-20_W7.62mm_Socket, symbol 74xx:74LS245
- added U11: IS61LV5128AL-10TLI, Package_SO:TSSOP-44_4.4x11.2mm_P0.5mm, symbol IS61LV5128AL-10TLI:IS61LV5128AL-10TLI
- added U12: 74LS245, Package_DIP:DIP-20_W7.62mm_Socket, symbol 74xx:74LS245
- added unit 1 of U2
- U13: footprint digikey-footprints:DIP-20_W7.62mm -> Package_DIP:DIP-20_W7.62mm_Socket
- U22: value 74LS245 -> 74LS245A; footprint Package_DIP:DIP-22_W7.62mm_Socket -> Package_DIP:DIP-20_W7.62mm_Socket
- U7, U9: value 74LS245 -> 74LS245A
Connections:
- net labels added: GEnd(inv), VA18, XA18
- net labels removed: CS, CS(inv), CountReset
- wire segments 546 -> 514
Other:
- moved on the sheet: RN1, U17, U18, U19, U1A, U1B, U20, U23, U24, U25, U26, U27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

Commit message: Fixed some schematics errors, EOD sync
Parts:
- added H1, H2: MountingHole, MountingHole:MountingHole_2.2mm_M2, symbol Mechanical:MountingHole
- U11: symbol IS61LV5128AL-10TLI:IS61LV5128AL-10TLI -> VGA-GraphicsAdapter-rescue:IS61LV5128AL-10TLI-IS61LV5128AL-10TLI
Changed lines of the file:
@@
 Entry Wire Line
 	5850 8000 5950 8100
-Text GLabel 11850 4250 0    50   BiDi ~ 0
+Text GLabel 11850 4350 0    50   BiDi ~ 0
 GClock
 $Comp
@@
 Wire Wire Line
 	4300 1200 4050 1200
-Text GLabel 4050 1100 2    50   BiDi ~ 0
+Text GLabel 14100 6950 2    50   BiDi ~ 0
 DE
 Text GLabel 11850 4450 0    50   BiDi ~ 0
@@
 $EndComp
 $Comp
-L IS61LV5128AL-10TLI:IS61LV5128AL-10TLI U11
+L VGA-GraphicsAdapter-rescue:IS61LV5128AL-10TLI-IS61LV5128AL-10TLI U11
 U 1 1 5C745693
 P 5300 3500
@@
 Wire Bus Line
 	2150 8000 2150 9700
-Wire Wire Line
-	3550 5550 4250 5550
-Wire Wire Line
-	3600 5450 4200 5450
+Text GLabel 6050 3150 2    50   BiDi ~ 0
+LoadEnable
+$Comp
+L power:GND #PWR0142
+U 1 1 5ED95BF7
+P 4550 3150
+F 0 "#PWR0142" H 4550 2900 50  0001 C CNN
+F 1 "GND" H 4555 2977 50  0000 C CNN
+F 2 "" H 4550 3150 50  0001 C CNN
+F 3 "" H 4550 3150 50  0001 C CNN
+	1    4550 3150
+	0    1    1    0
+$EndComp
 Wire Wire Line
 	3450 6050 4050 6050
@@
 	1650 8000 2150 8000
 Wire Wire Line
-	3650 5350 4150 5350
-Wire Wire Line
 	3500 5650 4050 5650
 Wire Bus Line
@@
 Wire Wire Line
 	3700 5250 4100 5250
-Wire Bus Line
-	4050 4850 4050 5650
+Wire Wire Line
+	3650 5350 4150 5350
+Wire Wire Line
+	3600 5450 4200 5450
+Wire Wire Line
+	3550 5550 4250 5550
 Wire Bus Line
 	4400 3350 4400 4800
@@
 	9850 8950 9850 9800
 Wire Bus Line
+	4050 4850 4050 5650
+Wire Bus Line
 	4050 5650 4050 6700
 Wire Bus Line
@@
 Wire Bus Line
 	2150 8000 5950 8000
-Text GLabel 6050 3150 2    50   BiDi ~ 0
-LoadEnable
 $Comp
-L power:GND #PWR?
-U 1 1 5ED95BF7
-P 4550 3150
-F 0 "#PWR?" H 4550 2900 50  0001 C CNN
-F 1 "GND" H 4555 2977 50  0000 C CNN
-F 2 "" H 4550 3150 50  0001 C CNN
-F 3 "" H 4550 3150 50  0001 C CNN
-	1    4550 3150
-	0    1    1    0
+L Mechanical:MountingHole H1
+U 1 1 5C63632C
+P 15550 1450
+F 0 "H1" H 15650 1496 50  0000 L CNN
+F 1 "MountingHole" H 15650 1405 50  0000 L CNN
+F 2 "MountingHole:MountingHole_2.2mm_M2" H 15550 1450 50  0001 C CNN
+F 3 "~" H 15550 1450 50  0001 C CNN
+	1    15550 1450
+	1    0    0    -1
+$EndComp
+$Comp
+L Mechanical:MountingHole H2
+U 1 1 5C6363FC
+P 15550 6150
+F 0 "H2" H 15650 6196 50  0000 L CNN
+F 1 "MountingHole" H 15650 6105 50  0000 L CNN
+F 2 "MountingHole:MountingHole_2.2mm_M2" H 15550 6150 50  0001 C CNN
+F 3 "~" H 15550 6150 50  0001 C CNN
+	1    15550 6150
+	1    0    0    -1
 $EndComp
 $EndSCHEMATC
