File: Motherboard/HDD.sch (KiCad schematic (older format))
At the start: 3 parts, among them J1 SD_Connector, U39 ATF750LVC, U7 ATmega328-PU

Commit message: from pc sync
Parts:
- U39: symbol fdc:ATF750LVC -> Motherboard-rescue:ATF750LVC-fdc
- U7: symbol MCU_Microchip_ATmega:ATmega328-PU -> Motherboard-rescue:ATmega328-PU-MCU_Microchip_ATmega
Changed lines of the file:
@@
 $EndDescr
 $Comp
-L MCU_Microchip_ATmega:ATmega328-PU U7
+L Motherboard-rescue:ATmega328-PU-MCU_Microchip_ATmega U7
 U 1 1 5C0AE12C
 P 9700 2875
@@
 SCK
 $Comp
-L fdc:ATF750LVC U39
+L Motherboard-rescue:ATF750LVC-fdc U39
 U 1 1 5C45A3F7
 P 5900 3450
