File: Motherboard/HDD.sch (KiCad schematic (older format))
At the start: 3 parts, among them J1 SD_Connector, U39 ATF750LVC, U7 ATmega328-PU

Commit message: LARGE sync
Other:
- note added: "Port 32xh"
Changed lines of the file:
@@
 EESchema Schematic File Version 4
 LIBS:Motherboard-cache
-EELAYER 26 0
+EELAYER 29 0
 EELAYER END
 $Descr A4 11693 8268
@@
 Wire Wire Line
 	8775 2775 9100 2775
+Text Notes 5725 2375 0    50   ~ 0
+Port 32xh
 Wire Bus Line
 	8675 2525 8675 2675

Commit message: Large Sync
Parts:
- J1: symbol Connector_Generic:Conn_02x03_Counter_Clockwise -> Motherboard-rescue:Conn_02x03_Counter_Clockwise-Connector_Generic
Changed lines of the file:
@@
 	8550 3575 9100 3575
 $Comp
-L power:GND #PWR07
+L Motherboard-rescue:GND-power #PWR07
 U 1 1 5C0B5FAE
 P 7050 5425
@@
 $EndComp
 $Comp
-L power:+5V #PWR08
+L Motherboard-rescue:+5V-power #PWR08
 U 1 1 5C0B60D5
 P 7050 4925
@@
 $EndComp
 $Comp
-L power:+5V #PWR013
+L Motherboard-rescue:+5V-power #PWR013
 U 1 1 5C0BB8CB
 P 10300 4075
@@
 $EndComp
 $Comp
-L power:+5V #PWR011
+L Motherboard-rescue:+5V-power #PWR011
 U 1 1 5C0BB915
 P 9650 4425
@@
 	9650 4375 9700 4375
 $Comp
-L power:GND #PWR012
+L Motherboard-rescue:GND-power #PWR012
 U 1 1 5C0BD791
 P 9700 1375
@@
 A[0...19]
 $Comp
-L Connector_Generic:Conn_02x03_Counter_Clockwise J1
+L Motherboard-rescue:Conn_02x03_Counter_Clockwise-Connector_Generic J1
 U 1 1 5C17F343
 P 7150 5125
@@
 A5
 $Comp
-L power:GND #PWR09
+L Motherboard-rescue:GND-power #PWR09
 U 1 1 5C46903C
 P 5175 3950
@@
 $EndComp
 $Comp
-L power:+5V #PWR010
+L Motherboard-rescue:+5V-power #PWR010
 U 1 1 5C469186
 P 6625 2850
