File: Motherboard/Motherboard.kicad_pcb (KiCad board)
At the start: 2 copper layers, 244.1 x 244.2 mm, 75 parts, among them J1 SD_Connector, J2 Bus_ISA_8bit, J3 Bus_ISA_8bit, J4 ATX24, J5 Bus_ISA_8bit, J6 Bus_ISA_8bit, J7 Bus_ISA_8bit, J8 3.3V_HEADER, SW1 TURBO, SW2 FREEZE, SW3 SW_SPST_LED, SW4 RESET, SW5 SW_DIP_x01, U1 82C54_PLCC, U15 74LS257, U2 8088, U22 74HC74, U23 8237, U24 74LS04, U25 74LS573, U26 74LS573, U27 74LS670, U28 8288, U29 74LS245, U3 8259, U30 74LS04, U31 74LS573, U32 74LS244, U33 74LS573, U34 74LS04, U35 74LS04, U36 74LS00, U37 74LS00, U38 74LS10, U39 ATF750LVC, U4 CD40147, U40 74LS27, U41 74LS04, U43 74LS244, U44 74LS244, U45 74LS244, U46 74LS245, U47 4077, U48 SST39SF010, U49 74LS243, U5 ATF750LVC, U50 74LS04, U51 ATF750LVC, U52 74LS74, U53 74LS00, U54 74LS08, U55 74LS138, U56 4077, U57 DS1100Z-100+ (TTLDL-20), U7 ATmega328-PU, U9 40106, Y1 14.31818 MHz, Y2 24.000 MHz

Commit message: Revert "sync"
This reverts commit d2aa285ba7e3cb3ef6eb4c4ce9647a2fe4c4c3fa.
Parts:
- moved RN2 256.8 mm to (346.8, 131.0), turned to 0 degrees
Routing:
- net /IO-Decoder/XA8: track 117.8 -> 0.00 mm, vias 3 -> 0
- net /IO-Decoder/XA14: track 109.9 -> 0.00 mm, vias 3 -> 0
- net /IO-Decoder/XA9: track 106.1 -> 0.00 mm, vias 3 -> 0
- net /IO-Decoder/XA13: track 99.4 -> 0.00 mm, vias 3 -> 0
- net /IO-Decoder/XA12: track 93.4 -> 0.00 mm, vias 3 -> 0
- net /IO-Decoder/XA10: track 89.9 -> 0.00 mm, vias 2 -> 0
- net /IO-Decoder/XA11: track 86.7 -> 0.00 mm, vias 3 -> 0
- net /IO-Decoder/XA3: track 68.8 -> 0.00 mm, vias 2 -> 0
- net /IO-Decoder/XA2: track 65.8 -> 0.00 mm, vias 2 -> 0
- net /IO-Decoder/XA1: track 65.0 -> 0.00 mm, vias 3 -> 0
- net /IO-Decoder/XA0: track 62.1 -> 0.00 mm, vias 3 -> 0
- net /IO-Decoder/XA4: track 58.6 -> 0.00 mm, vias 3 -> 0
- net +5V: track 275.2 -> 217.1 mm, vias 2 -> 0
- net /IO-Decoder/XA5: track 51.2 -> 0.00 mm, vias 3 -> 0
- net /IO-Decoder/A12: track 44.1 -> 0.00 mm, vias 2 -> 0
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Other:
- board text added: "Are these reversible?"

Commit message: Revert "Revert "sync""
This reverts commit dae598a70117e78f748d18ec5b1edcfaf1b843c6.
Parts:
- moved RN2 256.8 mm to (110.8, 29.8), turned to 270 degrees
Routing:
- net /IO-Decoder/XA8: track 0.00 -> 117.8 mm, vias 0 -> 3
- net /IO-Decoder/XA14: track 0.00 -> 109.9 mm, vias 0 -> 3
- net /IO-Decoder/XA9: track 0.00 -> 106.1 mm, vias 0 -> 3
- net /IO-Decoder/XA13: track 0.00 -> 99.4 mm, vias 0 -> 3
- net /IO-Decoder/XA12: track 0.00 -> 93.4 mm, vias 0 -> 3
- net /IO-Decoder/XA10: track 0.00 -> 89.9 mm, vias 0 -> 2
- net /IO-Decoder/XA11: track 0.00 -> 86.7 mm, vias 0 -> 3
- net /IO-Decoder/XA3: track 0.00 -> 68.8 mm, vias 0 -> 2
- net /IO-Decoder/XA2: track 0.00 -> 65.8 mm, vias 0 -> 2
- net /IO-Decoder/XA1: track 0.00 -> 65.0 mm, vias 0 -> 3
- net /IO-Decoder/XA0: track 0.00 -> 62.1 mm, vias 0 -> 3
- net /IO-Decoder/XA4: track 0.00 -> 58.6 mm, vias 0 -> 3
- net +5V: track 217.1 -> 275.2 mm, vias 0 -> 2
- net /IO-Decoder/XA5: track 0.00 -> 51.2 mm, vias 0 -> 3
- net /IO-Decoder/A12: track 0.00 -> 44.1 mm, vias 0 -> 2
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Other:
- board text removed: "Are these reversible?"
