File: Motherboard/Motherboard.kicad_pcb (KiCad board)
At the start: 2 copper layers, 43 parts, among them J1 SD_Card, SW1 TURBO, SW2 FREEZE, U1 82C54_PLCC, U10 4081, U11 4081, U12 74LS32, U13 74LS14, U14 74LS77, U15 74LS257, U16 4069, U17 74LS32, U18 4081, U19 74HC74, U2 8088_Max_Mode, U20 7402, U21 40106, U22 74HC74, U23 8237, U24 74LS04, U25 74LS573, U26 74LS573, U27 74LS670, U3 8259, U4 4081, U5 4001, U6 4081, U7 ATmega328-PU, U8 4069, U9 40106, Y1 18.432 MHz, Y2 32.768 MHz

Commit message: Added ISA Footprint
Parts:
- removed REF***: OSHW-Logo_28.5x30mm_SilkScreen, Symbols:OSHW-Logo_28.5x30mm_SilkScreen
- removed RN1: 50k, Resistors_THT:R_Array_SIP6
- added J2: Bus_ISA_8bit, RetPC:ISA-8-bit, F.Cu at (288.7, 93.4)
- added J3: Bus_ISA_8bit, RetPC:ISA-8-bit, F.Cu at (296.0, 93.4)
- J1: value SD_Card -> SD_Connector; footprint Connectors:SD_Card_Receptacle -> Connectors_Molex:Molex_KK-6410-06_06x2.54mm_Straight
- U1: footprint Housings_LCC:PLCC-28_THT-Socket -> Housings_DIP:DIP-28_W15.24mm_Socket
- U6: footprint Housings_DIP:DIP-40_W15.24mm_Socket -> Housings_DIP:DIP-14_W7.62mm_Socket
- moved U5 231.8 mm to (40.6, 134.0)
- moved U4 230.2 mm to (17.8, 130.2)
- moved U6 209.5 mm to (17.8, 151.8)
- moved J1 28.3 mm to (57.8, 171.4)
Connections:
- J1 pad 1: Net-(J1-Pad1) -> /HDD Controller/MISO
- J1 pad 2: Net-(J1-Pad2) -> /HDD Controller/SCK
- J1 pad 3: GND -> +5V
- J1 pad 4: +5V -> GND
- J1 pad 5: Net-(J1-Pad5) -> /HDD Controller/SS-CS
- J1 pad 6: GND -> /HDD Controller/MOSI
- U7 pad 16: Net-(J1-Pad1) -> /HDD Controller/SS-CS
- U7 pad 17: Net-(J1-Pad2) -> /HDD Controller/MOSI
- U7 pad 18: Net-(J1-Pad7) -> /HDD Controller/MISO
- U7 pad 19: Net-(J1-Pad5) -> /HDD Controller/SCK
Routing:
- net /HDD Controller/ADDR_LO: track 0.00 -> 78.3 mm
- net /A8: track 0.00 -> 65.6 mm
- net /A9: track 0.00 -> 63.1 mm
- net Net-(J1-Pad5): track 58.6 -> 0.00 mm, vias 1 -> 0
- net /A19: track 0.00 -> 56.3 mm
- net /A18: track 0.00 -> 54.2 mm, vias 0 -> 1
- net /A13: track 0.00 -> 50.9 mm
- net Net-(J1-Pad7): track 49.2 -> 0.00 mm, vias 2 -> 0
- net /A5: track 44.6 -> 92.8 mm, vias 0 -> 1
- net Net-(J1-Pad1): track 34.1 -> 0.00 mm
- net Net-(U4-Pad6): track 0.00 -> 30.2 mm
- net Net-(U5-Pad11): track 0.00 -> 29.8 mm, vias 0 -> 1
- net Net-(J1-Pad2): track 29.5 -> 0.00 mm
- net Net-(J1-Pad8): track 29.0 -> 0.00 mm, vias 1 -> 0
- net /HDD Controller/SCK: track 0.00 -> 23.1 mm
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
Commit message: A VERY large sync...
Parts:
- added J4: ATX24, Connectors_Molex:Molex_MiniFit-JR-5556-24B_2x12x4.20mm_Straight, F.Cu at (24.1, 179.1)
- added R6: 1k, Resistors_THT:R_Axial_DIN0204_L3.6mm_D1.6mm_P2.54mm_Vertical, F.Cu at (38.1, 190.5)
- added R7: 220, Resistors_THT:R_Axial_DIN0204_L3.6mm_D1.6mm_P2.54mm_Vertical, F.Cu at (31.8, 203.2)
- added R8: 1k, Resistors_THT:R_Axial_DIN0204_L3.6mm_D1.6mm_P2.54mm_Vertical, F.Cu at (30.5, 190.5)
- added SW3: SW_SPST_LED, Pin_Headers:Pin_Header_Straight_1x04_Pitch2.00mm, F.Cu at (36.8, 196.8)
- added SW4: RESET, Pin_Headers:Pin_Header_Straight_1x02_Pitch2.00mm, F.Cu at (31.8, 196.8)
- moved J2 169.0 mm to (121.3, 70.7)
- moved J3 154.9 mm to (142.7, 70.7)
Connections:
- J2 pad 1: Net-(J2-Pad1) -> GND
- J2 pad 10: Net-(J2-Pad10) -> GND
- J2 pad 29: Net-(J2-Pad29) -> +5V
- J2 pad 3: Net-(J2-Pad3) -> +5V
- J2 pad 31: Net-(J2-Pad31) -> GND
- J2 pad 5: Net-(J2-Pad5) -> -5V
- J2 pad 7: Net-(J2-Pad7) -> -12V
- J2 pad 9: Net-(J2-Pad9) -> +12V
- J3 pad 1: Net-(J3-Pad1) -> GND
- J3 pad 10: Net-(J3-Pad10) -> GND
- J3 pad 29: Net-(J3-Pad29) -> +5V
- J3 pad 3: Net-(J3-Pad3) -> +5V
- J3 pad 31: Net-(J3-Pad31) -> GND
- J3 pad 5: Net-(J3-Pad5) -> -5V
- J3 pad 7: Net-(J3-Pad7) -> -12V
- J3 pad 9: Net-(J3-Pad9) -> +12V
- U22 pad 3: /DMA/CLK -> /SYS_CLK
- U23 pad 13: /DMA/RESET -> /RESET
- U23 pad 15: /DMA/DACK3 -> /DACK3
- U23 pad 16: /DMA/DREQ3 -> /DREQ3
- U23 pad 6: /DMA/READY -> /READY
- U27 pad 5: /DMA/DACK3 -> /DACK3
Routing:
- net /Divisible Clock/~RES: track 0.00 -> 115.9 mm, vias 0 -> 2
- net /A6: track 44.6 -> 89.7 mm, vias 0 -> 2
- net /A15: track 0.00 -> 33.0 mm, vias 0 -> 1
- net /A17: track 0.00 -> 31.1 mm
- net /A16: track 0.00 -> 28.3 mm
- net /A14: track 0.00 -> 23.1 mm
- net Net-(J4-Pad16): track 0.00 -> 18.5 mm
- net +3V3: track 0.00 -> 9.70 mm
- net Net-(R6-Pad1): track 0.00 -> 8.88 mm
- net Net-(R8-Pad1): track 0.00 -> 7.42 mm
- net Net-(R7-Pad2): track 0.00 -> 6.28 mm
- net /HDD Controller/ADDR_LO: vias 0 -> 1
Other:
- net class Power added: clearance 0.2, trace_width 0.4, via_dia 0.8, via_drill 0.4

Commit message: Large sync
Parts:
- added R10: 470R, Resistors_THT:R_Axial_DIN0204_L3.6mm_D1.6mm_P7.62mm_Horizontal, F.Cu at (252.5, 128.4)
- added R11: 6k2, Resistors_THT:R_Axial_DIN0204_L3.6mm_D1.6mm_P7.62mm_Horizontal, F.Cu at (242.9, 128.4)
- added R9: R, Resistors_THT:R_Axial_DIN0204_L3.6mm_D1.6mm_P7.62mm_Horizontal, F.Cu at (231.3, 130.9)
- added REF***: OSHW-Logo_5.7x6mm_SilkScreen, Symbols:OSHW-Logo_5.7x6mm_SilkScreen, F.Cu at (16.4, 21.6)
- added SW5: SW_DIP_x01, Housings_DIP:DIP-4_W7.62mm, F.Cu at (221.6, 128.1)
- added U29: 74LS245, Housings_DIP:DIP-20_W7.62mm_Socket, F.Cu at (251.2, 31.6)
- added U30: 74LS04, Housings_DIP:DIP-14_W7.62mm_Socket, F.Cu at (272.7, 57.7)
- added U31: 74LS573, Housings_DIP:DIP-20_W7.62mm_Socket, F.Cu at (261.9, 31.6)
- added U32: 74LS244, Housings_DIP:DIP-20_W7.62mm_Socket, F.Cu at (240.4, 57.7)
- added U33: 74LS573, Housings_DIP:DIP-20_W7.62mm_Socket, F.Cu at (251.2, 57.7)
- added U34: 74LS04, Housings_DIP:DIP-14_W7.62mm_Socket, F.Cu at (254.3, 91.8)
- added U35: 74LS04, Housings_DIP:DIP-14_W7.62mm_Socket, F.Cu at (275.8, 91.8)
- added U36: 74LS00, Housings_DIP:DIP-14_W7.62mm_Socket, F.Cu at (275.8, 110.3)
- added U37: 74LS00, Housings_DIP:DIP-14_W7.62mm_Socket, F.Cu at (265.0, 110.3)
- added U38: 74LS10, Housings_DIP:DIP-14_W7.62mm_Socket, F.Cu at (286.5, 91.8)
- added U39: ATF750LVC, Housings_DIP:DIP-28_W7.62mm_Socket, F.Cu at (326.7, 31.6)
- added U40: 74LS27, Housings_DIP:DIP-14_W7.62mm_Socket, F.Cu at (304.9, 31.6)
- added U41: 74LS04, Housings_DIP:DIP-14_W7.62mm_Socket, F.Cu at (283.4, 57.7)
- added U42: 74LS157, Housings_SOIC:SOIC-16_3.9x9.9mm_Pitch1.27mm, F.Cu at (288.7, 114.0)
- added U43: 74LS244, Housings_DIP:DIP-20_W7.62mm_Socket, F.Cu at (283.4, 31.6)
- added U44: 74LS244, Housings_DIP:DIP-20_W7.62mm_Socket, F.Cu at (261.9, 57.7)
- added U45: 74LS244, Housings_DIP:DIP-20_W7.62mm_Socket, F.Cu at (272.7, 31.6)
- added U46: 74LS245, Housings_DIP:DIP-20_W7.62mm_Socket, F.Cu at (240.4, 31.6)
- added U47: 4077, Housings_DIP:DIP-14_W7.62mm_Socket, F.Cu at (294.2, 31.6)
- added U48: SST39SF010, Housings_DIP:DIP-32_W15.24mm_Socket, F.Cu at (222.0, 31.6)
- added U49: 74LS243, Housings_DIP:DIP-12_W7.62mm_Socket, F.Cu at (294.2, 50.1)
- added U50: 74LS04, Housings_DIP:DIP-14_W7.62mm_Socket, F.Cu at (243.5, 91.8)
- added U51: ATF750LVC, Housings_DIP:DIP-28_W7.62mm_Socket, F.Cu at (222.0, 91.8)
- added U52: 74LS74, Housings_DIP:DIP-14_W7.62mm_Socket, F.Cu at (232.8, 112.9)
- added U53: 74LS00, Housings_DIP:DIP-14_W7.62mm_Socket, F.Cu at (243.5, 110.3)
- added U54: 74LS08, Housings_DIP:DIP-14_W7.62mm_Socket, F.Cu at (254.3, 110.3)
- added U55: 74LS138, Housings_DIP:DIP-16_W7.62mm_Socket, F.Cu at (232.8, 91.8)
- added U56: 4077, Housings_DIP:DIP-14_W7.62mm_Socket, F.Cu at (265.0, 91.8)
- added U57: DS1100Z-100+ (TTLDL-20), Housings_SOIC:SOIC-8_3.9x4.9mm_Pitch1.27mm, F.Cu at (264.9, 129.9)
Connections:
- J2 pad 11: Net-(J2-Pad11) -> (no net)
- J2 pad 12: Net-(J2-Pad12) -> (no net)
- J2 pad 13: Net-(J2-Pad13) -> (no net)
- J2 pad 14: Net-(J2-Pad14) -> (no net)
- J2 pad 15: Net-(J2-Pad15) -> (no net)
- J2 pad 16: Net-(J2-Pad16) -> (no net)
- J2 pad 17: Net-(J2-Pad17) -> (no net)
- J2 pad 18: Net-(J2-Pad18) -> (no net)
- J2 pad 19: Net-(J2-Pad19) -> (no net)
- J2 pad 2: Net-(J2-Pad2) -> /ISA/RESET
- J2 pad 20: Net-(J2-Pad20) -> (no net)
- J2 pad 21: Net-(J2-Pad21) -> (no net)
- J2 pad 22: Net-(J2-Pad22) -> (no net)
- J2 pad 23: Net-(J2-Pad23) -> (no net)
- J2 pad 24: Net-(J2-Pad24) -> (no net)
- J2 pad 25: Net-(J2-Pad25) -> (no net)
- J2 pad 26: Net-(J2-Pad26) -> (no net)
- J2 pad 27: Net-(J2-Pad27) -> (no net)
- J2 pad 28: Net-(J2-Pad28) -> (no net)
- J2 pad 30: Net-(J2-Pad30) -> (no net)
- J2 pad 32: Net-(J2-Pad32) -> (no net)
- J2 pad 33: Net-(J2-Pad33) -> (no net)
- J2 pad 34: Net-(J2-Pad34) -> (no net)
- J2 pad 35: Net-(J2-Pad35) -> (no net)
- J2 pad 36: Net-(J2-Pad36) -> (no net)
- J2 pad 37: Net-(J2-Pad37) -> (no net)
- J2 pad 38: Net-(J2-Pad38) -> (no net)
- J2 pad 39: Net-(J2-Pad39) -> (no net)
- J2 pad 4: Net-(J2-Pad4) -> (no net)
- J2 pad 40: Net-(J2-Pad40) -> (no net)
- J2 pad 41: Net-(J2-Pad41) -> (no net)
- J2 pad 42: Net-(J2-Pad42) -> (no net)
- J2 pad 43: Net-(J2-Pad43) -> (no net)
- J2 pad 44: Net-(J2-Pad44) -> (no net)
- J2 pad 45: Net-(J2-Pad45) -> (no net)
- J2 pad 46: Net-(J2-Pad46) -> (no net)
- J2 pad 47: Net-(J2-Pad47) -> (no net)
- J2 pad 48: Net-(J2-Pad48) -> (no net)
- J2 pad 49: Net-(J2-Pad49) -> (no net)
- J2 pad 50: Net-(J2-Pad50) -> (no net)
- J2 pad 51: Net-(J2-Pad51) -> (no net)
- J2 pad 52: Net-(J2-Pad52) -> (no net)
- J2 pad 53: Net-(J2-Pad53) -> (no net)
- J2 pad 54: Net-(J2-Pad54) -> (no net)
- J2 pad 55: Net-(J2-Pad55) -> (no net)
- J2 pad 56: Net-(J2-Pad56) -> (no net)
- J2 pad 57: Net-(J2-Pad57) -> (no net)
- J2 pad 58: Net-(J2-Pad58) -> (no net)
- J2 pad 59: Net-(J2-Pad59) -> (no net)
- J2 pad 6: Net-(J2-Pad6) -> (no net)
- J2 pad 60: Net-(J2-Pad60) -> (no net)
- J2 pad 61: Net-(J2-Pad61) -> (no net)
- J2 pad 62: Net-(J2-Pad62) -> (no net)
- J2 pad 8: Net-(J2-Pad8) -> (no net)
- J3 pad 11: Net-(J3-Pad11) -> (no net)
- J3 pad 12: Net-(J3-Pad12) -> (no net)
- J3 pad 13: Net-(J3-Pad13) -> (no net)
- J3 pad 14: Net-(J3-Pad14) -> (no net)
- J3 pad 15: Net-(J3-Pad15) -> (no net)
- J3 pad 16: Net-(J3-Pad16) -> (no net)
- J3 pad 17: Net-(J3-Pad17) -> (no net)
- J3 pad 18: Net-(J3-Pad18) -> (no net)
- J3 pad 19: Net-(J3-Pad19) -> (no net)
- J3 pad 2: Net-(J3-Pad2) -> /ISA/RESET
- J3 pad 20: Net-(J3-Pad20) -> (no net)
- J3 pad 21: Net-(J3-Pad21) -> (no net)
- J3 pad 22: Net-(J3-Pad22) -> (no net)
- J3 pad 23: Net-(J3-Pad23) -> (no net)
- J3 pad 24: Net-(J3-Pad24) -> (no net)
- J3 pad 25: Net-(J3-Pad25) -> (no net)
- J3 pad 26: Net-(J3-Pad26) -> (no net)
- J3 pad 27: Net-(J3-Pad27) -> (no net)
- J3 pad 28: Net-(J3-Pad28) -> (no net)
- J3 pad 30: Net-(J3-Pad30) -> (no net)
- J3 pad 32: Net-(J3-Pad32) -> (no net)
- J3 pad 33: Net-(J3-Pad33) -> (no net)
- J3 pad 34: Net-(J3-Pad34) -> (no net)
- J3 pad 35: Net-(J3-Pad35) -> (no net)
- J3 pad 36: Net-(J3-Pad36) -> (no net)
- J3 pad 37: Net-(J3-Pad37) -> (no net)
- J3 pad 38: Net-(J3-Pad38) -> (no net)
- J3 pad 39: Net-(J3-Pad39) -> (no net)
- J3 pad 4: Net-(J3-Pad4) -> (no net)
- J3 pad 40: Net-(J3-Pad40) -> (no net)
- J3 pad 41: Net-(J3-Pad41) -> (no net)
- J3 pad 42: Net-(J3-Pad42) -> (no net)
- J3 pad 43: Net-(J3-Pad43) -> (no net)
- J3 pad 44: Net-(J3-Pad44) -> (no net)
- J3 pad 45: Net-(J3-Pad45) -> (no net)
- J3 pad 46: Net-(J3-Pad46) -> (no net)
- J3 pad 47: Net-(J3-Pad47) -> (no net)
- J3 pad 48: Net-(J3-Pad48) -> (no net)
- J3 pad 49: Net-(J3-Pad49) -> (no net)
- J3 pad 50: Net-(J3-Pad50) -> (no net)
- J3 pad 51: Net-(J3-Pad51) -> (no net)
- J3 pad 52: Net-(J3-Pad52) -> (no net)
- J3 pad 53: Net-(J3-Pad53) -> (no net)
- J3 pad 54: Net-(J3-Pad54) -> (no net)
- J3 pad 55: Net-(J3-Pad55) -> (no net)
- J3 pad 56: Net-(J3-Pad56) -> (no net)
- J3 pad 57: Net-(J3-Pad57) -> (no net)
- J3 pad 58: Net-(J3-Pad58) -> (no net)
- J3 pad 59: Net-(J3-Pad59) -> (no net)
- J3 pad 6: Net-(J3-Pad6) -> (no net)
- J3 pad 60: Net-(J3-Pad60) -> (no net)
- J3 pad 61: Net-(J3-Pad61) -> (no net)
- J3 pad 62: Net-(J3-Pad62) -> (no net)
- J3 pad 8: Net-(J3-Pad8) -> (no net)
- J4 pad 9: /PSU/+5V_SB -> (no net)
- U1 pad 1: Net-(U1-Pad1) -> (no net)
- U1 pad 10: Net-(U1-Pad10) -> (no net)
- U1 pad 11: Net-(U1-Pad11) -> (no net)
- U1 pad 12: Net-(U1-Pad12) -> (no net)
- U1 pad 13: Net-(U1-Pad13) -> (no net)
- U1 pad 14: Net-(U1-Pad14) -> (no net)
- U1 pad 15: Net-(U1-Pad15) -> (no net)
- U1 pad 16: Net-(U1-Pad16) -> (no net)
- U1 pad 17: Net-(U1-Pad17) -> (no net)
- U1 pad 18: Net-(U1-Pad18) -> (no net)
- U1 pad 19: Net-(U1-Pad19) -> (no net)
- U1 pad 2: Net-(U1-Pad2) -> (no net)
- U1 pad 20: Net-(U1-Pad20) -> (no net)
- U1 pad 21: Net-(U1-Pad21) -> (no net)
- U1 pad 22: Net-(U1-Pad22) -> (no net)
- U1 pad 23: Net-(U1-Pad23) -> (no net)
- U1 pad 24: Net-(U1-Pad24) -> (no net)
- U1 pad 25: Net-(U1-Pad25) -> (no net)
- U1 pad 26: Net-(U1-Pad26) -> (no net)
- U1 pad 27: Net-(U1-Pad27) -> (no net)
- U1 pad 28: Net-(U1-Pad28) -> (no net)
- U1 pad 3: Net-(U1-Pad3) -> (no net)
- U1 pad 4: Net-(U1-Pad4) -> (no net)
- U1 pad 5: Net-(U1-Pad5) -> (no net)
- U1 pad 6: Net-(U1-Pad6) -> (no net)
- U1 pad 7: Net-(U1-Pad7) -> (no net)
- U1 pad 8: Net-(U1-Pad8) -> (no net)
- U1 pad 9: Net-(U1-Pad9) -> (no net)
- U10 pad 1: (no net) -> Net-(U10-Pad1)
- U10 pad 2: (no net) -> Net-(U10-Pad2)
- U10 pad 3: (no net) -> Net-(U10-Pad3)
- U10 pad 5: /Divisible Clock/RDY1 -> (no net)
- U11 pad 8: /Divisible Clock/RDY2 -> (no net)
- U12 pad 9: /Divisible Clock/~ASYNC -> (no net)
- U14 pad 6: Net-(U14-Pad6) -> (no net)
- U14 pad 8: Net-(U14-Pad8) -> (no net)
- U15 pad 10: Net-(U15-Pad10) -> (no net)
- U15 pad 11: Net-(U15-Pad11) -> (no net)
- U15 pad 12: Net-(U15-Pad12) -> (no net)
- U15 pad 13: Net-(U15-Pad13) -> (no net)
- U15 pad 14: Net-(U15-Pad14) -> (no net)
- U15 pad 5: Net-(U15-Pad5) -> (no net)
- U15 pad 6: Net-(U15-Pad6) -> (no net)
- U15 pad 7: Net-(U15-Pad7) -> (no net)
- U15 pad 9: Net-(U15-Pad9) -> (no net)
- U18 pad 1: Net-(U18-Pad1) -> (no net)
- U18 pad 2: Net-(U15-Pad4) -> (no net)
- U18 pad 3: Net-(U18-Pad3) -> (no net)
- U19 pad 10: Net-(U19-Pad10) -> (no net)
- U19 pad 11: Net-(U18-Pad1) -> Net-(U15-Pad4)
- U19 pad 13: Net-(U19-Pad13) -> (no net)
- U19 pad 2: Net-(U19-Pad2) -> Net-(U10-Pad3)
- U19 pad 5: Net-(U18-Pad1) -> Net-(U19-Pad12)
- U19 pad 6: Net-(U19-Pad2) -> Net-(U10-Pad1)
- U19 pad 8: Net-(U19-Pad12) -> Net-(U10-Pad2)
- U19 pad 9: Net-(U19-Pad9) -> /SYS_CLK
- U2 pad 10: /A6 -> (no net)
- U2 pad 11: /A5 -> (no net)
- U2 pad 12: /A4 -> (no net)
- U2 pad 13: /A3 -> (no net)
- U2 pad 14: /A2 -> (no net)
- U2 pad 15: /A1 -> (no net)
- U2 pad 16: /A0 -> (no net)
- U2 pad 17: Net-(U2-Pad17) -> (no net)
- U2 pad 18: Net-(U2-Pad18) -> (no net)
- U2 pad 2: /A14 -> (no net)
- U2 pad 23: Net-(U2-Pad23) -> (no net)
- U2 pad 24: Net-(U2-Pad24) -> (no net)
- U2 pad 25: Net-(U2-Pad25) -> (no net)
- U2 pad 26: Net-(U2-Pad26) -> (no net)
- U2 pad 27: Net-(U2-Pad27) -> (no net)
- U2 pad 28: Net-(U2-Pad28) -> (no net)
- U2 pad 29: Net-(U2-Pad29) -> (no net)
- U2 pad 3: /A13 -> (no net)
- U2 pad 30: /HLDA -> (no net)
- U2 pad 31: /HRQ -> (no net)
- U2 pad 32: Net-(U2-Pad32) -> (no net)
- U2 pad 34: Net-(U2-Pad34) -> (no net)
- U2 pad 35: /A19 -> (no net)
- U2 pad 36: /A18 -> (no net)
- U2 pad 37: /A17 -> (no net)
- U2 pad 38: /A16 -> (no net)
- U2 pad 39: /A15 -> (no net)
- U2 pad 4: /A12 -> (no net)
- U2 pad 5: /A11 -> (no net)
- U2 pad 6: /A10 -> (no net)
- U2 pad 7: /A9 -> (no net)
- U2 pad 8: /A8 -> (no net)
- U2 pad 9: /A7 -> (no net)
- U20 pad 1: /SYS_CLK -> (no net)
- U20 pad 2: Net-(U19-Pad9) -> (no net)
- U20 pad 3: Net-(U18-Pad3) -> (no net)
- U22 pad 3: /SYS_CLK -> /DCLK
- U23 pad 1: /DMA/~IOR -> (no net)
- U23 pad 10: /DMA/HRQ -> (no net)
- U23 pad 11: Net-(U23-Pad11) -> (no net)
- U23 pad 17: /DMA/DREQ2 -> (no net)
- U23 pad 18: /DMA/DREQ1 -> (no net)
- U23 pad 19: /DMA/DREQ0 -> (no net)
- U23 pad 2: /DMA/~IOW -> (no net)
- U23 pad 21: Net-(U23-Pad21) -> (no net)
- U23 pad 22: Net-(U23-Pad22) -> (no net)
- U23 pad 23: Net-(U23-Pad23) -> (no net)
- U23 pad 24: /DMA/DACK1 -> (no net)
- U23 pad 25: /DMA/DACK0 -> (no net)
- U23 pad 26: Net-(U23-Pad26) -> (no net)
- U23 pad 27: Net-(U23-Pad27) -> (no net)
- U23 pad 28: Net-(U23-Pad28) -> (no net)
- U23 pad 29: Net-(U23-Pad29) -> (no net)
- U23 pad 3: Net-(U23-Pad3) -> (no net)
- U23 pad 30: Net-(U23-Pad30) -> (no net)
- U23 pad 32: Net-(U23-Pad32) -> (no net)
- U23 pad 33: Net-(U23-Pad33) -> (no net)
- U23 pad 34: Net-(U23-Pad34) -> (no net)
- U23 pad 35: Net-(U23-Pad35) -> (no net)
- U23 pad 37: Net-(U23-Pad37) -> (no net)
- U23 pad 38: Net-(U23-Pad38) -> (no net)
- U23 pad 39: Net-(U23-Pad39) -> (no net)
- U23 pad 4: Net-(U23-Pad4) -> (no net)
- U23 pad 40: Net-(U23-Pad40) -> (no net)
- U23 pad 7: /DMA/HLDA -> (no net)
- U24 pad 4: /DMA/TC -> (no net)
- U25 pad 12: Net-(U25-Pad12) -> (no net)
- U25 pad 13: Net-(U25-Pad13) -> (no net)
- U25 pad 14: Net-(U25-Pad14) -> (no net)
- U25 pad 15: Net-(U25-Pad15) -> (no net)
- U25 pad 16: Net-(U25-Pad16) -> (no net)
- U25 pad 17: Net-(U25-Pad17) -> (no net)
- U25 pad 18: Net-(U25-Pad18) -> (no net)
- U25 pad 19: Net-(U25-Pad19) -> (no net)
- U25 pad 2: Net-(U25-Pad2) -> (no net)
- U25 pad 3: Net-(U25-Pad3) -> (no net)
- U25 pad 4: Net-(U25-Pad4) -> (no net)
- U25 pad 5: Net-(U25-Pad5) -> (no net)
- U25 pad 6: Net-(U25-Pad6) -> (no net)
- U25 pad 7: Net-(U25-Pad7) -> (no net)
- U25 pad 8: Net-(U25-Pad8) -> (no net)
- U25 pad 9: Net-(U25-Pad9) -> (no net)
- U26 pad 12: Net-(U26-Pad12) -> (no net)
- U26 pad 13: Net-(U26-Pad13) -> (no net)
- U26 pad 14: Net-(U26-Pad14) -> (no net)
- U26 pad 15: Net-(U26-Pad15) -> (no net)
- U26 pad 16: Net-(U26-Pad16) -> (no net)
- U26 pad 17: Net-(U26-Pad17) -> (no net)
- U26 pad 18: Net-(U26-Pad18) -> (no net)
- U26 pad 19: Net-(U26-Pad19) -> (no net)
- U26 pad 2: Net-(U26-Pad2) -> (no net)
- U26 pad 3: Net-(U26-Pad3) -> (no net)
- U26 pad 4: Net-(U26-Pad4) -> (no net)
- U26 pad 5: Net-(U26-Pad5) -> (no net)
- U26 pad 6: Net-(U26-Pad6) -> (no net)
- U26 pad 7: Net-(U26-Pad7) -> (no net)
- U26 pad 8: Net-(U26-Pad8) -> (no net)
- U26 pad 9: Net-(U26-Pad9) -> (no net)
- U27 pad 1: Net-(U27-Pad1) -> (no net)
- U27 pad 10: Net-(U27-Pad10) -> (no net)
- U27 pad 12: /DMA/~WRTDMAPGRES -> (no net)
- U27 pad 13: /DMA/A1 -> (no net)
- U27 pad 14: /DMA/A0 -> (no net)
- U27 pad 15: Net-(U27-Pad15) -> (no net)
- U27 pad 16: Net-(U27-Pad16) -> (no net)
- U27 pad 2: Net-(U27-Pad2) -> (no net)
- U27 pad 3: Net-(U27-Pad3) -> (no net)
- U27 pad 6: Net-(U27-Pad6) -> (no net)
- U27 pad 7: Net-(U27-Pad7) -> (no net)
- U27 pad 8: Net-(U27-Pad8) -> (no net)
- U27 pad 9: Net-(U27-Pad9) -> (no net)
- U3 pad 1: Net-(U3-Pad1) -> (no net)
- U3 pad 10: /A1 -> /D1
- U3 pad 11: /A0 -> /D0
- U3 pad 12: Net-(U3-Pad12) -> (no net)
- U3 pad 13: Net-(U3-Pad13) -> (no net)
- U3 pad 14: Net-(U3-Pad14) -> (no net)
- U3 pad 15: Net-(U3-Pad15) -> (no net)
- U3 pad 16: Net-(U3-Pad16) -> (no net)
- U3 pad 17: Net-(U3-Pad17) -> (no net)
- U3 pad 18: Net-(U3-Pad18) -> (no net)
- U3 pad 19: Net-(U3-Pad19) -> (no net)
- U3 pad 2: Net-(U3-Pad2) -> (no net)
- U3 pad 20: Net-(U3-Pad20) -> (no net)
- U3 pad 21: Net-(U3-Pad21) -> (no net)
- U3 pad 22: Net-(U3-Pad22) -> (no net)
- U3 pad 23: Net-(U3-Pad23) -> (no net)
- U3 pad 24: Net-(U3-Pad24) -> (no net)
- U3 pad 25: Net-(U3-Pad25) -> (no net)
- U3 pad 26: Net-(U3-Pad26) -> /~INTA
- U3 pad 27: Net-(U3-Pad27) -> (no net)
- U3 pad 28: Net-(U3-Pad28) -> (no net)
- U3 pad 3: Net-(U3-Pad3) -> (no net)
- U3 pad 4: /A7 -> /D7
- U3 pad 5: /A6 -> /D6
- U3 pad 6: /A5 -> /D5
- U3 pad 7: /A4 -> /D4
- U3 pad 8: /A3 -> /D3
- U3 pad 9: /A2 -> /D2
- U4 pad 1: /A19 -> /HDD Controller/A19
- U4 pad 11: /HDD Controller/ADDR_HI -> (no net)
- U4 pad 2: /A18 -> /HDD Controller/A18
- U4 pad 9: /A13 -> /HDD Controller/A13
- U5 pad 1: /A17 -> /HDD Controller/A17
- U5 pad 12: /A7 -> /HDD Controller/A7
- U5 pad 13: /A6 -> /HDD Controller/A6
- U5 pad 2: /A16 -> /HDD Controller/A16
- U5 pad 5: /A15 -> /HDD Controller/A15
- U5 pad 6: /A14 -> /HDD Controller/A14
- U6 pad 1: /A9 -> /HDD Controller/A9
- U6 pad 10: /HDD Controller/ADDR_LO -> (no net)
- U6 pad 2: /A8 -> /HDD Controller/A8
- U6 pad 9: /A5 -> /HDD Controller/A5
- U7 pad 10: /HDD Controller/AEN -> (no net)
- U7 pad 11: /A5 -> (no net)
- U7 pad 12: /A6 -> (no net)
- U7 pad 13: /A7 -> (no net)
- U7 pad 2: /A0 -> (no net)
- U7 pad 23: /HDD Controller/~IOW -> (no net)
- U7 pad 24: /HDD Controller/~IOR -> (no net)
- U7 pad 25: /HDD Controller/ADDR_HI -> (no net)
- U7 pad 26: /HDD Controller/ADDR_LO -> /HDD Controller/ADDR
- U7 pad 27: /A1 -> (no net)
- U7 pad 28: /A0 -> (no net)
- U7 pad 3: /A1 -> (no net)
- U7 pad 4: /A2 -> (no net)
- U7 pad 5: /A3 -> (no net)
- U7 pad 6: /A4 -> (no net)
- U7 pad 9: /HDD Controller/IRQ5 -> (no net)
- U8 pad 1: /Divisible Clock/~AEN1 -> (no net)
- U8 pad 3: /Divisible Clock/~AEN2 -> (no net)
- U8 pad 6: /Divisible Clock/OSC -> (no net)
- U9 pad 14: Net-(U9-Pad14) -> (no net)
- U9 pad 7: Net-(U9-Pad7) -> (no net)
Routing:
- net /HDD Controller/ADDR_LO: track 78.3 -> 0.00 mm, vias 1 -> 0
- net /HDD Controller/ADDR: track 0.00 -> 78.3 mm, vias 0 -> 1
- net /HDD Controller/A8: track 0.00 -> 65.6 mm
- net /A8: track 65.6 -> 0.00 mm
- net /HDD Controller/A9: track 0.00 -> 63.1 mm
- net /A9: track 63.1 -> 0.00 mm
- net /D1: track 0.00 -> 60.3 mm
- net /D0: track 0.00 -> 60.3 mm
- net /A1: track 60.3 -> 0.00 mm
- net /A0: track 60.3 -> 0.00 mm
- net /HDD Controller/A19: track 0.00 -> 56.3 mm
- net /A19: track 56.3 -> 0.00 mm
- net /HDD Controller/A18: track 0.00 -> 54.2 mm, vias 0 -> 1
- net /A18: track 54.2 -> 0.00 mm, vias 1 -> 0
- net /HDD Controller/A13: track 0.00 -> 50.9 mm
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Other:
- board outline added: 244.1 x 244.2 mm

Commit message: Work on motherboard  - Integrating glue logic into CPLD  - Began work on routing
Parts:
- removed REF***: OSHW-Logo_5.7x6mm_SilkScreen, Symbols:OSHW-Logo_5.7x6mm_SilkScreen
- removed U10, U11, U18, U6: 4081, Housings_DIP:DIP-14_W7.62mm_Socket
- removed U12, U17: 74LS32, Housings_DIP:DIP-14_W7.62mm_Socket
- removed U13: 74LS14, Housings_DIP:DIP-14_W7.62mm_Socket
- removed U14: 74LS77, Housings_DIP:DIP-14_W7.62mm_Socket
- removed U16, U8: 4069, Housings_DIP:DIP-14_W7.62mm_Socket
- removed U19: 74HC74, Housings_DIP:DIP-14_W7.62mm_Socket
- removed U20: 7402, Housings_DIP:DIP-14_W7.62mm_Socket
- removed U21: 40106, Housings_DIP:DIP-40_W15.24mm_Socket
- removed U42: 74LS157, Housings_SOIC:SOIC-16_3.9x9.9mm_Pitch1.27mm
- added J5: Bus_ISA_8bit, RetPC:ISA-8-bit, F.Cu at (164.3, 70.7)
- added J6: Bus_ISA_8bit, RetPC:ISA-8-bit, F.Cu at (185.8, 70.7)
- added J7: Bus_ISA_8bit, RetPC:ISA-8-bit, F.Cu at (207.3, 70.7)
- added J8: 3.3V_HEADER, Pin_Headers:Pin_Header_Straight_2x03_Pitch2.54mm, F.Cu at (34.9, 88.5)
- added RN1: 4.7k, Resistors_THT:R_Array_SIP6, F.Cu at (346.8, 127.7)
- added RN2: 4.7k, Resistors_THT:R_Array_SIP5, F.Cu at (346.8, 131.0)
- added U28: 8288, Housings_DIP:DIP-20_W7.62mm_Socket, F.Cu at (68.1, 40.0)
- C2, C4: value 33p -> 30p
- U1: footprint Housings_DIP:DIP-28_W15.24mm_Socket -> Housings_LCC:PLCC-28_THT-Socket
- U2: value 8088_Max_Mode -> 8088
- U4: value 4081 -> CD40147; footprint Housings_DIP:DIP-14_W7.62mm_Socket -> Housings_DIP:DIP-16_W7.62mm_Socket
- U49: footprint Housings_DIP:DIP-12_W7.62mm_Socket -> Housings_DIP:DIP-14_W7.62mm_Socket
- U5: value 4001 -> ATF750LVC; footprint Housings_LCC:PLCC-28_THT-Socket -> Housings_DIP:DIP-24_W7.62mm_Socket
- Y1: value 18.432 MHz -> 14.31818 MHz
- Y2: value 32.768 MHz -> 24.000 MHz
- moved U1 258.3 mm to (25.9, 64.3)
- moved U39 257.1 mm to (104.5, 160.9)
- moved U43 254.6 mm to (50.8, 135.1), turned to 180 degrees
- moved U46 201.7 mm to (66.7, 134.0), turned to 90 degrees
- moved U33 198.3 mm to (56.5, 95.6), turned to 90 degrees
- moved U32 190.8 mm to (56.5, 108.6), turned to 90 degrees
- moved U31 171.4 mm to (92.5, 57.0)
- moved U29 170.1 mm to (100.1, 109.7), turned to 180 degrees
- moved U48 142.2 mm to (294.8, 153.8)
- moved U51 117.0 mm to (325.5, 146.6)
- moved J4 92.1 mm to (24.6, 86.9)
- moved R6 92.1 mm to (38.6, 98.4)
- moved R8 92.1 mm to (30.9, 98.4)
- moved SW3 92.1 mm to (37.3, 104.7)
- moved SW4 92.1 mm to (32.2, 104.7)
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Connections:
- U1 pad 19: (no net) -> Net-(U1-Pad19)
- U1 pad 25: (no net) -> Net-(U1-Pad25)
- U1 pad 26: (no net) -> Net-(U1-Pad26)
- U15 pad 2: Net-(U15-Pad2) -> /Divisible Clock/OSC_INT
- U2 pad 10: (no net) -> /AD6
- U2 pad 11: (no net) -> /AD5
- U2 pad 12: (no net) -> /AD4
- U2 pad 13: (no net) -> /AD3
- U2 pad 14: (no net) -> /AD2
- U2 pad 15: (no net) -> /AD1
- U2 pad 16: (no net) -> /AD0
- U2 pad 2: (no net) -> /AD14
- U2 pad 26: (no net) -> /IO-Decoder/~S0
- U2 pad 27: (no net) -> /IO-Decoder/~S1
- U2 pad 28: (no net) -> /IO-Decoder/~S2
- U2 pad 3: (no net) -> /AD13
- U2 pad 35: (no net) -> /AD19
- U2 pad 36: (no net) -> /AD18
- U2 pad 37: (no net) -> /AD17
- U2 pad 38: (no net) -> /AD16
- U2 pad 39: (no net) -> /AD15
- U2 pad 4: (no net) -> /AD12
- U2 pad 5: (no net) -> /AD11
- U2 pad 6: (no net) -> /AD10
- U2 pad 7: (no net) -> /AD9
- U2 pad 8: (no net) -> /AD8
- U2 pad 9: (no net) -> /AD7
- U29 pad 1: (no net) -> /IO-Decoder/DT_~R
- U29 pad 2: /IO-Decoder/AD7 -> /AD7
- U29 pad 3: /IO-Decoder/AD6 -> /AD6
- U29 pad 4: /IO-Decoder/AD5 -> /AD5
- U29 pad 5: /IO-Decoder/AD4 -> /AD4
- U29 pad 6: /IO-Decoder/AD3 -> /AD3
- U29 pad 7: /IO-Decoder/AD2 -> /AD2
- U29 pad 8: /IO-Decoder/AD1 -> /AD1
- U29 pad 9: /IO-Decoder/AD0 -> /AD0
- U30 pad 1: (no net) -> Net-(U28-Pad16)
- U31 pad 2: (no net) -> /AD19
- U31 pad 3: (no net) -> /AD18
- U31 pad 4: (no net) -> /AD17
- U31 pad 5: (no net) -> /AD16
- U31 pad 6: (no net) -> /AD15
- U31 pad 7: (no net) -> /AD14
- U31 pad 8: (no net) -> /AD13
- U31 pad 9: (no net) -> /AD12
- U32 pad 2: (no net) -> /AD11
- U32 pad 4: (no net) -> /AD10
- U32 pad 6: (no net) -> /AD9
- U32 pad 8: (no net) -> /AD8
- U33 pad 2: /IO-Decoder/AD7 -> /AD7
- U33 pad 3: /IO-Decoder/AD6 -> /AD6
- U33 pad 4: /IO-Decoder/AD5 -> /AD5
- U33 pad 5: /IO-Decoder/AD4 -> /AD4
- U33 pad 6: /IO-Decoder/AD3 -> /AD3
- U33 pad 7: /IO-Decoder/AD2 -> /AD2
- U33 pad 8: /IO-Decoder/AD1 -> /AD1
- U33 pad 9: /IO-Decoder/AD0 -> /AD0
- U39 pad 1: /HDD Controller/A19 -> (no net)
- U39 pad 10: /HDD Controller/A7 -> (no net)
- U39 pad 11: /HDD Controller/A6 -> (no net)
- U39 pad 13: /HDD Controller/A5 -> (no net)
- U39 pad 2: /HDD Controller/A18 -> (no net)
- U39 pad 21: (no net) -> /HDD Controller/~RESET
- U39 pad 3: /HDD Controller/A17 -> (no net)
- U39 pad 4: /HDD Controller/A16 -> (no net)
- U39 pad 5: /HDD Controller/A15 -> (no net)
- U39 pad 6: /HDD Controller/A14 -> (no net)
- U39 pad 7: /HDD Controller/A13 -> (no net)
- U39 pad 8: /HDD Controller/A9 -> (no net)
- U39 pad 9: /HDD Controller/A8 -> (no net)
- U4 pad 1: /HDD Controller/A19 -> (no net)
- U4 pad 10: Net-(U4-Pad10) -> (no net)
- U4 pad 12: Net-(U4-Pad12) -> (no net)
- U4 pad 13: Net-(U4-Pad10) -> (no net)
- U4 pad 14: +5V -> (no net)
- U4 pad 2: /HDD Controller/A18 -> (no net)
- U4 pad 3: Net-(U4-Pad3) -> (no net)
- U4 pad 4: Net-(U4-Pad12) -> (no net)
- U4 pad 5: Net-(U4-Pad3) -> (no net)
- U4 pad 6: Net-(U4-Pad6) -> (no net)
- U4 pad 7: GND -> (no net)
- U4 pad 8: Net-(U4-Pad8) -> (no net)
- U4 pad 9: /HDD Controller/A13 -> (no net)
- U49 pad 1: (no net) -> /IO-Decoder/~DMAAEN
- U49 pad 10: (no net) -> /IO-Decoder/~XIOW
- U49 pad 3: (no net) -> /IO-Decoder/~MRDC
- U49 pad 4: (no net) -> /IO-Decoder/~IOW
- U49 pad 5: (no net) -> /IO-Decoder/~MEMW
- U49 pad 8: (no net) -> /IO-Decoder/~XIOR
- U5 pad 1: /HDD Controller/A17 -> Net-(U15-Pad4)
- U5 pad 10: /HDD Controller/~RESET -> (no net)
- U5 pad 11: Net-(U5-Pad11) -> (no net)
- U5 pad 12: /HDD Controller/A7 -> GND
- U5 pad 13: /HDD Controller/A6 -> (no net)
- U5 pad 14: +5V -> /RESET
- U5 pad 15: (no net) -> /READY
- U5 pad 2: /HDD Controller/A16 -> (no net)
- U5 pad 24: (no net) -> +5V
- U5 pad 3: Net-(U4-Pad6) -> (no net)
- U5 pad 4: Net-(U4-Pad8) -> (no net)
- U5 pad 5: /HDD Controller/A15 -> (no net)
- U5 pad 6: /HDD Controller/A14 -> /Divisible Clock/~RES
- U5 pad 7: GND -> (no net)
- U5 pad 8: /HDD Controller/RESET -> /Divisible Clock/OSC_INT
- U5 pad 9: /HDD Controller/RESET -> /SYS_CLK
- U9 pad 14: (no net) -> +5V
- U9 pad 3: Net-(C2-Pad1) -> Net-(C3-Pad1)
- U9 pad 4: Net-(C4-Pad1) -> /Divisible Clock/OSC_INT
- U9 pad 5: Net-(C3-Pad1) -> Net-(C2-Pad1)
- U9 pad 6: Net-(U15-Pad2) -> Net-(C4-Pad1)
- U9 pad 7: (no net) -> GND
Routing:
- net GND: track 0.00 -> 286.6 mm
- net -5V: track 0.00 -> 263.7 mm, vias 0 -> 3
- net +12V: track 0.00 -> 261.4 mm, vias 0 -> 2
- net -12V: track 0.00 -> 229.7 mm, vias 0 -> 3
- net +5V: track 8.25 -> 217.1 mm
- net /~INTA: track 0.00 -> 101.5 mm, vias 0 -> 2
- net /A5: track 92.8 -> 0.00 mm, vias 1 -> 0
- net /ISA/RESET: track 0.00 -> 89.8 mm
- net /A6: track 89.7 -> 0.00 mm, vias 2 -> 0
- net /HDD Controller/ADDR: track 78.3 -> 0.00 mm, vias 1 -> 0
- net /AD7: track 0.00 -> 66.3 mm
- net /IO-Decoder/A0: track 0.00 -> 66.0 mm, vias 0 -> 1
- net /HDD Controller/A8: track 65.6 -> 0.00 mm
- net +3V3: track 9.70 -> 73.0 mm
- net /HDD Controller/A9: track 63.1 -> 0.00 mm
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- added copper zone on F.Cu, net +5V
- added copper zone on B.Cu, net GND

Commit message: routed two pieces
sync
Parts:
- moved RN1 270.2 mm to (96.0, 27.1), turned to 270 degrees
- moved U48 242.7 mm to (52.1, 155.4), turned to 90 degrees
- moved U49 241.1 mm to (99.8, 24.6)
- moved U40 234.2 mm to (142.7, 142.9)
- moved U45 213.9 mm to (105.2, 56.8)
- moved U44 204.2 mm to (104.6, 86.9)
- moved U47 167.1 mm to (224.7, 155.4)
Routing:
- net /IO-Decoder/A8: track 0.00 -> 45.1 mm, vias 0 -> 2
- net /IO-Decoder/~MRDC: track 0.00 -> 28.1 mm, vias 0 -> 3
- net /IO-Decoder/~MEMW: track 0.00 -> 21.8 mm, vias 0 -> 2
- net /IO-Decoder/~IORC: track 0.00 -> 21.0 mm, vias 0 -> 2
- net /IO-Decoder/A19: track 0.00 -> 19.8 mm, vias 0 -> 2
- net /IO-Decoder/A16: track 0.00 -> 16.8 mm, vias 0 -> 1
- net /IO-Decoder/A18: track 0.00 -> 12.3 mm, vias 0 -> 2
- net /IO-Decoder/~MWTC: track 0.00 -> 12.1 mm, vias 0 -> 1
- net /IO-Decoder/~IOW: track 0.00 -> 8.87 mm
- net /SYS_CLK: track 89.2 -> 97.9 mm
- net /IO-Decoder/A17: track 0.00 -> 5.19 mm
- net GND: track 286.6 -> 291.2 mm
Other:
- board text added: "Are these reversible?"
