File: Motherboard/Motherboard.kicad_pcb (KiCad board)
At the start: 2 copper layers, 244.1 x 244.2 mm, 75 parts, among them J1 SD_Connector, J2 Bus_ISA_8bit, J3 Bus_ISA_8bit, J4 ATX24, J5 Bus_ISA_8bit, J6 Bus_ISA_8bit, J7 Bus_ISA_8bit, J8 3.3V_HEADER, SW1 TURBO, SW2 FREEZE, SW3 SW_SPST_LED, SW4 RESET, SW5 SW_DIP_x01, U1 82C54_PLCC, U15 74LS257, U2 8088, U22 74HC74, U23 8237, U24 74LS04, U25 74LS573, U26 74LS573, U27 74LS670, U28 8288, U29 74LS245, U3 8259, U30 74LS04, U31 74LS573, U32 74LS244, U33 74LS573, U34 74LS04, U35 74LS04, U36 74LS00, U37 74LS00, U38 74LS10, U39 ATF750LVC, U4 CD40147, U40 74LS27, U41 74LS04, U43 74LS244, U44 74LS244, U45 74LS244, U46 74LS245, U47 4077, U48 SST39SF010, U49 74LS243, U5 ATF750LVC, U50 74LS04, U51 ATF750LVC, U52 74LS74, U53 74LS00, U54 74LS08, U55 74LS138, U56 4077, U57 DS1100Z-100+ (TTLDL-20), U7 ATmega328-PU, U9 40106, Y1 14.31818 MHz, Y2 24.000 MHz

Commit message: Large sync
Parts:
- added BT1: Battery_Cell, Connectors:CR2032H, F.Cu at (238.8, 70.9)
- added C10: C_Small, Capacitors_THT:C_Disc_D3.8mm_W2.6mm_P2.50mm, F.Cu at (242.8, 49.8)
- added C11: C_Small, Capacitors_THT:C_Disc_D3.8mm_W2.6mm_P2.50mm, F.Cu at (242.8, 54.6)
- added C12: C_Small, Capacitors_THT:C_Disc_D3.8mm_W2.6mm_P2.50mm, F.Cu at (246.6, 28.7)
- added C13: C_Small, Capacitors_THT:C_Disc_D3.8mm_W2.6mm_P2.50mm, F.Cu at (252.5, 29.0)
- added C5: 1u, Capacitors_THT:CP_Radial_D4.0mm_P2.00mm, F.Cu at (122.4, 113.3)
- added C6: 1u, Capacitors_THT:CP_Radial_D4.0mm_P2.00mm, F.Cu at (144.0, 113.3)
- added C7: 1u, Capacitors_THT:CP_Radial_D4.0mm_P2.00mm, F.Cu at (165.6, 113.3)
- added C8: 1u, Capacitors_THT:CP_Radial_D4.0mm_P2.00mm, F.Cu at (187.2, 113.3)
- added C9: 1u, Capacitors_THT:CP_Radial_D4.0mm_P2.00mm, F.Cu at (208.5, 113.3)
- added J10: Conn_02x17_Odd_Even, IDC:IDC-Header_2x17_P2.54mm_Vertical, F.Cu at (248.4, 38.1)
- added J11: USB_B, Connectors:USB_B, F.Cu at (244.6, 25.1)
- added J12: DB9_Male, Connnectors_DSUB:DSUB-9_Male_Horizontal_Pitch2.77x2.84mm_EdgePinOffset4.94mm_Housed_MountingHolesOffset7.48mm, F.Cu at (227.1, 20.1)
- added J15: DB25_Female, Connnectors_DSUB:DSUB-25_Female_Horizontal_Pitch2.77x2.84mm_EdgePinOffset4.94mm_Housed_MountingHolesOffset7.48mm, F.Cu at (68.1, 19.6)
- added R12: R_Small, Resistors_THT:R_Axial_DIN0411_L9.9mm_D3.6mm_P5.08mm_Vertical, F.Cu at (230.6, 25.9)
- added R13: R_Small, Resistors_THT:R_Axial_DIN0411_L9.9mm_D3.6mm_P5.08mm_Vertical, F.Cu at (226.3, 25.9)
- added U10: GD75232N, Housings_DIP:DIP-20_W7.62mm_Socket, F.Cu at (201.7, 17.0)
- added U6: p.7_pack0, Housings_QFP:LQFP-128_14x20mm_Pitch0.5mm, F.Cu at (222.2, 43.9)
- added U8: FT231XS, RetPC:SSOP-24_3.9x8.7mm_Pitch0.635mm, F.Cu at (238.3, 36.3)
- added Y3: 32.768kHz, Crystals:Crystal_HC49-U_Vertical, F.Cu at (235.7, 49.8)
- moved U55 243.7 mm to (37.6, 134.9), turned to 180 degrees
- moved U40 47.3 mm to (104.9, 114.6)
Connections:
- net /IO-Decoder/~MEMW renamed /~MEMW
- J2 pad 13: (no net) -> /~IOW
- J2 pad 2: /ISA/RESET -> /RESET
- J2 pad 20: (no net) -> /CLK
- J2 pad 27: (no net) -> /DMA/TC
- J2 pad 28: (no net) -> /ALE
- J2 pad 30: (no net) -> /OSC
- J2 pad 33: (no net) -> /D7
- J2 pad 34: (no net) -> /D6
- J2 pad 35: (no net) -> /D5
- J2 pad 36: (no net) -> /D4
- J2 pad 37: (no net) -> /D3
- J2 pad 38: (no net) -> /D2
- J2 pad 39: (no net) -> /D1
- J2 pad 40: (no net) -> /D0
- J2 pad 42: (no net) -> /AEN
- J2 pad 43: (no net) -> /HDD Controller/A19
- J2 pad 44: (no net) -> /HDD Controller/A18
- J2 pad 45: (no net) -> /HDD Controller/A17
- J2 pad 46: (no net) -> /HDD Controller/A16
- J2 pad 47: (no net) -> /FDC-Serial/A15
- J2 pad 48: (no net) -> /FDC-Serial/A14
- J2 pad 49: (no net) -> /FDC-Serial/A13
- J2 pad 50: (no net) -> /FDC-Serial/A12
- J2 pad 51: (no net) -> /FDC-Serial/A11
- J2 pad 52: (no net) -> /FDC-Serial/A10
- J2 pad 53: (no net) -> /FDC-Serial/A9
- J2 pad 54: (no net) -> /FDC-Serial/A8
- J2 pad 55: (no net) -> /FDC-Serial/A7
- J2 pad 56: (no net) -> /FDC-Serial/A6
- J2 pad 57: (no net) -> /FDC-Serial/A5
- J2 pad 58: (no net) -> /FDC-Serial/A4
- J2 pad 59: (no net) -> /FDC-Serial/A3
- J2 pad 60: (no net) -> /FDC-Serial/A2
- J2 pad 61: (no net) -> /FDC-Serial/A1
- J2 pad 62: (no net) -> /FDC-Serial/A0
- J3 pad 13: (no net) -> /~IOW
- J3 pad 2: /ISA/RESET -> /RESET
- J3 pad 20: (no net) -> /CLK
- J3 pad 27: (no net) -> /DMA/TC
- J3 pad 28: (no net) -> /ALE
- J3 pad 30: (no net) -> /OSC
- J3 pad 33: (no net) -> /D7
- J3 pad 34: (no net) -> /D6
- J3 pad 35: (no net) -> /D5
- J3 pad 36: (no net) -> /D4
- J3 pad 37: (no net) -> /D3
- J3 pad 38: (no net) -> /D2
- J3 pad 39: (no net) -> /D1
- J3 pad 40: (no net) -> /D0
- J3 pad 42: (no net) -> /AEN
- J3 pad 43: (no net) -> /HDD Controller/A19
- J3 pad 44: (no net) -> /HDD Controller/A18
- J3 pad 45: (no net) -> /HDD Controller/A17
- J3 pad 46: (no net) -> /HDD Controller/A16
- J3 pad 47: (no net) -> /FDC-Serial/A15
- J3 pad 48: (no net) -> /FDC-Serial/A14
- J3 pad 49: (no net) -> /FDC-Serial/A13
- J3 pad 50: (no net) -> /FDC-Serial/A12
- J3 pad 51: (no net) -> /FDC-Serial/A11
- J3 pad 52: (no net) -> /FDC-Serial/A10
- J3 pad 53: (no net) -> /FDC-Serial/A9
- J3 pad 54: (no net) -> /FDC-Serial/A8
- J3 pad 55: (no net) -> /FDC-Serial/A7
- J3 pad 56: (no net) -> /FDC-Serial/A6
- J3 pad 57: (no net) -> /FDC-Serial/A5
- J3 pad 58: (no net) -> /FDC-Serial/A4
- J3 pad 59: (no net) -> /FDC-Serial/A3
- J3 pad 60: (no net) -> /FDC-Serial/A2
- J3 pad 61: (no net) -> /FDC-Serial/A1
- J3 pad 62: (no net) -> /FDC-Serial/A0
- J4 pad 9: (no net) -> /5V_SB
- J5 pad 13: (no net) -> /~IOW
- J5 pad 2: /ISA/RESET -> /RESET
- J5 pad 20: (no net) -> /CLK
- J5 pad 27: (no net) -> /DMA/TC
- J5 pad 28: (no net) -> /ALE
- J5 pad 30: (no net) -> /OSC
- J5 pad 33: (no net) -> /D7
- J5 pad 34: (no net) -> /D6
- J5 pad 35: (no net) -> /D5
- J5 pad 36: (no net) -> /D4
- J5 pad 37: (no net) -> /D3
- J5 pad 38: (no net) -> /D2
- J5 pad 39: (no net) -> /D1
- J5 pad 40: (no net) -> /D0
- J5 pad 42: (no net) -> /AEN
- J5 pad 43: (no net) -> /HDD Controller/A19
- J5 pad 44: (no net) -> /HDD Controller/A18
- J5 pad 45: (no net) -> /HDD Controller/A17
- J5 pad 46: (no net) -> /HDD Controller/A16
- J5 pad 47: (no net) -> /FDC-Serial/A15
- J5 pad 48: (no net) -> /FDC-Serial/A14
- J5 pad 49: (no net) -> /FDC-Serial/A13
- J5 pad 50: (no net) -> /FDC-Serial/A12
- J5 pad 51: (no net) -> /FDC-Serial/A11
- J5 pad 52: (no net) -> /FDC-Serial/A10
- J5 pad 53: (no net) -> /FDC-Serial/A9
- J5 pad 54: (no net) -> /FDC-Serial/A8
- J5 pad 55: (no net) -> /FDC-Serial/A7
- J5 pad 56: (no net) -> /FDC-Serial/A6
- J5 pad 57: (no net) -> /FDC-Serial/A5
- J5 pad 58: (no net) -> /FDC-Serial/A4
- J5 pad 59: (no net) -> /FDC-Serial/A3
- J5 pad 60: (no net) -> /FDC-Serial/A2
- J5 pad 61: (no net) -> /FDC-Serial/A1
- J5 pad 62: (no net) -> /FDC-Serial/A0
- J6 pad 13: (no net) -> /~IOW
- J6 pad 2: /ISA/RESET -> /RESET
- J6 pad 20: (no net) -> /CLK
- J6 pad 27: (no net) -> /DMA/TC
- J6 pad 28: (no net) -> /ALE
- J6 pad 30: (no net) -> /OSC
- J6 pad 33: (no net) -> /D7
- J6 pad 34: (no net) -> /D6
- J6 pad 35: (no net) -> /D5
- J6 pad 36: (no net) -> /D4
- J6 pad 37: (no net) -> /D3
- J6 pad 38: (no net) -> /D2
- J6 pad 39: (no net) -> /D1
- J6 pad 40: (no net) -> /D0
- J6 pad 42: (no net) -> /AEN
- J6 pad 43: (no net) -> /HDD Controller/A19
- J6 pad 44: (no net) -> /HDD Controller/A18
- J6 pad 45: (no net) -> /HDD Controller/A17
- J6 pad 46: (no net) -> /HDD Controller/A16
- J6 pad 47: (no net) -> /FDC-Serial/A15
- J6 pad 48: (no net) -> /FDC-Serial/A14
- J6 pad 49: (no net) -> /FDC-Serial/A13
- J6 pad 50: (no net) -> /FDC-Serial/A12
- J6 pad 51: (no net) -> /FDC-Serial/A11
- J6 pad 52: (no net) -> /FDC-Serial/A10
- J6 pad 53: (no net) -> /FDC-Serial/A9
- J6 pad 54: (no net) -> /FDC-Serial/A8
- J6 pad 55: (no net) -> /FDC-Serial/A7
- J6 pad 56: (no net) -> /FDC-Serial/A6
- J6 pad 57: (no net) -> /FDC-Serial/A5
- J6 pad 58: (no net) -> /FDC-Serial/A4
- J6 pad 59: (no net) -> /FDC-Serial/A3
- J6 pad 60: (no net) -> /FDC-Serial/A2
- J6 pad 61: (no net) -> /FDC-Serial/A1
- J6 pad 62: (no net) -> /FDC-Serial/A0
- J7 pad 13: (no net) -> /~IOW
- J7 pad 2: /ISA/RESET -> /RESET
- J7 pad 20: (no net) -> /CLK
- J7 pad 27: (no net) -> /DMA/TC
- J7 pad 28: (no net) -> /ALE
- J7 pad 30: (no net) -> /OSC
- J7 pad 33: (no net) -> /D7
- J7 pad 34: (no net) -> /D6
- J7 pad 35: (no net) -> /D5
- J7 pad 36: (no net) -> /D4
- J7 pad 37: (no net) -> /D3
- J7 pad 38: (no net) -> /D2
- J7 pad 39: (no net) -> /D1
- J7 pad 40: (no net) -> /D0
- J7 pad 42: (no net) -> /AEN
- J7 pad 43: (no net) -> /HDD Controller/A19
- J7 pad 44: (no net) -> /HDD Controller/A18
- J7 pad 45: (no net) -> /HDD Controller/A17
- J7 pad 46: (no net) -> /HDD Controller/A16
- J7 pad 47: (no net) -> /FDC-Serial/A15
- J7 pad 48: (no net) -> /FDC-Serial/A14
- J7 pad 49: (no net) -> /FDC-Serial/A13
- J7 pad 50: (no net) -> /FDC-Serial/A12
- J7 pad 51: (no net) -> /FDC-Serial/A11
- J7 pad 52: (no net) -> /FDC-Serial/A10
- J7 pad 53: (no net) -> /FDC-Serial/A9
- J7 pad 54: (no net) -> /FDC-Serial/A8
- J7 pad 55: (no net) -> /FDC-Serial/A7
- J7 pad 56: (no net) -> /FDC-Serial/A6
- J7 pad 57: (no net) -> /FDC-Serial/A5
- J7 pad 58: (no net) -> /FDC-Serial/A4
- J7 pad 59: (no net) -> /FDC-Serial/A3
- J7 pad 60: (no net) -> /FDC-Serial/A2
- J7 pad 61: (no net) -> /FDC-Serial/A1
- J7 pad 62: (no net) -> /FDC-Serial/A0
- RN1 pad 2: /IO-Decoder/~IOW -> /~IOW
- U23 pad 1: (no net) -> /~IOR
- U23 pad 2: (no net) -> /~IOW
- U24 pad 4: (no net) -> /DMA/TC
- U28 pad 12: /IO-Decoder/~IOW -> /~IOW
- U28 pad 15: (no net) -> /~AEN
- U28 pad 5: /IO-Decoder/ALE -> /ALE
- U31 pad 11: /IO-Decoder/ALE -> /ALE
- U31 pad 12: /IO-Decoder/A12 -> /FDC-Serial/A12
- U31 pad 13: /IO-Decoder/A13 -> /FDC-Serial/A13
- U31 pad 14: /IO-Decoder/A14 -> /FDC-Serial/A14
- U31 pad 15: /IO-Decoder/A15 -> /FDC-Serial/A15
- U31 pad 16: /IO-Decoder/A16 -> /HDD Controller/A16
- U31 pad 17: /IO-Decoder/A17 -> /HDD Controller/A17
- U31 pad 18: /IO-Decoder/A18 -> /HDD Controller/A18
- U31 pad 19: /IO-Decoder/A19 -> /HDD Controller/A19
- U32 pad 12: /IO-Decoder/A8 -> /FDC-Serial/A8
- U32 pad 14: /IO-Decoder/A9 -> /FDC-Serial/A9
- U32 pad 16: /IO-Decoder/A10 -> /FDC-Serial/A10
- U32 pad 18: /IO-Decoder/A11 -> /FDC-Serial/A11
- U33 pad 11: /IO-Decoder/ALE -> /ALE
- U33 pad 12: /IO-Decoder/A0 -> /FDC-Serial/A0
- U33 pad 13: /IO-Decoder/A1 -> /FDC-Serial/A1
- U33 pad 14: /IO-Decoder/A2 -> /FDC-Serial/A2
- U33 pad 15: /IO-Decoder/A3 -> /FDC-Serial/A3
- U33 pad 16: /IO-Decoder/A4 -> /FDC-Serial/A4
- U33 pad 17: /IO-Decoder/A5 -> /FDC-Serial/A5
- U33 pad 18: /IO-Decoder/A6 -> /FDC-Serial/A6
- U33 pad 19: /IO-Decoder/A7 -> /FDC-Serial/A7
- U39 pad 1: (no net) -> /HDD Controller/A19
- U39 pad 10: (no net) -> /FDC-Serial/A7
- U39 pad 11: (no net) -> /FDC-Serial/A6
- U39 pad 13: (no net) -> /FDC-Serial/A5
- U39 pad 2: (no net) -> /HDD Controller/A18
- U39 pad 22: (no net) -> /RESET
- U39 pad 3: (no net) -> /HDD Controller/A17
- U39 pad 4: (no net) -> /HDD Controller/A16
- U39 pad 5: (no net) -> /FDC-Serial/A15
- U39 pad 6: (no net) -> /FDC-Serial/A14
- U39 pad 7: (no net) -> /FDC-Serial/A13
- U39 pad 8: (no net) -> /FDC-Serial/A9
- U39 pad 9: (no net) -> /FDC-Serial/A8
- U43 pad 11: /IO-Decoder/A4 -> /FDC-Serial/A4
- U43 pad 13: /IO-Decoder/A5 -> /FDC-Serial/A5
- U43 pad 15: /IO-Decoder/A6 -> /FDC-Serial/A6
- U43 pad 17: /IO-Decoder/A7 -> /FDC-Serial/A7
- U43 pad 2: /IO-Decoder/A0 -> /FDC-Serial/A0
- U43 pad 4: /IO-Decoder/A1 -> /FDC-Serial/A1
- U43 pad 6: /IO-Decoder/A2 -> /FDC-Serial/A2
- U43 pad 8: /IO-Decoder/A3 -> /FDC-Serial/A3
- U44 pad 11: /IO-Decoder/A12 -> /FDC-Serial/A12
- U44 pad 13: /IO-Decoder/A13 -> /FDC-Serial/A13
- U44 pad 15: /IO-Decoder/A14 -> /FDC-Serial/A14
- U44 pad 17: /IO-Decoder/A15 -> /FDC-Serial/A15
- U44 pad 2: /IO-Decoder/A8 -> /FDC-Serial/A8
- U44 pad 4: /IO-Decoder/A9 -> /FDC-Serial/A9
- U44 pad 6: /IO-Decoder/A10 -> /FDC-Serial/A10
- U44 pad 8: /IO-Decoder/A11 -> /FDC-Serial/A11
- U45 pad 2: /IO-Decoder/A16 -> /HDD Controller/A16
- U45 pad 4: /IO-Decoder/A17 -> /HDD Controller/A17
- U45 pad 6: /IO-Decoder/A18 -> /HDD Controller/A18
- U45 pad 8: /IO-Decoder/A19 -> /HDD Controller/A19
- U49 pad 4: /IO-Decoder/~IOW -> /~IOW
- U5 pad 16: (no net) -> /OSC
- U7 pad 10: (no net) -> /~AEN
- U7 pad 11: (no net) -> /D5
- U7 pad 12: (no net) -> /D6
- U7 pad 13: (no net) -> /D7
- U7 pad 2: (no net) -> /D0
- U7 pad 23: (no net) -> /~IOW
- U7 pad 24: (no net) -> /~IOR
- U7 pad 27: (no net) -> /FDC-Serial/A1
- U7 pad 28: (no net) -> /FDC-Serial/A0
- U7 pad 3: (no net) -> /D1
- U7 pad 4: (no net) -> /D2
- U7 pad 5: (no net) -> /D3
- U7 pad 6: (no net) -> /D4
Routing:
- net /RESET: track 65.6 -> 155.4 mm
- net /ISA/RESET: track 89.8 -> 0.00 mm
- net /D7: track 31.6 -> 121.2 mm
- net /D6: track 35.2 -> 124.7 mm
- net /IO-Decoder/A0: track 66.0 -> 0.00 mm, vias 1 -> 0
- net /FDC-Serial/A0: track 0.00 -> 66.0 mm, vias 0 -> 1
- net /IO-Decoder/A1: track 60.3 -> 0.00 mm, vias 1 -> 0
- net /FDC-Serial/A1: track 0.00 -> 60.3 mm, vias 0 -> 1
- net /IO-Decoder/A7: track 58.0 -> 0.00 mm, vias 1 -> 0
- net /FDC-Serial/A7: track 0.00 -> 58.0 mm, vias 0 -> 1
- net /IO-Decoder/A6: track 54.5 -> 0.00 mm, vias 1 -> 0
- net /FDC-Serial/A6: track 0.00 -> 54.5 mm, vias 0 -> 1
- net /IO-Decoder/A2: track 54.0 -> 0.00 mm, vias 1 -> 0
- net /FDC-Serial/A2: track 0.00 -> 54.0 mm, vias 0 -> 1
- net /IO-Decoder/A5: track 51.0 -> 0.00 mm, vias 1 -> 0
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Other:
- board text removed: "Are these reversible?"
