File: Motherboard/Motherboard.kicad_pcb (KiCad board)
At the start: 2 copper layers, 244.1 x 244.2 mm, 75 parts, among them J1 SD_Connector, J2 Bus_ISA_8bit, J3 Bus_ISA_8bit, J4 ATX24, J5 Bus_ISA_8bit, J6 Bus_ISA_8bit, J7 Bus_ISA_8bit, J8 3.3V_HEADER, SW1 TURBO, SW2 FREEZE, SW3 SW_SPST_LED, SW4 RESET, SW5 SW_DIP_x01, U1 82C54_PLCC, U15 74LS257, U2 8088, U22 74HC74, U23 8237, U24 74LS04, U25 74LS573, U26 74LS573, U27 74LS670, U28 8288, U29 74LS245, U3 8259, U30 74LS04, U31 74LS573, U32 74LS244, U33 74LS573, U34 74LS04, U35 74LS04, U36 74LS00, U37 74LS00, U38 74LS10, U39 ATF750LVC, U4 CD40147, U40 74LS27, U41 74LS04, U43 74LS244, U44 74LS244, U45 74LS244, U46 74LS245, U47 4077, U48 SST39SF010, U49 74LS243, U5 ATF750LVC, U50 74LS04, U51 ATF750LVC, U52 74LS74, U53 74LS00, U54 74LS08, U55 74LS138, U56 4077, U57 DS1100Z-100+ (TTLDL-20), U7 ATmega328-PU, U9 40106, Y1 14.31818 MHz, Y2 24.000 MHz

Commit message: LARGE sync
Parts:
- removed U22: 74HC74, Housings_DIP:DIP-14_W7.62mm_Socket
- removed U4: CD40147, Housings_DIP:DIP-16_W7.62mm_Socket
- removed U53: 74LS00, Housings_DIP:DIP-14_W7.62mm_Socket
- removed U54: 74LS08, Housings_DIP:DIP-14_W7.62mm_Socket
- removed U55: 74LS138, Housings_DIP:DIP-16_W7.62mm_Socket
- removed U56: 4077, Housings_DIP:DIP-14_W7.62mm_Socket
- removed U57: DS1100Z-100+ (TTLDL-20), Housings_SOIC:SOIC-8_3.9x4.9mm_Pitch1.27mm
- added BT1: Battery_Cell, Connectors:CR2032H, F.Cu at (54.6, 61.0)
- added C10: C_Small, Capacitors_THT:C_Disc_D3.8mm_W2.6mm_P2.50mm, F.Cu at (59.7, 35.5)
- added C11: C_Small, Capacitors_THT:C_Disc_D3.8mm_W2.6mm_P2.50mm, F.Cu at (66.0, 35.5)
- added C12: C_Small, Capacitors_THT:C_Disc_D3.8mm_W2.6mm_P2.50mm, F.Cu at (200.7, 24.1)
- added C13: C_Small, Capacitors_THT:C_Disc_D3.8mm_W2.6mm_P2.50mm, F.Cu at (195.6, 24.1)
- added C14: 50n, Capacitors_THT:C_Disc_D5.0mm_W2.5mm_P2.50mm, F.Cu at (245.1, 71.7)
- added C15: 270u, Capacitors_THT:CP_Radial_D12.5mm_P5.00mm, F.Cu at (235.6, 81.3)
- added C16: 100n, Capacitors_THT:C_Disc_D5.0mm_W2.5mm_P2.50mm, F.Cu at (248.9, 14.0)
- added C17: 50n, Capacitors_THT:C_Disc_D5.0mm_W2.5mm_P2.50mm, F.Cu at (254.0, 88.9)
- added C18: 270u, Capacitors_THT:CP_Radial_D12.5mm_P5.00mm, F.Cu at (235.6, 94.6)
- added C19: 50n, Capacitors_THT:C_Disc_D5.0mm_W2.5mm_P2.50mm, F.Cu at (254.6, 14.0)
- added C20: 270u, Capacitors_THT:CP_Radial_D12.5mm_P5.00mm, F.Cu at (249.6, 37.5)
- added C21: 22u, Capacitor_THT:CP_Radial_D5.0mm_P2.50mm, F.Cu at (29.2, 73.7)
- added C22: 10u, Capacitor_THT:CP_Radial_D5.0mm_P2.50mm, F.Cu at (50.8, 73.7)
- added C5: 1u, Capacitors_THT:CP_Radial_D4.0mm_P2.00mm, F.Cu at (122.0, 113.0)
- added C6: 1u, Capacitors_THT:CP_Radial_D4.0mm_P2.00mm, F.Cu at (143.6, 113.0)
- added C7: 1u, Capacitors_THT:CP_Radial_D4.0mm_P2.00mm, F.Cu at (165.2, 113.0)
- added C8: 1u, Capacitors_THT:CP_Radial_D4.0mm_P2.00mm, F.Cu at (186.7, 113.0)
- added C9: 1u, Capacitors_THT:CP_Radial_D4.0mm_P2.00mm, F.Cu at (207.7, 113.0)
- added D1: 1N4001, Diode_THT:D_DO-41_SOD81_P10.16mm_Horizontal, F.Cu at (35.6, 76.2)
- added J10: Conn_02x17_Odd_Even, IDC:IDC-Header_2x17_P2.54mm_Vertical, F.Cu at (18.4, 31.8)
- added J11: USB_B, Connectors:USB_B, F.Cu at (222.2, 20.3)
- added J12: DB9_Male, Connnectors_DSUB:DSUB-9_Male_Horizontal_Pitch2.77x2.84mm_EdgePinOffset4.94mm_Housed_MountingHolesOffset7.48mm, F.Cu at (88.9, 20.3)
- added J15: DB25_Female, Connnectors_DSUB:DSUB-25_Female_Horizontal_Pitch2.77x2.84mm_EdgePinOffset4.94mm_Housed_MountingHolesOffset7.48mm, F.Cu at (23.3, 20.6)
- added J9: AudioJack3_SwitchTR, Pin_Headers:Pin_Header_Straight_1x05_Pitch2.54mm, F.Cu at (250.2, 49.5)
- added LS1: Speaker, Pin_Headers:Pin_Header_Straight_1x02_Pitch2.54mm, F.Cu at (254.0, 49.5)
- added R12: R_Small, Resistors_THT:R_Axial_DIN0411_L9.9mm_D3.6mm_P5.08mm_Vertical, F.Cu at (214.0, 29.2)
- added R13: R_Small, Resistors_THT:R_Axial_DIN0411_L9.9mm_D3.6mm_P5.08mm_Vertical, F.Cu at (219.7, 29.2)
- added R14: 10, Resistors_THT:R_Axial_DIN0204_L3.6mm_D1.6mm_P7.62mm_Horizontal, F.Cu at (245.1, 66.0)
- added R15: 10, Resistors_THT:R_Axial_DIN0204_L3.6mm_D1.6mm_P7.62mm_Horizontal, F.Cu at (254.0, 83.8)
- added R16: 10, Resistors_THT:R_Axial_DIN0204_L3.6mm_D1.6mm_P7.62mm_Horizontal, F.Cu at (230.5, 24.1)
- added R17: 4k7, Resistor_THT:R_Axial_DIN0204_L3.6mm_D1.6mm_P5.08mm_Vertical, F.Cu at (61.0, 79.4)
- added R18: 4k7, Resistor_THT:R_Axial_DIN0204_L3.6mm_D1.6mm_P5.08mm_Vertical, F.Cu at (81.3, 79.4)
- added R19: 4k7, Resistor_THT:R_Axial_DIN0204_L3.6mm_D1.6mm_P5.08mm_Vertical, F.Cu at (73.7, 79.4)
- added R20: R_Small, Resistor_THT:R_Axial_DIN0204_L3.6mm_D1.6mm_P5.08mm_Vertical, F.Cu at (230.5, 78.7)
- added RN3: 470R, Resistors_THT:R_Array_SIP4, F.Cu at (246.4, 57.1)
- added RV1: 10k, Pin_Headers:Pin_Header_Straight_1x03_Pitch2.54mm, F.Cu at (230.5, 64.8)
- added RV2: 10k, Pin_Headers:Pin_Header_Straight_1x03_Pitch2.54mm, F.Cu at (247.7, 103.5)
- added RV3: 10k, Pin_Headers:Pin_Header_Straight_1x03_Pitch2.54mm, F.Cu at (247.7, 19.1)
- added U10: GD75232N, Housings_DIP:DIP-20_W7.62mm_Socket, F.Cu at (94.0, 26.7)
- added U11: 8087, Housings_DIP:DIP-40_W15.24mm_Socket, F.Cu at (43.2, 118.1)
- added U12: ATF750LVC-fdc, Package_DIP:DIP-24_W7.62mm_Socket, F.Cu at (227.3, 113.0)
- added U13: ATmega328-PU, Housings_DIP:DIP-28_W7.62mm_Socket, F.Cu at (241.3, 58.4)
- added U14: SN76489A-ALT, Housings_DIP:DIP-16_W7.62mm_Socket, F.Cu at (227.3, 80.0)
- added U16: LM386, Housings_DIP:DIP-8_W7.62mm_Socket, F.Cu at (234.3, 64.1)
- added U17: MAX538BEPA+, Housings_DIP:DIP-8_W7.62mm_Socket, F.Cu at (234.9, 21.6)
- added U18: ATF750LVC-fdc, Housings_DIP:DIP-24_W7.62mm_Socket, F.Cu at (280.0, 148.0)
- added U20: LM386, Housings_DIP:DIP-8_W7.62mm_Socket, F.Cu at (246.4, 92.1)
- added U21: LM386, Housings_DIP:DIP-8_W7.62mm_Socket, F.Cu at (254.0, 30.5)
- added U42: AS6C8008, Package_SO:TSSOP-44_4.4x11.2mm_P0.5mm, F.Cu at (172.1, 139.7)
- added U6: FDC37B787-NS, Housings_QFP:LQFP-128_14x20mm_Pitch0.5mm, F.Cu at (43.2, 36.8)
- added U8: FT231XS, RetPC:SSOP-24_3.9x8.7mm_Pitch0.635mm, F.Cu at (209.6, 17.8)
- added Y3: 32.768kHz, Crystals:Crystal_HC49-U_Vertical, F.Cu at (59.7, 29.2)
- R5: value R -> 1k
- R9: value R -> 1k; footprint Resistors_THT:R_Axial_DIN0204_L3.6mm_D1.6mm_P7.62mm_Horizontal -> Resistors_THT:R_Axial_DIN0204_L3.6mm_D1.6mm_P2.54mm_Vertical
- U24: footprint Housings_DIP:DIP-20_W7.62mm_Socket -> Package_DIP:DIP-14_W7.62mm_Socket
- U25: value 74LS573 -> 74LS244
- U26: value 74LS573 -> 74LS373
- U35: value 74LS04 -> 74LS245; footprint Housings_DIP:DIP-14_W7.62mm_Socket -> Housings_DIP:DIP-20_W7.62mm_Socket
- U37: value 74LS00 -> 74LS74; footprint Housings_DIP:DIP-14_W7.62mm_Socket -> Package_DIP:DIP-14_W7.62mm_Socket
- U38: value 74LS10 -> L79L05_TO92; footprint Housings_DIP:DIP-14_W7.62mm_Socket -> Package_TO_SOT_THT:TO-92_Inline
- U47: value 4077 -> 74LS245; footprint Housings_DIP:DIP-14_W7.62mm_Socket -> Package_DIP:DIP-20_W7.62mm_Socket
- U50: value 74LS04 -> 7400; footprint Housings_DIP:DIP-14_W7.62mm_Socket -> Package_DIP:DIP-14_W7.62mm_Socket
- U52: value 74LS74 -> 74LS32; footprint Housings_DIP:DIP-14_W7.62mm_Socket -> Package_DIP:DIP-14_W7.62mm_Socket
- U7: footprint Housings_DIP:DIP-28_W15.24mm_Socket -> Housings_DIP:DIP-28_W7.62mm_Socket
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Connections:
- net /DREQ3 renamed /DRQ3
- net /IO-Decoder/~DMAAEN renamed /~DMAEN
- net /IO-Decoder/~S0 renamed /~S0
- net /IO-Decoder/~S1 renamed /~S1
- net /IO-Decoder/~S2 renamed /~S2
- net /~MEMW renamed /IO-Decoder/~MEMW
- J2 pad 11: (no net) -> /ISA/~MEMW
- J2 pad 12: (no net) -> /ISA/~MEMR
- J2 pad 14: (no net) -> /ISA/~IOR
- J2 pad 15: (no net) -> /ISA/~DACK3
- J2 pad 16: (no net) -> /ISA/DRQ3
- J2 pad 17: (no net) -> /ISA/~DACK1
- J2 pad 18: (no net) -> /ISA/DRQ1
- J2 pad 19: (no net) -> /ISA/~DACK0
- J2 pad 20: /CLK -> /SYS_CLK
- J2 pad 21: (no net) -> /ISA/IRQ7
- J2 pad 22: (no net) -> /ISA/IRQ6
- J2 pad 23: (no net) -> /ISA/IRQ5
- J2 pad 24: (no net) -> /ISA/IRQ4
- J2 pad 25: (no net) -> /ISA/IRQ3
- J2 pad 26: (no net) -> /ISA/~DACK2
- J2 pad 27: /DMA/TC -> /TC
- J2 pad 32: (no net) -> /ISA/IOCHCK
- J2 pad 33: /D7 -> /HDD Controller/D7
- J2 pad 34: /D6 -> /HDD Controller/D6
- J2 pad 35: /D5 -> /HDD Controller/D5
- J2 pad 36: /D4 -> /HDD Controller/D4
- J2 pad 37: /D3 -> /HDD Controller/D3
- J2 pad 38: /D2 -> /HDD Controller/D2
- J2 pad 39: /D1 -> /HDD Controller/D1
- J2 pad 4: (no net) -> /ISA/IRQ2
- J2 pad 40: /D0 -> /HDD Controller/D0
- J2 pad 41: (no net) -> /IO_READY
- J2 pad 6: (no net) -> /ISA/DRQ2
- J2 pad 8: (no net) -> Net-(J2-Pad8)
- J3 pad 11: (no net) -> /ISA/~MEMW
- J3 pad 12: (no net) -> /ISA/~MEMR
- J3 pad 14: (no net) -> /ISA/~IOR
- J3 pad 15: (no net) -> /ISA/~DACK3
- J3 pad 16: (no net) -> /ISA/DRQ3
- J3 pad 17: (no net) -> /ISA/~DACK1
- J3 pad 18: (no net) -> /ISA/DRQ1
- J3 pad 19: (no net) -> /ISA/~DACK0
- J3 pad 20: /CLK -> /SYS_CLK
- J3 pad 21: (no net) -> /ISA/IRQ7
- J3 pad 22: (no net) -> /ISA/IRQ6
- J3 pad 23: (no net) -> /ISA/IRQ5
- J3 pad 24: (no net) -> /ISA/IRQ4
- J3 pad 25: (no net) -> /ISA/IRQ3
- J3 pad 26: (no net) -> /ISA/~DACK2
- J3 pad 27: /DMA/TC -> /TC
- J3 pad 32: (no net) -> Net-(J3-Pad32)
- J3 pad 33: /D7 -> /HDD Controller/D7
- J3 pad 34: /D6 -> /HDD Controller/D6
- J3 pad 35: /D5 -> /HDD Controller/D5
- J3 pad 36: /D4 -> /HDD Controller/D4
- J3 pad 37: /D3 -> /HDD Controller/D3
- J3 pad 38: /D2 -> /HDD Controller/D2
- J3 pad 39: /D1 -> /HDD Controller/D1
- J3 pad 4: (no net) -> /ISA/IRQ2
- J3 pad 40: /D0 -> /HDD Controller/D0
- J3 pad 41: (no net) -> /IO_READY
- J3 pad 6: (no net) -> /ISA/DRQ2
- J3 pad 8: (no net) -> Net-(J3-Pad8)
- J5 pad 11: (no net) -> /ISA/~MEMW
- J5 pad 12: (no net) -> /ISA/~MEMR
- J5 pad 14: (no net) -> /ISA/~IOR
- J5 pad 15: (no net) -> /ISA/~DACK3
- J5 pad 16: (no net) -> /ISA/DRQ3
- J5 pad 17: (no net) -> /ISA/~DACK1
- J5 pad 18: (no net) -> /ISA/DRQ1
- J5 pad 19: (no net) -> /ISA/~DACK0
- J5 pad 20: /CLK -> /SYS_CLK
- J5 pad 21: (no net) -> /ISA/IRQ7
- J5 pad 22: (no net) -> /ISA/IRQ6
- J5 pad 23: (no net) -> /ISA/IRQ5
- J5 pad 24: (no net) -> /ISA/IRQ4
- J5 pad 25: (no net) -> /ISA/IRQ3
- J5 pad 26: (no net) -> /ISA/~DACK2
- J5 pad 27: /DMA/TC -> /TC
- J5 pad 32: (no net) -> Net-(J5-Pad32)
- J5 pad 33: /D7 -> /HDD Controller/D7
- J5 pad 34: /D6 -> /HDD Controller/D6
- J5 pad 35: /D5 -> /HDD Controller/D5
- J5 pad 36: /D4 -> /HDD Controller/D4
- J5 pad 37: /D3 -> /HDD Controller/D3
- J5 pad 38: /D2 -> /HDD Controller/D2
- J5 pad 39: /D1 -> /HDD Controller/D1
- J5 pad 4: (no net) -> Net-(J5-Pad4)
- J5 pad 40: /D0 -> /HDD Controller/D0
- J5 pad 41: (no net) -> /IO_READY
- J5 pad 6: (no net) -> Net-(J5-Pad6)
- J5 pad 8: (no net) -> Net-(J5-Pad8)
- J6 pad 11: (no net) -> /ISA/~MEMW
- J6 pad 12: (no net) -> /ISA/~MEMR
- J6 pad 14: (no net) -> /ISA/~IOR
- J6 pad 15: (no net) -> /ISA/~DACK3
- J6 pad 16: (no net) -> /ISA/DRQ3
- J6 pad 17: (no net) -> /ISA/~DACK1
- J6 pad 18: (no net) -> /ISA/DRQ1
- J6 pad 19: (no net) -> /ISA/~DACK0
- J6 pad 20: /CLK -> /SYS_CLK
- J6 pad 21: (no net) -> /ISA/IRQ7
- J6 pad 22: (no net) -> /ISA/IRQ6
- J6 pad 23: (no net) -> /ISA/IRQ5
- J6 pad 24: (no net) -> /ISA/IRQ4
- J6 pad 25: (no net) -> /ISA/IRQ3
- J6 pad 26: (no net) -> /ISA/~DACK2
- J6 pad 27: /DMA/TC -> /TC
- J6 pad 32: (no net) -> Net-(J6-Pad32)
- J6 pad 33: /D7 -> /HDD Controller/D7
- J6 pad 34: /D6 -> /HDD Controller/D6
- J6 pad 35: /D5 -> /HDD Controller/D5
- J6 pad 36: /D4 -> /HDD Controller/D4
- J6 pad 37: /D3 -> /HDD Controller/D3
- J6 pad 38: /D2 -> /HDD Controller/D2
- J6 pad 39: /D1 -> /HDD Controller/D1
- J6 pad 4: (no net) -> Net-(J6-Pad4)
- J6 pad 40: /D0 -> /HDD Controller/D0
- J6 pad 41: (no net) -> /IO_READY
- J6 pad 6: (no net) -> Net-(J6-Pad6)
- J6 pad 8: (no net) -> Net-(J6-Pad8)
- J7 pad 11: (no net) -> /ISA/~MEMW
- J7 pad 12: (no net) -> /ISA/~MEMR
- J7 pad 14: (no net) -> /ISA/~IOR
- J7 pad 15: (no net) -> /ISA/~DACK3
- J7 pad 16: (no net) -> /ISA/DRQ3
- J7 pad 17: (no net) -> /ISA/~DACK1
- J7 pad 18: (no net) -> /ISA/DRQ1
- J7 pad 19: (no net) -> /ISA/~DACK0
- J7 pad 20: /CLK -> /SYS_CLK
- J7 pad 21: (no net) -> /ISA/IRQ7
- J7 pad 22: (no net) -> /ISA/IRQ6
- J7 pad 23: (no net) -> /ISA/IRQ5
- J7 pad 24: (no net) -> /ISA/IRQ4
- J7 pad 25: (no net) -> /ISA/IRQ3
- J7 pad 26: (no net) -> /ISA/~DACK2
- J7 pad 27: /DMA/TC -> /TC
- J7 pad 32: (no net) -> Net-(J7-Pad32)
- J7 pad 33: /D7 -> /HDD Controller/D7
- J7 pad 34: /D6 -> /HDD Controller/D6
- J7 pad 35: /D5 -> /HDD Controller/D5
- J7 pad 36: /D4 -> /HDD Controller/D4
- J7 pad 37: /D3 -> /HDD Controller/D3
- J7 pad 38: /D2 -> /HDD Controller/D2
- J7 pad 39: /D1 -> /HDD Controller/D1
- J7 pad 4: (no net) -> Net-(J7-Pad4)
- J7 pad 40: /D0 -> /HDD Controller/D0
- J7 pad 41: (no net) -> /IO_READY
- J7 pad 6: (no net) -> Net-(J7-Pad6)
- J7 pad 8: (no net) -> Net-(J7-Pad8)
- R9 pad 1: +5V -> /IO-Decoder/IO_SigDecoder/IOCHCK
- R9 pad 2: /IO-Decoder/IO_SigDecoder/IOCHCK -> +5V
- RN1 pad 6: /IO-Decoder/~IORC -> /~IOR
- RN2 pad 3: /IO-Decoder/~XIOW -> /~XIOW
- RN2 pad 5: /IO-Decoder/~XIOR -> /~XIOR
- U1 pad 1: (no net) -> Net-(U1-Pad1)
- U1 pad 10: (no net) -> Net-(U1-Pad10)
- U1 pad 11: (no net) -> Net-(U1-Pad11)
- U1 pad 12: (no net) -> /IRQ0
- U1 pad 13: (no net) -> +5V
- U1 pad 14: (no net) -> GND
- U1 pad 15: (no net) -> Net-(U1-Pad15)
- U1 pad 16: (no net) -> Net-(U1-Pad16)
- U1 pad 17: (no net) -> +5V
- U1 pad 18: (no net) -> Net-(U1-Pad10)
- U1 pad 2: (no net) -> /XD7
- U1 pad 20: (no net) -> /SPEAKER
- U1 pad 21: (no net) -> Net-(U1-Pad10)
- U1 pad 22: (no net) -> /XA0
- U1 pad 23: (no net) -> /XA1
- U1 pad 24: (no net) -> Net-(U1-Pad24)
- U1 pad 26: Net-(U1-Pad26) -> /~XIOR
- U1 pad 27: (no net) -> /~XIOW
- U1 pad 28: (no net) -> +5V
- U1 pad 3: (no net) -> /XD6
- U1 pad 4: (no net) -> /XD5
- U1 pad 5: (no net) -> /XD4
- U1 pad 6: (no net) -> /XD3
- U1 pad 7: (no net) -> /XD2
- U1 pad 8: (no net) -> /XD1
- U1 pad 9: (no net) -> /XD0
- U15 pad 10: (no net) -> Net-(U15-Pad10)
- U15 pad 11: (no net) -> Net-(U15-Pad11)
- U15 pad 12: (no net) -> Net-(U15-Pad12)
- U15 pad 13: (no net) -> Net-(U15-Pad13)
- U15 pad 14: (no net) -> Net-(U15-Pad14)
- U15 pad 5: (no net) -> Net-(U15-Pad5)
- U15 pad 6: (no net) -> Net-(U15-Pad6)
- U15 pad 7: (no net) -> Net-(U15-Pad7)
- U15 pad 9: (no net) -> Net-(U15-Pad9)
- U2 pad 17: (no net) -> /NMI
- U2 pad 18: (no net) -> /INTR
- U2 pad 23: (no net) -> /BSY
- U2 pad 24: (no net) -> /QS1
- U2 pad 25: (no net) -> /QS0
- U2 pad 29: (no net) -> /~LOCK
- U2 pad 30: (no net) -> /HLDA
- U2 pad 31: (no net) -> /PU
- U2 pad 32: (no net) -> Net-(U2-Pad32)
- U2 pad 34: (no net) -> Net-(U2-Pad34)
- U23 pad 1: /~IOR -> /DMA/~XIOR
- U23 pad 10: (no net) -> /DMA/HRQ
- U23 pad 11: (no net) -> Net-(U23-Pad11)
- U23 pad 12: Net-(U22-Pad5) -> /DCLK
- U23 pad 17: (no net) -> /DRQ2
- U23 pad 18: (no net) -> /DRQ1
- U23 pad 19: (no net) -> /DRQ0
- U23 pad 2: /~IOW -> /DMA/~XIOW
- U23 pad 21: (no net) -> /DMA/XD7
- U23 pad 22: (no net) -> /DMA/XD6
- U23 pad 23: (no net) -> /DMA/XD5
- U23 pad 24: (no net) -> /DMA/DACK1
- U23 pad 25: (no net) -> /~DACK0BRD
- U23 pad 26: (no net) -> /DMA/XD4
- U23 pad 27: (no net) -> /DMA/XD3
- U23 pad 28: (no net) -> /DMA/XD2
- U23 pad 29: (no net) -> /DMA/XD1
- U23 pad 3: (no net) -> /DMA/~XMEMR
- U23 pad 30: (no net) -> /DMA/XD0
- U23 pad 32: (no net) -> /DMA/XA0
- U23 pad 33: (no net) -> /DMA/XA1
- U23 pad 34: (no net) -> /DMA/XA2
- U23 pad 35: (no net) -> /DMA/XA3
- U23 pad 37: (no net) -> /DMA/XA4
- U23 pad 38: (no net) -> /DMA/XA5
- U23 pad 39: (no net) -> /DMA/XA6
- U23 pad 4: (no net) -> /DMA/~XMEMW
- U23 pad 40: (no net) -> /DMA/XA7
- U23 pad 7: (no net) -> /DMA/HLDA
- U23 pad 9: /DMA/BUSEN -> Net-(U23-Pad9)
- U24 pad 1: /DMA/BUSEN -> (no net)
- U24 pad 2: Net-(U24-Pad2) -> (no net)
- U25 pad 1: Net-(U24-Pad2) -> /DMA/~DMAEN
- U25 pad 11: Net-(U23-Pad8) -> /DMA/XA3
- U25 pad 12: (no net) -> /DMA/A4
- U25 pad 13: (no net) -> /DMA/XA2
- U25 pad 14: (no net) -> /DMA/A5
- U25 pad 15: (no net) -> /DMA/XA1
- U25 pad 16: (no net) -> /DMA/A6
- U25 pad 17: (no net) -> /DMA/XA0
- U25 pad 18: (no net) -> /DMA/A7
- U25 pad 19: (no net) -> /DMA/~DMAEN
- U25 pad 2: (no net) -> /DMA/XA7
- U25 pad 3: (no net) -> /DMA/A0
- U25 pad 4: (no net) -> /DMA/XA6
- U25 pad 5: (no net) -> /DMA/A1
- U25 pad 6: (no net) -> /DMA/XA5
- U25 pad 7: (no net) -> /DMA/A2
- U25 pad 8: (no net) -> /DMA/XA4
- U25 pad 9: (no net) -> /DMA/A3
- U26 pad 1: Net-(U24-Pad2) -> /DMA/~DMAEN
- U26 pad 12: (no net) -> /DMA/A11
- U26 pad 13: (no net) -> /DMA/XD3
- U26 pad 14: (no net) -> /DMA/XD2
- U26 pad 15: (no net) -> /DMA/A10
- U26 pad 16: (no net) -> /DMA/A9
- U26 pad 17: (no net) -> /DMA/XD1
- U26 pad 18: (no net) -> /DMA/XD0
- U26 pad 19: (no net) -> /DMA/A8
- U26 pad 2: (no net) -> /DMA/A15
- U26 pad 3: (no net) -> /DMA/XD7
- U26 pad 4: (no net) -> /DMA/XD6
- U26 pad 5: (no net) -> /DMA/A14
- U26 pad 6: (no net) -> /DMA/A13
- U26 pad 7: (no net) -> /DMA/XD5
- U26 pad 8: (no net) -> /DMA/XD4
- U26 pad 9: (no net) -> /DMA/A12
- U27 pad 1: (no net) -> /DMA/XD1
- U27 pad 10: (no net) -> /DMA/A16
- U27 pad 11: Net-(U24-Pad2) -> /DMA/~DMAEN
- U27 pad 12: (no net) -> /DMA/~WRTDMAPGRES
- U27 pad 13: (no net) -> /DMA/XA1
- U27 pad 14: (no net) -> /DMA/XA0
- U27 pad 15: (no net) -> /DMA/XD0
- U27 pad 16: (no net) -> Net-(U27-Pad16)
- U27 pad 2: (no net) -> /DMA/XD2
- U27 pad 3: (no net) -> /DMA/XD3
- U27 pad 6: (no net) -> /DMA/A19
- U27 pad 7: (no net) -> /DMA/A18
- U27 pad 8: (no net) -> Net-(U27-Pad8)
- U27 pad 9: (no net) -> /DMA/A17
- U28 pad 11: (no net) -> Net-(U28-Pad11)
- U28 pad 13: /IO-Decoder/~IORC -> /~IOR
- U28 pad 17: (no net) -> Net-(U28-Pad17)
- U28 pad 5: /ALE -> /IO-Decoder/ALE
- U29 pad 11: /D0 -> /HDD Controller/D0
- U29 pad 12: /D1 -> /HDD Controller/D1
- U29 pad 13: /D2 -> /HDD Controller/D2
- U29 pad 14: /D3 -> /HDD Controller/D3
- U29 pad 15: /D4 -> /HDD Controller/D4
- U29 pad 16: /D5 -> /HDD Controller/D5
- U29 pad 17: /D6 -> /HDD Controller/D6
- U29 pad 18: /D7 -> /HDD Controller/D7
- U3 pad 1: (no net) -> /INT_CS
- U3 pad 10: /D1 -> /XD1
- U3 pad 11: /D0 -> /XD0
- U3 pad 12: (no net) -> Net-(U3-Pad12)
- U3 pad 13: (no net) -> Net-(U3-Pad13)
- U3 pad 14: (no net) -> GND
- U3 pad 15: (no net) -> Net-(U3-Pad15)
- U3 pad 16: (no net) -> /PU
- U3 pad 17: (no net) -> /INTR
- U3 pad 18: (no net) -> /IRQ0
- U3 pad 19: (no net) -> /IRQ1
- U3 pad 2: (no net) -> /~XIOR
- U3 pad 20: (no net) -> /IRQ2
- U3 pad 21: (no net) -> /IRQ3
- U3 pad 22: (no net) -> /IRQ4
- U3 pad 23: (no net) -> /IRQ5
- U3 pad 24: (no net) -> /IRQ6
- U3 pad 25: (no net) -> /IRQ7
- U3 pad 27: (no net) -> /XA0
- U3 pad 28: (no net) -> +5V
- U3 pad 3: (no net) -> /~XIOW
- U3 pad 4: /D7 -> /XD7
- U3 pad 5: /D6 -> /XD6
- U3 pad 6: /D5 -> /XD5
- U3 pad 7: /D4 -> /XD4
- U3 pad 8: /D3 -> /XD3
- U3 pad 9: /D2 -> /XD2
- U30 pad 3: /SYS_CLK -> /IO-Decoder/XCLK
- U31 pad 11: /ALE -> /IO-Decoder/ALE
- U31 pad 20: (no net) -> Net-(U31-Pad20)
- U32 pad 11: (no net) -> Net-(U32-Pad11)
- U32 pad 13: (no net) -> Net-(U32-Pad13)
- U32 pad 15: (no net) -> Net-(U32-Pad15)
- U32 pad 17: (no net) -> Net-(U32-Pad17)
- U32 pad 19: (no net) -> Net-(U32-Pad19)
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Routing:
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- added copper zone on PWR, net +5V
- added copper zone on GND, net GND
- removed copper zone on F.Cu, net +5V
- removed copper zone on B.Cu, net GND
Other:
- copper layers 2 -> 4
- board text added: "U38, C21, D1, C22 Only if -5V not present on PSU"

Commit message: end of day commit, routed major parts of the motherboard
Parts:
- added U53: 74LS322, Package_DIP:DIP-20_W7.62mm_Socket, F.Cu at (194.1, 214.9)
- moved U34 314.2 mm to (42.7, 275.3)
- moved U25 305.1 mm to (109.2, 223.5)
- moved R5 296.3 mm to (96.4, 286.3)
- moved U30 296.3 mm to (108.4, 268.0)
- moved U41 296.3 mm to (119.1, 268.0)
- moved R10 296.3 mm to (55.8, 301.8)
- moved U36 296.3 mm to (79.1, 283.8)
- moved U40 296.3 mm to (92.8, 262.6)
- moved U24 294.2 mm to (84.6, 364.2)
- moved U26 281.5 mm to (53.3, 194.3)
- moved U27 261.0 mm to (86.4, 201.9), turned to 270 degrees
- moved U23 260.0 mm to (114.3, 180.3), turned to 270 degrees
- moved U49 252.1 mm to (137.2, 181.6), turned to 270 degrees
- moved RN1 235.6 mm to (111.8, 144.8), turned to 180 degrees
- moved RN2 223.5 mm to (132.1, 193.0), turned to 180 degrees
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Connections:
- net /DMA/~WRTDMAPGRES renamed /~WRTDMAPGREG
- net /INT_CS renamed /~INTRCS
- net /IO-Decoder/XA5 renamed /XA5
- net /IO-Decoder/XA6 renamed /XA6
- net /IO-Decoder/XA7 renamed /XA7
- net /IO-Decoder/XA8 renamed /XA8
- net /IO-Decoder/XA9 renamed /XA9
- net /IRQ2 renamed /SIRQ
- J5 pad 4: Net-(J5-Pad4) -> /ISA/IRQ2
- J5 pad 6: Net-(J5-Pad6) -> /ISA/DRQ2
- J6 pad 4: Net-(J6-Pad4) -> /ISA/IRQ2
- J6 pad 6: Net-(J6-Pad6) -> /ISA/DRQ2
- J7 pad 4: Net-(J7-Pad4) -> /ISA/IRQ2
- J7 pad 6: Net-(J7-Pad6) -> /ISA/DRQ2
- RN2 pad 2: /IO-Decoder/~XMEMR -> /~XMEMR
- RN2 pad 4: /IO-Decoder/~XMEMW -> /~XMEMW
- U23 pad 3: /DMA/~XMEMR -> /~XMEMR
- U23 pad 4: /DMA/~XMEMW -> /~XMEMW
- U24 pad 4: /DMA/TC -> /TC
- U42 pad 17: /IO-Decoder/~XMEMW -> /~XMEMW
- U42 pad 41: /IO-Decoder/~XMEMR -> /~XMEMR
- U45 pad 17: /IO-Decoder/~XMEMW -> /~XMEMW
- U47 pad 1: /IO-Decoder/~XMEMR -> /~XMEMR
- U49 pad 11: /IO-Decoder/~XMEMR -> /~XMEMR
- U49 pad 9: /IO-Decoder/~XMEMW -> /~XMEMW
- U51 pad 9: /IO-Decoder/~XMEMR -> /~XMEMR
Routing:
- net /FDC-Serial/A7: track 0.00 -> 407.8 mm, vias 0 -> 10
- net /FDC-Serial/A0: track 0.00 -> 386.5 mm, vias 0 -> 9
- net /FDC-Serial/A5: track 0.00 -> 374.0 mm, vias 0 -> 11
- net /FDC-Serial/A4: track 0.00 -> 364.6 mm, vias 0 -> 8
- net /FDC-Serial/A2: track 0.00 -> 339.7 mm, vias 0 -> 10
- net /FDC-Serial/A3: track 0.00 -> 334.6 mm, vias 0 -> 8
- net /FDC-Serial/A6: track 0.00 -> 329.5 mm, vias 0 -> 10
- net /FDC-Serial/A1: track 0.00 -> 316.1 mm, vias 0 -> 11
- net +3V3: track 29.7 -> 334.1 mm
- net /SYS_CLK: track 0.00 -> 283.6 mm, vias 0 -> 6
- net /HDD Controller/A16: track 0.00 -> 282.1 mm, vias 0 -> 4
- net /FDC-Serial/A8: track 0.00 -> 279.5 mm, vias 0 -> 5
- net /FDC-Serial/A9: track 0.00 -> 277.7 mm, vias 0 -> 3
- net +12V: track 0.00 -> 274.1 mm, vias 0 -> 2
- net /FDC-Serial/A11: track 0.00 -> 271.3 mm, vias 0 -> 7
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Other:
- net class Default: via_dia 0.8 -> 0.45

Commit message: end of day commit, almost finished routing motherboard
Parts:
- moved U53 164.7 mm to (31.0, 238.4), turned to 90 degrees
- moved U24 114.3 mm to (73.7, 250.4), turned to 90 degrees
- moved R10 113.6 mm to (77.9, 190.4)
- moved U36 112.0 mm to (78.0, 171.8)
- moved U34 106.2 mm to (66.4, 171.8)
- moved U40 105.1 mm to (174.4, 196.4)
- moved U26 98.6 mm to (145.6, 228.9), turned to 270 degrees
- moved U30 89.6 mm to (90.0, 180.3)
- moved R5 86.3 mm to (93.8, 200.1)
- moved U41 77.6 mm to (157.3, 200.5)
- moved U25 48.0 mm to (66.6, 201.5), turned to 0 degrees
- moved U23 47.0 mm to (88.7, 219.7), turned to 90 degrees
- moved U27 39.4 mm to (115.2, 228.8)
- moved U49 37.1 mm to (102.1, 193.9), turned to 90 degrees
- moved RN2 27.0 mm to (107.2, 182.4), turned to 0 degrees
Routing:
- net /~IOR: track 16.8 -> 506.9 mm, vias 1 -> 19
- net /~DACK0: track 0.00 -> 329.0 mm, vias 0 -> 8
- net /DRQ2: track 0.00 -> 305.8 mm, vias 0 -> 4
- net /DRQ0: track 0.00 -> 302.8 mm, vias 0 -> 8
- net /DRQ1: track 0.00 -> 300.9 mm, vias 0 -> 6
- net /DRQ3: track 0.00 -> 275.6 mm, vias 0 -> 10
- net /N.P.NPI: track 0.00 -> 275.0 mm, vias 0 -> 3
- net /RESET: track 111.0 -> 383.6 mm, vias 0 -> 11
- net /~XMEMR: track 3.81 -> 273.6 mm, vias 0 -> 9
- net /IO-Decoder/AENBRD: track 0.00 -> 265.4 mm, vias 0 -> 6
- net /~XMEMW: track 3.81 -> 253.5 mm, vias 0 -> 9
- net /IRQ6: track 32.1 -> 241.7 mm, vias 2 -> 4
- net /IRQ7: track 32.6 -> 240.3 mm, vias 2 -> 6
- net /IRQ4: track 31.4 -> 238.3 mm, vias 2 -> 4
- net /~DACK0BRD: track 0.00 -> 206.9 mm, vias 0 -> 2
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
Commit message: done all routing for available traces, 2 traces have a netlist issue
Connections:
- net /ISA/~MEMW renamed /~MEMW
- net Net-(U1-Pad24) renamed /~TCCS
- net Net-(U6-Pad39) renamed /IRQ14
- net Net-(U6-Pad40) renamed /IRQ15
- net Net-(U6-Pad89) renamed /IRQ8
- net Net-(U6-Pad90) renamed /IRQ10
- net Net-(U6-Pad91) renamed /IRQ11
- net Net-(U6-Pad92) renamed /IRQ12
- J2 pad 12: /ISA/~MEMR -> /~MEMR
- J2 pad 15: /ISA/~DACK3 -> /~DACK3
- J2 pad 16: /ISA/DRQ3 -> /DRQ3
- J2 pad 17: /ISA/~DACK1 -> /~DACK1
- J2 pad 18: /ISA/DRQ1 -> /DRQ1
- J2 pad 19: /ISA/~DACK0 -> /~DACK0BRD
- J2 pad 26: /ISA/~DACK2 -> /~DACK2
- J2 pad 33: /HDD Controller/D7 -> /FDC-Serial/D7
- J2 pad 34: /HDD Controller/D6 -> /FDC-Serial/D6
- J2 pad 35: /HDD Controller/D5 -> /FDC-Serial/D5
- J2 pad 36: /HDD Controller/D4 -> /FDC-Serial/D4
- J2 pad 37: /HDD Controller/D3 -> /FDC-Serial/D3
- J2 pad 38: /HDD Controller/D2 -> /FDC-Serial/D2
- J2 pad 39: /HDD Controller/D1 -> /FDC-Serial/D1
- J2 pad 40: /HDD Controller/D0 -> /FDC-Serial/D0
- J2 pad 43: /HDD Controller/A19 -> /DMA/A19
- J2 pad 44: /HDD Controller/A18 -> /DMA/A18
- J2 pad 45: /HDD Controller/A17 -> /DMA/A17
- J2 pad 46: /HDD Controller/A16 -> /DMA/A16
- J2 pad 47: /FDC-Serial/A15 -> /DMA/A15
- J2 pad 48: /FDC-Serial/A14 -> /DMA/A14
- J2 pad 49: /FDC-Serial/A13 -> /DMA/A13
- J2 pad 50: /FDC-Serial/A12 -> /DMA/A12
- J2 pad 51: /FDC-Serial/A11 -> /DMA/A11
- J2 pad 52: /FDC-Serial/A10 -> /DMA/A10
- J2 pad 53: /FDC-Serial/A9 -> /DMA/A9
- J2 pad 54: /FDC-Serial/A8 -> /DMA/A8
- J2 pad 55: /FDC-Serial/A7 -> /DMA/A7
- J2 pad 56: /FDC-Serial/A6 -> /DMA/A6
- J2 pad 57: /FDC-Serial/A5 -> /DMA/A5
- J2 pad 58: /FDC-Serial/A4 -> /DMA/A4
- J2 pad 59: /FDC-Serial/A3 -> /DMA/A3
- J2 pad 6: /ISA/DRQ2 -> /DRQ2
- J2 pad 60: /FDC-Serial/A2 -> /DMA/A2
- J2 pad 61: /FDC-Serial/A1 -> /DMA/A1
- J2 pad 62: /FDC-Serial/A0 -> /DMA/A0
- J3 pad 12: /ISA/~MEMR -> /~MEMR
- J3 pad 15: /ISA/~DACK3 -> /~DACK3
- J3 pad 16: /ISA/DRQ3 -> /DRQ3
- J3 pad 17: /ISA/~DACK1 -> /~DACK1
- J3 pad 18: /ISA/DRQ1 -> /DRQ1
- J3 pad 19: /ISA/~DACK0 -> /~DACK0BRD
- J3 pad 26: /ISA/~DACK2 -> /~DACK2
- J3 pad 32: Net-(J3-Pad32) -> /ISA/IOCHCK
- J3 pad 33: /HDD Controller/D7 -> /FDC-Serial/D7
- J3 pad 34: /HDD Controller/D6 -> /FDC-Serial/D6
- J3 pad 35: /HDD Controller/D5 -> /FDC-Serial/D5
- J3 pad 36: /HDD Controller/D4 -> /FDC-Serial/D4
- J3 pad 37: /HDD Controller/D3 -> /FDC-Serial/D3
- J3 pad 38: /HDD Controller/D2 -> /FDC-Serial/D2
- J3 pad 39: /HDD Controller/D1 -> /FDC-Serial/D1
- J3 pad 40: /HDD Controller/D0 -> /FDC-Serial/D0
- J3 pad 43: /HDD Controller/A19 -> /DMA/A19
- J3 pad 44: /HDD Controller/A18 -> /DMA/A18
- J3 pad 45: /HDD Controller/A17 -> /DMA/A17
- J3 pad 46: /HDD Controller/A16 -> /DMA/A16
- J3 pad 47: /FDC-Serial/A15 -> /DMA/A15
- J3 pad 48: /FDC-Serial/A14 -> /DMA/A14
- J3 pad 49: /FDC-Serial/A13 -> /DMA/A13
- J3 pad 50: /FDC-Serial/A12 -> /DMA/A12
- J3 pad 51: /FDC-Serial/A11 -> /DMA/A11
- J3 pad 52: /FDC-Serial/A10 -> /DMA/A10
- J3 pad 53: /FDC-Serial/A9 -> /DMA/A9
- J3 pad 54: /FDC-Serial/A8 -> /DMA/A8
- J3 pad 55: /FDC-Serial/A7 -> /DMA/A7
- J3 pad 56: /FDC-Serial/A6 -> /DMA/A6
- J3 pad 57: /FDC-Serial/A5 -> /DMA/A5
- J3 pad 58: /FDC-Serial/A4 -> /DMA/A4
- J3 pad 59: /FDC-Serial/A3 -> /DMA/A3
- J3 pad 6: /ISA/DRQ2 -> /DRQ2
- J3 pad 60: /FDC-Serial/A2 -> /DMA/A2
- J3 pad 61: /FDC-Serial/A1 -> /DMA/A1
- J3 pad 62: /FDC-Serial/A0 -> /DMA/A0
- J5 pad 12: /ISA/~MEMR -> /~MEMR
- J5 pad 15: /ISA/~DACK3 -> /~DACK3
- J5 pad 16: /ISA/DRQ3 -> /DRQ3
- J5 pad 17: /ISA/~DACK1 -> /~DACK1
- J5 pad 18: /ISA/DRQ1 -> /DRQ1
- J5 pad 19: /ISA/~DACK0 -> /~DACK0BRD
- J5 pad 26: /ISA/~DACK2 -> /~DACK2
- J5 pad 32: Net-(J5-Pad32) -> /ISA/IOCHCK
- J5 pad 33: /HDD Controller/D7 -> /FDC-Serial/D7
- J5 pad 34: /HDD Controller/D6 -> /FDC-Serial/D6
- J5 pad 35: /HDD Controller/D5 -> /FDC-Serial/D5
- J5 pad 36: /HDD Controller/D4 -> /FDC-Serial/D4
- J5 pad 37: /HDD Controller/D3 -> /FDC-Serial/D3
- J5 pad 38: /HDD Controller/D2 -> /FDC-Serial/D2
- J5 pad 39: /HDD Controller/D1 -> /FDC-Serial/D1
- J5 pad 4: /ISA/IRQ2 -> Net-(J5-Pad4)
- J5 pad 40: /HDD Controller/D0 -> /FDC-Serial/D0
- J5 pad 43: /HDD Controller/A19 -> /DMA/A19
- J5 pad 44: /HDD Controller/A18 -> /DMA/A18
- J5 pad 45: /HDD Controller/A17 -> /DMA/A17
- J5 pad 46: /HDD Controller/A16 -> /DMA/A16
- J5 pad 47: /FDC-Serial/A15 -> /DMA/A15
- J5 pad 48: /FDC-Serial/A14 -> /DMA/A14
- J5 pad 49: /FDC-Serial/A13 -> /DMA/A13
- J5 pad 50: /FDC-Serial/A12 -> /DMA/A12
- J5 pad 51: /FDC-Serial/A11 -> /DMA/A11
- J5 pad 52: /FDC-Serial/A10 -> /DMA/A10
- J5 pad 53: /FDC-Serial/A9 -> /DMA/A9
- J5 pad 54: /FDC-Serial/A8 -> /DMA/A8
- J5 pad 55: /FDC-Serial/A7 -> /DMA/A7
- J5 pad 56: /FDC-Serial/A6 -> /DMA/A6
- J5 pad 57: /FDC-Serial/A5 -> /DMA/A5
- J5 pad 58: /FDC-Serial/A4 -> /DMA/A4
- J5 pad 59: /FDC-Serial/A3 -> /DMA/A3
- J5 pad 6: /ISA/DRQ2 -> Net-(J5-Pad6)
- J5 pad 60: /FDC-Serial/A2 -> /DMA/A2
- J5 pad 61: /FDC-Serial/A1 -> /DMA/A1
- J5 pad 62: /FDC-Serial/A0 -> /DMA/A0
- J6 pad 12: /ISA/~MEMR -> /~MEMR
- J6 pad 15: /ISA/~DACK3 -> /~DACK3
- J6 pad 16: /ISA/DRQ3 -> /DRQ3
- J6 pad 17: /ISA/~DACK1 -> /~DACK1
- J6 pad 18: /ISA/DRQ1 -> /DRQ1
- J6 pad 19: /ISA/~DACK0 -> /~DACK0BRD
- J6 pad 26: /ISA/~DACK2 -> /~DACK2
- J6 pad 32: Net-(J6-Pad32) -> /ISA/IOCHCK
- J6 pad 33: /HDD Controller/D7 -> /FDC-Serial/D7
- J6 pad 34: /HDD Controller/D6 -> /FDC-Serial/D6
- J6 pad 35: /HDD Controller/D5 -> /FDC-Serial/D5
- J6 pad 36: /HDD Controller/D4 -> /FDC-Serial/D4
- J6 pad 37: /HDD Controller/D3 -> /FDC-Serial/D3
- J6 pad 38: /HDD Controller/D2 -> /FDC-Serial/D2
- J6 pad 39: /HDD Controller/D1 -> /FDC-Serial/D1
- J6 pad 4: /ISA/IRQ2 -> Net-(J6-Pad4)
- J6 pad 40: /HDD Controller/D0 -> /FDC-Serial/D0
- J6 pad 43: /HDD Controller/A19 -> /DMA/A19
- J6 pad 44: /HDD Controller/A18 -> /DMA/A18
- J6 pad 45: /HDD Controller/A17 -> /DMA/A17
- J6 pad 46: /HDD Controller/A16 -> /DMA/A16
- J6 pad 47: /FDC-Serial/A15 -> /DMA/A15
- J6 pad 48: /FDC-Serial/A14 -> /DMA/A14
- J6 pad 49: /FDC-Serial/A13 -> /DMA/A13
- J6 pad 50: /FDC-Serial/A12 -> /DMA/A12
- J6 pad 51: /FDC-Serial/A11 -> /DMA/A11
- J6 pad 52: /FDC-Serial/A10 -> /DMA/A10
- J6 pad 53: /FDC-Serial/A9 -> /DMA/A9
- J6 pad 54: /FDC-Serial/A8 -> /DMA/A8
- J6 pad 55: /FDC-Serial/A7 -> /DMA/A7
- J6 pad 56: /FDC-Serial/A6 -> /DMA/A6
- J6 pad 57: /FDC-Serial/A5 -> /DMA/A5
- J6 pad 58: /FDC-Serial/A4 -> /DMA/A4
- J6 pad 59: /FDC-Serial/A3 -> /DMA/A3
- J6 pad 6: /ISA/DRQ2 -> Net-(J6-Pad6)
- J6 pad 60: /FDC-Serial/A2 -> /DMA/A2
- J6 pad 61: /FDC-Serial/A1 -> /DMA/A1
- J6 pad 62: /FDC-Serial/A0 -> /DMA/A0
- J7 pad 12: /ISA/~MEMR -> /~MEMR
- J7 pad 15: /ISA/~DACK3 -> /~DACK3
- J7 pad 16: /ISA/DRQ3 -> /DRQ3
- J7 pad 17: /ISA/~DACK1 -> /~DACK1
- J7 pad 18: /ISA/DRQ1 -> /DRQ1
- J7 pad 19: /ISA/~DACK0 -> /~DACK0BRD
- J7 pad 26: /ISA/~DACK2 -> /~DACK2
- J7 pad 32: Net-(J7-Pad32) -> /ISA/IOCHCK
- J7 pad 33: /HDD Controller/D7 -> /FDC-Serial/D7
- J7 pad 34: /HDD Controller/D6 -> /FDC-Serial/D6
- J7 pad 35: /HDD Controller/D5 -> /FDC-Serial/D5
- J7 pad 36: /HDD Controller/D4 -> /FDC-Serial/D4
- J7 pad 37: /HDD Controller/D3 -> /FDC-Serial/D3
- J7 pad 38: /HDD Controller/D2 -> /FDC-Serial/D2
- J7 pad 39: /HDD Controller/D1 -> /FDC-Serial/D1
- J7 pad 4: /ISA/IRQ2 -> Net-(J7-Pad4)
- J7 pad 40: /HDD Controller/D0 -> /FDC-Serial/D0
- J7 pad 43: /HDD Controller/A19 -> /DMA/A19
- J7 pad 44: /HDD Controller/A18 -> /DMA/A18
- J7 pad 45: /HDD Controller/A17 -> /DMA/A17
- J7 pad 46: /HDD Controller/A16 -> /DMA/A16
- J7 pad 47: /FDC-Serial/A15 -> /DMA/A15
- J7 pad 48: /FDC-Serial/A14 -> /DMA/A14
- J7 pad 49: /FDC-Serial/A13 -> /DMA/A13
- J7 pad 50: /FDC-Serial/A12 -> /DMA/A12
- J7 pad 51: /FDC-Serial/A11 -> /DMA/A11
- J7 pad 52: /FDC-Serial/A10 -> /DMA/A10
- J7 pad 53: /FDC-Serial/A9 -> /DMA/A9
- J7 pad 54: /FDC-Serial/A8 -> /DMA/A8
- J7 pad 55: /FDC-Serial/A7 -> /DMA/A7
- J7 pad 56: /FDC-Serial/A6 -> /DMA/A6
- J7 pad 57: /FDC-Serial/A5 -> /DMA/A5
- J7 pad 58: /FDC-Serial/A4 -> /DMA/A4
- J7 pad 59: /FDC-Serial/A3 -> /DMA/A3
- J7 pad 6: /ISA/DRQ2 -> Net-(J7-Pad6)
- J7 pad 60: /FDC-Serial/A2 -> /DMA/A2
- J7 pad 61: /FDC-Serial/A1 -> /DMA/A1
- J7 pad 62: /FDC-Serial/A0 -> /DMA/A0
- R9 pad 1: /IO-Decoder/IO_SigDecoder/IOCHCK -> /IO-Decoder/IO_SigDecoder/IOCHCK_I
- RN1 pad 5: /IO-Decoder/~MRDC -> /~MEMR
- U12 pad 10: /FDC-Serial/A8 -> /DMA/A8
- U12 pad 11: /FDC-Serial/A9 -> /DMA/A9
- U12 pad 2: /FDC-Serial/A0 -> /DMA/A0
- U12 pad 3: /FDC-Serial/A1 -> /DMA/A1
- U12 pad 4: /FDC-Serial/A2 -> /DMA/A2
- U12 pad 5: /FDC-Serial/A3 -> /DMA/A3
- U12 pad 6: /FDC-Serial/A4 -> /DMA/A4
- U12 pad 7: /FDC-Serial/A5 -> /DMA/A5
- U12 pad 8: /FDC-Serial/A6 -> /DMA/A6
- U12 pad 9: /FDC-Serial/A7 -> /DMA/A7
- U13 pad 27: /FDC-Serial/A0 -> /DMA/A0
- U14 pad 1: /HDD Controller/D2 -> /FDC-Serial/D2
- U14 pad 10: /HDD Controller/D7 -> /FDC-Serial/D7
- U14 pad 11: /HDD Controller/D6 -> /FDC-Serial/D6
- U14 pad 12: /HDD Controller/D5 -> /FDC-Serial/D5
- U14 pad 13: /HDD Controller/D4 -> /FDC-Serial/D4
- U14 pad 15: /HDD Controller/D3 -> /FDC-Serial/D3
- U14 pad 2: /HDD Controller/D1 -> /FDC-Serial/D1
- U14 pad 3: /HDD Controller/D0 -> /FDC-Serial/D0
- U23 pad 14: /DMA/DACK2 -> /~DACK2
- U23 pad 15: /DACK3 -> /~DACK3
- U23 pad 21: /DMA/XD7 -> /XD7
- U23 pad 22: /DMA/XD6 -> /XD6
- U23 pad 23: /DMA/XD5 -> /XD5
- U23 pad 24: /DMA/DACK1 -> /~DACK1
- U23 pad 26: /DMA/XD4 -> /XD4
- U23 pad 27: /DMA/XD3 -> /XD3
- U23 pad 28: /DMA/XD2 -> /XD2
- U23 pad 29: /DMA/XD1 -> /XD1
- U23 pad 30: /DMA/XD0 -> /XD0
- U23 pad 32: /DMA/XA0 -> /XA0
- U23 pad 33: /DMA/XA1 -> /XA1
- U23 pad 38: /DMA/XA5 -> /XA5
- U23 pad 39: /DMA/XA6 -> /XA6
- U23 pad 40: /DMA/XA7 -> /XA7
- U25 pad 15: /DMA/XA1 -> /XA1
- U25 pad 17: /DMA/XA0 -> /XA0
- U25 pad 2: /DMA/XA7 -> /XA7
- U25 pad 4: /DMA/XA6 -> /XA6
- U25 pad 6: /DMA/XA5 -> /XA5
- U26 pad 13: /DMA/XD3 -> /XD3
- U26 pad 14: /DMA/XD2 -> /XD2
- U26 pad 17: /DMA/XD1 -> /XD1
- U26 pad 18: /DMA/XD0 -> /XD0
- U26 pad 3: /DMA/XD7 -> /XD7
- U26 pad 4: /DMA/XD6 -> /XD6
- U26 pad 7: /DMA/XD5 -> /XD5
- U26 pad 8: /DMA/XD4 -> /XD4
- U27 pad 1: /DMA/XD1 -> /XD1
- U27 pad 13: /DMA/XA1 -> /XA1
- U27 pad 14: /DMA/XA0 -> /XA0
- U27 pad 15: /DMA/XD0 -> /XD0
- U27 pad 16: Net-(U27-Pad16) -> +5V
- U27 pad 2: /DMA/XD2 -> /XD2
- U27 pad 3: /DMA/XD3 -> /XD3
- U27 pad 4: /DMA/DACK2 -> /~DACK2
- U27 pad 5: /DACK3 -> /~DACK3
- U27 pad 8: Net-(U27-Pad8) -> GND
- U28 pad 5: /IO-Decoder/ALE -> /ALE
- U28 pad 7: /IO-Decoder/~MRDC -> /~MEMR
- U29 pad 11: /HDD Controller/D0 -> /FDC-Serial/D0
- U29 pad 12: /HDD Controller/D1 -> /FDC-Serial/D1
- U29 pad 13: /HDD Controller/D2 -> /FDC-Serial/D2
- U29 pad 14: /HDD Controller/D3 -> /FDC-Serial/D3
- U29 pad 15: /HDD Controller/D4 -> /FDC-Serial/D4
- U29 pad 16: /HDD Controller/D5 -> /FDC-Serial/D5
- U29 pad 17: /HDD Controller/D6 -> /FDC-Serial/D6
- U29 pad 18: /HDD Controller/D7 -> /FDC-Serial/D7
- U31 pad 11: /IO-Decoder/ALE -> /ALE
- U31 pad 12: /FDC-Serial/A12 -> /DMA/A12
- U31 pad 13: /FDC-Serial/A13 -> /DMA/A13
- U31 pad 14: /FDC-Serial/A14 -> /DMA/A14
- U31 pad 15: /FDC-Serial/A15 -> /DMA/A15
- U31 pad 16: /HDD Controller/A16 -> /DMA/A16
- U31 pad 17: /HDD Controller/A17 -> /DMA/A17
- U31 pad 18: /HDD Controller/A18 -> /DMA/A18
- U31 pad 19: /HDD Controller/A19 -> /DMA/A19
- U32 pad 12: /FDC-Serial/A8 -> /DMA/A8
- U32 pad 14: /FDC-Serial/A9 -> /DMA/A9
- U32 pad 16: /FDC-Serial/A10 -> /DMA/A10
- U32 pad 18: /FDC-Serial/A11 -> /DMA/A11
- U33 pad 11: /IO-Decoder/ALE -> /ALE
- U33 pad 12: /FDC-Serial/A0 -> /DMA/A0
- U33 pad 13: /FDC-Serial/A1 -> /DMA/A1
- U33 pad 14: /FDC-Serial/A2 -> /DMA/A2
- U33 pad 15: /FDC-Serial/A3 -> /DMA/A3
- U33 pad 16: /FDC-Serial/A4 -> /DMA/A4
- U33 pad 17: /FDC-Serial/A5 -> /DMA/A5
- U33 pad 18: /FDC-Serial/A6 -> /DMA/A6
- U33 pad 19: /FDC-Serial/A7 -> /DMA/A7
- U35 pad 11: /HDD Controller/D7 -> /FDC-Serial/D7
- U35 pad 12: /HDD Controller/D6 -> /FDC-Serial/D6
- U35 pad 13: /HDD Controller/D5 -> /FDC-Serial/D5
- U35 pad 14: /HDD Controller/D4 -> /FDC-Serial/D4
- U35 pad 15: /HDD Controller/D3 -> /FDC-Serial/D3
- U35 pad 16: /HDD Controller/D2 -> /FDC-Serial/D2
- U35 pad 17: /HDD Controller/D1 -> /FDC-Serial/D1
- U35 pad 18: /HDD Controller/D0 -> /FDC-Serial/D0
- U39 pad 1: /HDD Controller/A19 -> /DMA/A19
- U39 pad 10: /FDC-Serial/A7 -> /DMA/A7
- U39 pad 11: /FDC-Serial/A6 -> /DMA/A6
- U39 pad 13: /FDC-Serial/A5 -> /DMA/A5
- U39 pad 2: /HDD Controller/A18 -> /DMA/A18
- U39 pad 3: /HDD Controller/A17 -> /DMA/A17
- U39 pad 4: /HDD Controller/A16 -> /DMA/A16
- U39 pad 5: /FDC-Serial/A15 -> /DMA/A15
- U39 pad 6: /FDC-Serial/A14 -> /DMA/A14
- U39 pad 7: /FDC-Serial/A13 -> /DMA/A13
- U39 pad 8: /FDC-Serial/A9 -> /DMA/A9
- U39 pad 9: /FDC-Serial/A8 -> /DMA/A8
- U42 pad 1: /IO-Decoder/XA4 -> /DMA/XA4
- U42 pad 2: /IO-Decoder/XA3 -> /DMA/XA3
- U42 pad 3: /IO-Decoder/XA2 -> /DMA/XA2
- U43 pad 11: /FDC-Serial/A4 -> /DMA/A4
- U43 pad 12: /IO-Decoder/XA3 -> /DMA/XA3
- U43 pad 13: /FDC-Serial/A5 -> /DMA/A5
- U43 pad 14: /IO-Decoder/XA2 -> /DMA/XA2
- U43 pad 15: /FDC-Serial/A6 -> /DMA/A6
- U43 pad 17: /FDC-Serial/A7 -> /DMA/A7
- U43 pad 2: /FDC-Serial/A0 -> /DMA/A0
- U43 pad 4: /FDC-Serial/A1 -> /DMA/A1
- U43 pad 6: /FDC-Serial/A2 -> /DMA/A2
- U43 pad 8: /FDC-Serial/A3 -> /DMA/A3
- U43 pad 9: /IO-Decoder/XA4 -> /DMA/XA4
- U44 pad 11: /FDC-Serial/A12 -> /DMA/A12
- U44 pad 13: /FDC-Serial/A13 -> /DMA/A13
- U44 pad 15: /FDC-Serial/A14 -> /DMA/A14
- U44 pad 17: /FDC-Serial/A15 -> /DMA/A15
- U44 pad 2: /FDC-Serial/A8 -> /DMA/A8
- U44 pad 4: /FDC-Serial/A9 -> /DMA/A9
- U44 pad 6: /FDC-Serial/A10 -> /DMA/A10
- U44 pad 8: /FDC-Serial/A11 -> /DMA/A11
- U45 pad 2: /HDD Controller/A16 -> /DMA/A16
- U45 pad 4: /HDD Controller/A17 -> /DMA/A17
- U45 pad 6: /HDD Controller/A18 -> /DMA/A18
- U45 pad 8: /HDD Controller/A19 -> /DMA/A19
- U46 pad 2: /HDD Controller/D0 -> /FDC-Serial/D0
- U46 pad 3: /HDD Controller/D1 -> /FDC-Serial/D1
- U46 pad 4: /HDD Controller/D2 -> /FDC-Serial/D2
- U46 pad 5: /HDD Controller/D3 -> /FDC-Serial/D3
- U46 pad 6: /HDD Controller/D4 -> /FDC-Serial/D4
- U46 pad 7: /HDD Controller/D5 -> /FDC-Serial/D5
- U46 pad 8: /HDD Controller/D6 -> /FDC-Serial/D6
- U46 pad 9: /HDD Controller/D7 -> /FDC-Serial/D7
- U48 pad 10: /IO-Decoder/XA2 -> /DMA/XA2
- U48 pad 8: /IO-Decoder/XA4 -> /DMA/XA4
- U48 pad 9: /IO-Decoder/XA3 -> /DMA/XA3
- U49 pad 3: /IO-Decoder/~MRDC -> /~MEMR
- U51 pad 12: Net-(U51-Pad12) -> GND
- U51 pad 23: /IO-Decoder/IO_SigDecoder/IOCHCK -> /IO-Decoder/IO_SigDecoder/IOCHCK_O
- U51 pad 24: Net-(U51-Pad24) -> +5V
- U51 pad 5: /IO-Decoder/IO_SigDecoder/IOCHCK -> /IO-Decoder/IO_SigDecoder/IOCHCK_I
- U6 pad 23: /FDC-Serial/A0 -> /DMA/A0
- U6 pad 24: /FDC-Serial/A1 -> /DMA/A1
- U6 pad 25: /FDC-Serial/A2 -> /DMA/A2
- U6 pad 26: /FDC-Serial/A3 -> /DMA/A3
- U6 pad 27: /FDC-Serial/A4 -> /DMA/A4
- U6 pad 28: /FDC-Serial/A5 -> /DMA/A5
- U6 pad 29: /FDC-Serial/A6 -> /DMA/A6
- U6 pad 30: /FDC-Serial/A7 -> /DMA/A7
- U6 pad 31: /FDC-Serial/A8 -> /DMA/A8
- U6 pad 32: /FDC-Serial/A9 -> /DMA/A9
- U6 pad 33: /FDC-Serial/A10 -> /DMA/A10
- U6 pad 34: /FDC-Serial/A11 -> /DMA/A11
- U6 pad 35: /FDC-Serial/A12 -> /DMA/A12
- U6 pad 36: /FDC-Serial/A13 -> /DMA/A13
- U6 pad 37: /FDC-Serial/A14 -> /DMA/A14
- U6 pad 38: /FDC-Serial/A15 -> /DMA/A15
- U6 pad 53: /FDC-Serial/RESET_DRV -> /RESET
- U7 pad 11: /HDD Controller/D5 -> /FDC-Serial/D5
- U7 pad 12: /HDD Controller/D6 -> /FDC-Serial/D6
- U7 pad 13: /HDD Controller/D7 -> /FDC-Serial/D7
- U7 pad 15: /DACK3 -> /~DACK3
- U7 pad 2: /HDD Controller/D0 -> /FDC-Serial/D0
- U7 pad 27: /FDC-Serial/A1 -> /DMA/A1
- U7 pad 28: /FDC-Serial/A0 -> /DMA/A0
- U7 pad 3: /HDD Controller/D1 -> /FDC-Serial/D1
- U7 pad 4: /HDD Controller/D2 -> /FDC-Serial/D2
- U7 pad 5: /HDD Controller/D3 -> /FDC-Serial/D3
- U7 pad 6: /HDD Controller/D4 -> /FDC-Serial/D4
Routing:
- net /DMA/A18: track 0.00 -> 611.9 mm, vias 0 -> 12
- net /DMA/A19: track 0.00 -> 592.0 mm, vias 0 -> 8
- net /DMA/A8: track 0.00 -> 591.6 mm, vias 0 -> 10
- net /DMA/A9: track 0.00 -> 590.3 mm, vias 0 -> 6
- net /DMA/A13: track 0.00 -> 582.7 mm, vias 0 -> 18
- net /DMA/A17: track 0.00 -> 559.9 mm, vias 0 -> 8
- net /DMA/A14: track 0.00 -> 545.7 mm, vias 0 -> 9
- net /DMA/A15: track 0.00 -> 536.7 mm, vias 0 -> 9
- net /DMA/A16: track 0.00 -> 532.0 mm, vias 0 -> 6
- net /DMA/A0: track 0.00 -> 528.4 mm, vias 0 -> 13
- net /DMA/A4: track 0.00 -> 502.0 mm, vias 0 -> 12
- net /DMA/A7: track 0.00 -> 488.9 mm, vias 0 -> 12
- net /~DACK2: track 0.00 -> 484.1 mm, vias 0 -> 14
- net /DMA/A11: track 0.00 -> 479.1 mm, vias 0 -> 9
- net /DMA/A1: track 0.00 -> 470.2 mm, vias 0 -> 17
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
Commit message: Large Sync
Parts:
- added G***: LOGO, UC:UC, F.Cu at (76.0, 54.3)
- added REF**: MountingHole_3.2mm_M3, MountingHole:MountingHole_3.2mm_M3, F.Cu at (225.3, 28.9)
- added REF**: MountingHole_3.2mm_M3, MountingHole:MountingHole_3.2mm_M3, F.Cu at (164.1, 187.7)
- added REF**: MountingHole_3.2mm_M3, MountingHole:MountingHole_3.2mm_M3, F.Cu at (77.4, 69.9)
- added REF**: MountingHole_3.2mm_M3, MountingHole:MountingHole_3.2mm_M3, F.Cu at (178.1, 27.1)
- added REF**: MountingHole_3.2mm_M3, MountingHole:MountingHole_3.2mm_M3, F.Cu at (129.2, 27.1)
- added REF**: MountingHole_3.2mm_M3, MountingHole:MountingHole_3.2mm_M3, F.Cu at (172.5, 115.3)
- added REF**: MountingHole_3.2mm_M3, MountingHole:MountingHole_3.2mm_M3, F.Cu at (224.1, 197.5)
- added REF**: MountingHole_3.2mm_M3, MountingHole:MountingHole_3.2mm_M3, F.Cu at (65.6, 234.6)
- added REF**: MountingHole_3.2mm_M3, MountingHole:MountingHole_3.2mm_M3, F.Cu at (23.8, 151.2)
