File: Motherboard/ISA.sch (KiCad schematic (older format))
At the start: 5 parts, among them J2 Bus_ISA_8bit, J3 Bus_ISA_8bit, J5 Bus_ISA_8bit, J6 Bus_ISA_8bit, J7 Bus_ISA_8bit

Commit message: Large sync
Parts:
- added C5, C6, C7, C8, C9: 1u, Capacitors_THT:CP_Radial_D4.0mm_P2.00mm, symbol Device:CP
Connections:
- net +5V: now also C5.1, C6.1, C7.1, C8.1, C9.1
- net AEN: now also J2.42 (AEN), J3.42 (AEN), J5.42 (AEN), J6.42 (AEN), J7.42 (AEN)
- net ALE: now also J2.28 (ALE), J3.28 (ALE), J5.28 (ALE), J6.28 (ALE), J7.28 (ALE)
- net CLK: now also J2.20 (CLK), J3.20 (CLK), J5.20 (CLK), J6.20 (CLK), J7.20 (CLK)
- net GND: now also C5.2, C6.2, C7.2, C8.2, C9.2
- net OSC: now also J2.30 (OSC), J3.30 (OSC), J5.30 (OSC), J6.30 (OSC), J7.30 (OSC)
- net TC: now also J2.27 (TC), J3.27 (TC), J5.27 (TC), J6.27 (TC), J7.27 (TC)
- net ~IOW: now also J2.13 (~IOW), J3.13 (~IOW), J5.13 (~IOW), J6.13 (~IOW), J7.13 (~IOW)
- net D7: now reaches J2.33 (DB7)
- net D7: now also J3.33 (DB7), J5.33 (DB7), J6.33 (DB7), J7.33 (DB7)
- net D6: now reaches J2.34 (DB6)
- net D6: now also J3.34 (DB6), J5.34 (DB6), J6.34 (DB6), J7.34 (DB6)
- net D5: now reaches J2.35 (DB5)
- net D5: now also J3.35 (DB5), J5.35 (DB5), J6.35 (DB5), J7.35 (DB5)
- net D4: now reaches J2.36 (DB4)
- net D4: now also J3.36 (DB4), J5.36 (DB4), J6.36 (DB4), J7.36 (DB4)
- net D3: now reaches J2.37 (DB3)
- net D3: now also J3.37 (DB3), J5.37 (DB3), J6.37 (DB3), J7.37 (DB3)
- net D2: now reaches J2.38 (DB2)
- net D2: now also J3.38 (DB2), J5.38 (DB2), J6.38 (DB2), J7.38 (DB2)
- net D1: now reaches J2.39 (DB1)
- net D1: now also J3.39 (DB1), J5.39 (DB1), J6.39 (DB1), J7.39 (DB1)
- net D0: now reaches J2.40 (DB0)
- net D0: now also J3.40 (DB0), J5.40 (DB0), J6.40 (DB0), J7.40 (DB0)
- net A19: now reaches J2.43 (BA19)
- net A19: now also J3.43 (BA19), J5.43 (BA19), J6.43 (BA19), J7.43 (BA19)
- net A18: now reaches J2.44 (BA18)
- net A18: now also J3.44 (BA18), J5.44 (BA18), J6.44 (BA18), J7.44 (BA18)
- net A17: now reaches J2.45 (BA17)
- net A17: now also J3.45 (BA17), J5.45 (BA17), J6.45 (BA17), J7.45 (BA17)
- net A16: now reaches J2.46 (BA16)
- net A16: now also J3.46 (BA16), J5.46 (BA16), J6.46 (BA16), J7.46 (BA16)
- net A15: now reaches J2.47 (BA15)
- net A15: now also J3.47 (BA15), J5.47 (BA15), J6.47 (BA15), J7.47 (BA15)
- net A14: now reaches J2.48 (BA14)
- net A14: now also J3.48 (BA14), J5.48 (BA14), J6.48 (BA14), J7.48 (BA14)
- net A13: now reaches J2.49 (BA13)
- net A13: now also J3.49 (BA13), J5.49 (BA13), J6.49 (BA13), J7.49 (BA13)
- net A12: now reaches J2.50 (BA12)
- net A12: now also J3.50 (BA12), J5.50 (BA12), J6.50 (BA12), J7.50 (BA12)
- net A11: now reaches J2.51 (BA11)
- net A11: now also J3.51 (BA11), J5.51 (BA11), J6.51 (BA11), J7.51 (BA11)
- net A10: now reaches J2.52 (BA10)
- net A10: now also J3.52 (BA10), J5.52 (BA10), J6.52 (BA10), J7.52 (BA10)
- net A9: now reaches J2.53 (BA09)
- net A9: now also J3.53 (BA09), J5.53 (BA09), J6.53 (BA09), J7.53 (BA09)
- net A8: now reaches J2.54 (BA08)
- net A8: now also J3.54 (BA08), J5.54 (BA08), J6.54 (BA08), J7.54 (BA08)
- net A7: now reaches J2.55 (BA07)
- net A7: now also J3.55 (BA07), J5.55 (BA07), J6.55 (BA07), J7.55 (BA07)
- net A6: now reaches J2.56 (BA06)
- net A6: now also J3.56 (BA06), J5.56 (BA06), J6.56 (BA06), J7.56 (BA06)
- net A5: now reaches J2.57 (BA05)
- net A5: now also J3.57 (BA05), J5.57 (BA05), J6.57 (BA05), J7.57 (BA05)
- net A4: now reaches J2.58 (BA04)
- net A4: now also J3.58 (BA04), J5.58 (BA04), J6.58 (BA04), J7.58 (BA04)
- net A3: now reaches J2.59 (BA03)
- net A3: now also J3.59 (BA03), J5.59 (BA03), J6.59 (BA03), J7.59 (BA03)
- net A2: now reaches J2.60 (BA02)
- net A2: now also J3.60 (BA02), J5.60 (BA02), J6.60 (BA02), J7.60 (BA02)
- net A1: now reaches J2.61 (BA01)
- net A1: now also J3.61 (BA01), J5.61 (BA01), J6.61 (BA01), J7.61 (BA01)
- net A0: now reaches J2.62 (BA00)
- net A0: now also J3.62 (BA00), J5.62 (BA00), J6.62 (BA00), J7.62 (BA00)
- no-connect marks 5 -> 3
