File: Motherboard/ISA.sch (KiCad schematic (older format))
At the start: 10 parts, among them J2 Bus_ISA_8bit, J3 Bus_ISA_8bit, J5 Bus_ISA_8bit, J6 Bus_ISA_8bit, J7 Bus_ISA_8bit

Commit message: LARGE sync
Parts:
- removed J5, J7: Bus_ISA_8bit, RetPC:ISA-8-bit, symbol Motherboard-rescue:Bus_ISA_8bit-Connector
- added J5, J7: Bus_ISA_8bit, RetPC:ISA-8-bit, symbol Connector:Bus_ISA_8bit
- added R20: R_Small, Resistor_THT:R_Axial_DIN0204_L3.6mm_D1.6mm_P5.08mm_Vertical, symbol Device:R_Small
Connections:
- net +12V: now also J5.9 (+12V), J7.9 (+12V)
- net +5V: now also J5.29 (VCC), J5.3 (VCC), J7.29 (VCC), J7.3 (VCC), R20.1
- net -12V: now also J5.7 (-12V), J7.7 (-12V)
- net -5V: now also J5.5 (-5V), J7.5 (-5V)
- net A0: now also J5.62 (BA00), J7.62 (BA00)
- net A1: now also J5.61 (BA01), J7.61 (BA01)
- net A10: now also J5.52 (BA10), J7.52 (BA10)
- net A11: now also J5.51 (BA11), J7.51 (BA11)
- net A12: now also J5.50 (BA12), J7.50 (BA12)
- net A13: now also J5.49 (BA13), J7.49 (BA13)
- net A14: now also J5.48 (BA14), J7.48 (BA14)
- net A15: now also J5.47 (BA15), J7.47 (BA15)
- net A16: now also J5.46 (BA16), J7.46 (BA16)
- net A17: now also J5.45 (BA17), J7.45 (BA17)
- net A18: now also J5.44 (BA18), J7.44 (BA18)
- net A19: now also J5.43 (BA19), J7.43 (BA19)
- net A2: now also J5.60 (BA02), J7.60 (BA02)
- net A3: now also J5.59 (BA03), J7.59 (BA03)
- net A4: now also J5.58 (BA04), J7.58 (BA04)
- net A5: now also J5.57 (BA05), J7.57 (BA05)
- net A6: now also J5.56 (BA06), J7.56 (BA06)
- net A7: now also J5.55 (BA07), J7.55 (BA07)
- net A8: now also J5.54 (BA08), J7.54 (BA08)
- net A9: now also J5.53 (BA09), J7.53 (BA09)
- net AEN: now also J5.42 (AEN), J7.42 (AEN)
- net ALE: now also J5.28 (ALE), J7.28 (ALE)
- net CLK: now also J5.20 (CLK), J7.20 (CLK)
- net D0: now also J5.40 (DB0), J7.40 (DB0)
- net D1: now also J5.39 (DB1), J7.39 (DB1)
- net D2: now also J5.38 (DB2), J7.38 (DB2)
- net D3: now also J5.37 (DB3), J7.37 (DB3)
- net D4: now also J5.36 (DB4), J7.36 (DB4)
- net D5: now also J5.35 (DB5), J7.35 (DB5)
- net D6: now also J5.34 (DB6), J7.34 (DB6)
- net D7: now also J5.33 (DB7), J7.33 (DB7)
- net GND: now also J5.1 (GND), J5.10 (GND), J5.31 (GND), J7.1 (GND), J7.10 (GND), J7.31 (GND)
- net IO_READY: now also J2.41 (IO_READY), J3.41 (IO_READY), J6.41 (IO_READY), J5.41 (IO_READY), J7.41 (IO_READY), R20.2
- net OSC: now also J5.30 (OSC), J7.30 (OSC)
- net RESET: now also J5.2 (RESET), J7.2 (RESET)
- net TC: now also J5.27 (TC), J7.27 (TC)
- net ~IOW: now also J5.13 (~IOW), J7.13 (~IOW)
- net ~MEMW: now reaches J2.11 (~SMEMW)
- net ~MEMW: now also J3.11 (~SMEMW), J6.11 (~SMEMW), J5.11 (~SMEMW), J7.11 (~SMEMW)
- net ~MEMR: now reaches J2.12 (~SMEMR)
- net ~MEMR: now also J3.12 (~SMEMR), J6.12 (~SMEMR), J5.12 (~SMEMR), J7.12 (~SMEMR)
- net ~IOR: now reaches J2.14 (~IOR)
- net ~IOR: now also J3.14 (~IOR), J6.14 (~IOR), J5.14 (~IOR), J7.14 (~IOR)
- net ~DACK3: now reaches J2.15 (~DACK3)
- net ~DACK3: now also J3.15 (~DACK3), J6.15 (~DACK3), J5.15 (~DACK3), J7.15 (~DACK3)
- net DRQ3: now reaches J2.16 (DRQ3)
- net DRQ3: now also J3.16 (DRQ3), J6.16 (DRQ3), J5.16 (DRQ3), J7.16 (DRQ3)
- net ~DACK1: now reaches J2.17 (~DACK1)
- net ~DACK1: now also J3.17 (~DACK1), J6.17 (~DACK1), J5.17 (~DACK1), J7.17 (~DACK1)
- net DRQ1: now reaches J2.18 (DRQ1)
- net DRQ1: now also J3.18 (DRQ1), J6.18 (DRQ1), J5.18 (DRQ1), J7.18 (DRQ1)
- net ~DACK0: now reaches J2.19 (~DACK0)
- net ~DACK0: now also J3.19 (~DACK0), J6.19 (~DACK0), J5.19 (~DACK0), J7.19 (~DACK0)
- net IRQ7: now reaches J2.21 (IRQ7)
- net IRQ7: now also J3.21 (IRQ7), J6.21 (IRQ7), J5.21 (IRQ7), J7.21 (IRQ7)
- net IRQ6: now reaches J2.22 (IRQ6)
- net IRQ6: now also J3.22 (IRQ6), J6.22 (IRQ6), J5.22 (IRQ6), J7.22 (IRQ6)
- net IRQ5: now reaches J2.23 (IRQ5)
- net IRQ5: now also J3.23 (IRQ5), J6.23 (IRQ5), J5.23 (IRQ5), J7.23 (IRQ5)
- net IRQ4: now reaches J2.24 (IRQ4)
- net IRQ4: now also J3.24 (IRQ4), J6.24 (IRQ4), J5.24 (IRQ4), J7.24 (IRQ4)
- net IRQ3: now reaches J2.25 (IRQ3)
- net IRQ3: now also J3.25 (IRQ3), J6.25 (IRQ3), J5.25 (IRQ3), J7.25 (IRQ3)
- net ~DACK2: now reaches J2.26 (~DACK2)
- net ~DACK2: now also J3.26 (~DACK2), J6.26 (~DACK2), J5.26 (~DACK2), J7.26 (~DACK2)
- net IOCHCK: now reaches J2.32 (IO)
- net IRQ2: now reaches J2.4 (INQ2)
- net IRQ2: now also J3.4 (INQ2)
- net DRQ2: now reaches J2.6 (DRQ2)
- net DRQ2: now also J3.6 (DRQ2)
- no-connect marks 3 -> 5

Commit message: A LOT of work
Connections:
- net IOCHCK: now also J3.32 (IO), J5.32 (IO), J6.32 (IO), J7.32 (IO)
Changed lines of the file:
@@
 EESchema Schematic File Version 4
 LIBS:Motherboard-cache
-EELAYER 29 0
+EELAYER 30 0
 EELAYER END
 $Descr A3 16535 11693
@@
 Text HLabel 11555 1335 0    50   Input ~ 0
 OSC
-Text HLabel 11555 1410 0    50   Input ~ 0
-DRQ[0...3]
-Text HLabel 11555 1485 0    50   Input ~ 0
-~DACK~[0...3]
 Text HLabel 11555 1560 0    50   Input ~ 0
 CLK
 Text HLabel 11555 1635 0    50   Input ~ 0
 ~IOW
-Text HLabel 11555 1710 0    50   Input ~ 0
+Text HLabel 10080 2170 0    50   Input ~ 0
 IRQ[2...7]
 Text HLabel 11555 1785 0    50   Input ~ 0
@@
 Text HLabel 11555 1860 0    50   Input ~ 0
 ALE
-Text HLabel 11555 1935 0    50   Input ~ 0
+Text HLabel 10120 1090 0    50   Input ~ 0
 IOCHCK
 Text HLabel 11555 2010 0    50   Input ~ 0
@@
 Text HLabel 11555 2235 0    50   Input ~ 0
 AEN
-Text HLabel 11555 2310 0    50   Input ~ 0
+Text HLabel 11550 2320 0    50   Input ~ 0
 ~MEMW
-Text HLabel 11555 2385 0    50   Input ~ 0
+Text HLabel 11550 2410 0    50   Input ~ 0
 ~MEMR
 $Comp
@@
 NoConn ~ 2325 7075
 NoConn ~ 4900 7075
+Text HLabel 10100 1250 0    50   Output ~ 0
+DRQ0
+Text HLabel 10100 1330 0    50   Output ~ 0
+DRQ1
+Text HLabel 10100 1410 0    50   Output ~ 0
+DRQ2
+Text HLabel 10100 1490 0    50   Output ~ 0
+DRQ3
+Text HLabel 10100 1610 0    50   Input ~ 0
+~DACK0
+Text HLabel 10100 1700 0    50   Input ~ 0
+~DACK1
+Text HLabel 10100 1790 0    50   Input ~ 0
+~DACK2
+Text HLabel 10100 1880 0    50   Input ~ 0
+~DACK3
+Wire Wire Line
+	10100 1250 10300 1250
+Wire Wire Line
+	10100 1330 10300 1330
+Wire Wire Line
+	10100 1410 10300 1410
+Wire Wire Line
+	10100 1490 10300 1490
+Text Label 10300 1250 2    50   ~ 0
+DRQ0
+Text Label 10300 1330 2    50   ~ 0
+DRQ1
+Text Label 10300 1410 2    50   ~ 0
+DRQ2
+Text Label 10300 1490 2    50   ~ 0
+DRQ3
+Text Label 10350 1610 2    50   ~ 0
+~DACK0
+Wire Wire Line
+	10100 1610 10350 1610
+Wire Wire Line
+	10100 1700 10350 1700
+Wire Wire Line
+	10100 1790 10350 1790
+Wire Wire Line
+	10100 1880 10350 1880
+Text Label 10350 1700 2    50   ~ 0
+~DACK1
+Text Label 10350 1790 2    50   ~ 0
+~DACK2
+Text Label 10350 1880 2    50   ~ 0
+~DACK3
+Wire Wire Line
+	11550 2320 11800 2320
+Wire Wire Line
+	11550 2410 11800 2410
+Text Label 11800 2320 2    50   ~ 0
+~MEMW
+Text Label 11800 2410 2    50   ~ 0
+~MEMR
+Wire Wire Line
+	10120 1090 10430 1090
+Text Label 10430 1090 2    50   ~ 0
+IOCHCK
+Wire Bus Line
+	10080 2170 10200 2170
+Entry Wire Line
+	10200 2170 10300 2270
+Entry Wire Line
+	10200 2240 10300 2340
+Text Label 10470 2270 2    50   ~ 0
+IRQ2
+Wire Wire Line
+	10300 2270 10470 2270
+Wire Wire Line
+	10300 2340 10470 2340
+Text Label 10470 2340 2    50   ~ 0
+IRQ3
+Entry Wire Line
+	10200 2310 10300 2410
+Entry Wire Line
+	10200 2380 10300 2480
+Text Label 10470 2480 2    50   ~ 0
+IRQ5
+Wire Wire Line
+	10300 2480 10470 2480
+Wire Wire Line
+	10300 2410 10470 2410
+Text Label 10470 2410 2    50   ~ 0
+IRQ4
+Entry Wire Line
+	10200 2450 10300 2550
+Entry Wire Line
+	10200 2520 10300 2620
+Text Label 10470 2620 2    50   ~ 0
+IRQ7
+Wire Wire Line
+	10300 2620 10470 2620
+Wire Wire Line
+	10300 2550 10470 2550
+Text Label 10470 2550 2    50   ~ 0
+IRQ6
+Text Label 6600 1900 2    50   ~ 0
+IOCHCK
+Wire Wire Line
+	6325 1900 6600 1900
+Text Label 4000 6375 2    50   ~ 0
+IOCHCK
+Wire Wire Line
+	3725 6375 4000 6375
+Text Label 6575 6375 2    50   ~ 0
+IOCHCK
+Wire Wire Line
+	6300 6375 6575 6375
+Text Label 8975 6375 2    50   ~ 0
+IOCHCK
+Wire Wire Line
+	8700 6375 8975 6375
+Wire Bus Line
+	10200 2170 10200 2520
 Wire Bus Line
 	4050 6375 4050 7275

Commit message: Large Sync
Parts:
- added U53: 74LS175, Package_DIP:DIP-14_W7.62mm_Socket, symbol 74xx:74LS175
- added U54: 74LS244, Package_DIP:DIP-14_W7.62mm_Socket, symbol 74xx:74LS244
- added U?: 74LS74, symbol 74xx:74LS74
- C5, C6, C7, C8, C9: symbol Device:CP -> Motherboard-rescue:CP-Device
- J5, J7: symbol Connector:Bus_ISA_8bit -> Motherboard-rescue:Bus_ISA_8bit-Connector
- R20: symbol Device:R_Small -> Motherboard-rescue:R_Small-Device
Connections:
- net +5V: now also U?.2 (D), U?.3 (C)
- net D0: now also U53.4 (D0), U54.3 (O3b)
- net D1: now also U53.5 (D1), U54.5 (O2b)
- net D2: now also U53.12 (D2), U54.7 (O1b)
- net D3: now also U53.13 (D3), U54.9 (O0b)
- net D4: now also U54.12 (O3a)
- net D5: now also U54.14 (O2a)
- net D6: now also U54.16 (O1a)
- net D7: now also U54.18 (O0a)
- net IOCHCK: now also U?.4 (~S)
- new net: U53.15 (Q3), U54.11 (I0b)
- new net: U53.10 (Q2), U54.13 (I1b)
- new net: U54.4 (I1a), U?.5 (Q)
- new net ENA_IOCHCK: U53.14 (~Q3), U?.1 (~R)
- new net PORTB_RD: U54.1 (OEa), U54.19 (OEb)
- new net SPKR_DATA: U53.7 (Q1), U54.15 (I2b)
- new net TIM2GATE: U53.2 (Q0), U54.17 (I3b)
- new net ~RESET: U53.1 (~Mr)
- no-connect marks 5 -> 8
Other:
- note added: "Mot NMI\n"
