File: Motherboard/DMA.sch (KiCad schematic (older format))
At the start: 7 parts, among them U22 74HC74, U23 8237, U24 74LS04, U25 74LS573, U26 74LS573, U27 74LS670

Commit message: A VERY large sync...
Changed lines of the file:
@@
 $Descr A4 11693 8268
 encoding utf-8
-Sheet 4 5
+Sheet 4 8
 Title ""
 Date ""
@@
 ADDR
 Text Label 2150 1075 2    50   ~ 0
-ADDR[A0...19]
-Text HLabel 1375 1200 0    50   BiDi ~ 0
-DATA
-Wire Bus Line
-	1375 1200 2150 1200
-Text Label 2150 1200 2    50   ~ 0
-DATA[D0...7]
+A[0...19]
 Entry Wire Line
 	2525 3775 2625 3875
@@
 	2600 2275 2675 2275
 Text Label 2500 1625 0    50   ~ 0
-ADDR[A0...3]
+A[0...3]
 Entry Wire Line
 	4125 1975 4225 2075
@@
 	4075 2275 4125 2275
 Text Label 4225 1650 2    50   ~ 0
-ADDR[A4...7]
+A[4...7]
 Wire Wire Line
 	3375 1675 3425 1675

Commit message: LARGE sync
Parts:
- removed U22: 74HC74, Housings_DIP:DIP-14_W7.62mm_Socket, symbol 74xx:74HC74
- removed unit 1 of U24
- R5: value R -> 1k
- U24: footprint Housings_DIP:DIP-20_W7.62mm_Socket -> Package_DIP:DIP-14_W7.62mm_Socket
- U25: value 74LS573 -> 74LS244; symbol 74xx:74LS573 -> 74xx:74LS244
- U26: value 74LS573 -> 74LS373; symbol 74xx:74LS573 -> 74xx:74LS373
Connections:
- net A0: now also U25.3 (O3b); no longer U27.14 (Wa)
- net A1: now also U25.5 (O2b); no longer U27.13 (Wb)
- net CLK: now also U23.12 (CLK)
- net XD7: now reaches U23.21 (DB7)
- net XD7: now also U26.3 (D0)
- net XD6: now reaches U23.22 (DB6)
- net XD6: now also U26.4 (D1)
- net XD5: now reaches U23.23 (DB5)
- net XD5: now also U26.7 (D2)
- net XD4: now reaches U23.26 (DB4)
- net XD4: now also U26.8 (D3)
- net XD3: now reaches U23.27 (DB3)
- net XD3: now also U26.13 (D4), U27.3 (D4)
- net XD2: now reaches U23.28 (DB2)
- net XD2: now also U26.14 (D5), U27.2 (D3)
- net XD1: now reaches U23.29 (DB1)
- net XD1: now also U26.17 (D6), U27.1 (D2)
- net ~XMEMR: now reaches U23.3 (~MEMR~)
- net XD0: now reaches U23.30 (DB0)
- net XD0: now also U26.18 (D7), U27.15 (D1)
- net XA0: now reaches U23.32 (A0)
- net XA0: now also U25.17 (I3b), U27.14 (Wa)
- net XA1: now reaches U23.33 (A1)
- net XA1: now also U25.15 (I2b), U27.13 (Wb)
- net XA2: now reaches U23.34 (A2)
- net XA2: now also U25.13 (I1b)
- net XA3: now reaches U23.35 (A3)
- net XA3: now also U25.11 (I0b)
- net XA4: now reaches U23.37 (A4)
- net XA4: now also U25.8 (I3a)
- net XA5: now reaches U23.38 (A5)
- net XA5: now also U25.6 (I2a)
- net XA6: now reaches U23.39 (A6)
- net XA6: now also U25.4 (I1a)
- net ~XMEMW: now reaches U23.4 (~MEMW~)
- net XA7: now reaches U23.40 (A7)
- net XA7: now also U25.2 (I0a)
- net at U23.8 (ADSTB), U26.11 (LE): no longer U25.11 (Load)
- net ~DMAEN: now reaches U25.1 (OEa), U26.1 (OE), U27.11 (~Er)
- net ~DMAEN: now also U25.19 (OEb)
- net A4: now reaches U25.12 (O3a)
- net A5: now reaches U25.14 (O2a)
- net A6: now reaches U25.16 (O1a)
- net A7: now reaches U25.18 (O0a)
- net A2: now reaches U25.7 (O1b)
- net A3: now reaches U25.9 (O0b)
- net A11: now reaches U26.12 (O4)
- net A10: now reaches U26.15 (O5)
- net A9: now reaches U26.16 (O6)
- net A8: now reaches U26.19 (O7)
- net A15: now reaches U26.2 (O0)
- net A14: now reaches U26.5 (O1)
- net A13: now reaches U26.6 (O2)
- net A12: now reaches U26.9 (O3)
- net A16: now reaches U27.10 (Q1)
- net A19: now reaches U27.6 (Q4)
- net A18: now reaches U27.7 (Q3)
- net A17: now reaches U27.9 (Q2)
- net BUSEN: no longer names the net of U23.9 (AEN)
- net ~IOR renamed ~XIOR
- net ~IOW renamed ~XIOW
- no-connect marks 0 -> 1
