File: Motherboard/DMA.sch (KiCad schematic (older format))
At the start: 6 parts, among them U23 8237, U24 74LS04, U25 74LS244, U26 74LS373, U27 74LS670

Commit message: A LOT of work
Connections:
- net +5V: now also U27.16 (VCC)
- net GND: now also U27.8 (GND)
Changed lines of the file:
@@
 EESchema Schematic File Version 4
 LIBS:Motherboard-cache
-EELAYER 29 0
+EELAYER 30 0
 EELAYER END
 $Descr A4 11693 8268
@@
 Wire Bus Line
 	8425 5950 9675 5950
+$Comp
+L power:GND #PWR?
+U 1 1 5D4B52C2
+P 8700 3350
+F 0 "#PWR?" H 8700 3100 50  0001 C CNN
+F 1 "GND" H 8705 3177 50  0000 C CNN
+F 2 "" H 8700 3350 50  0001 C CNN
+F 3 "" H 8700 3350 50  0001 C CNN
+	1    8700 3350
+	1    0    0    -1
+$EndComp
+$Comp
+L power:+5V #PWR?
+U 1 1 5D4B569A
+P 8700 1650
+F 0 "#PWR?" H 8700 1500 50  0001 C CNN
+F 1 "+5V" V 8715 1778 50  0000 L CNN
+F 2 "" H 8700 1650 50  0001 C CNN
+F 3 "" H 8700 1650 50  0001 C CNN
+	1    8700 1650
+	0    1    1    0
+$EndComp
 $EndSCHEMATC

Commit message: Large Sync
Parts:
- R5: symbol Device:R -> Motherboard-rescue:R-Device
- U23: symbol Interface:8237 -> Motherboard-rescue:8237-Interface
- U24: symbol 74xx:74LS04 -> Motherboard-rescue:74LS04-74xx
- U25: symbol 74xx:74LS244 -> Motherboard-rescue:74LS244-74xx
- U26: symbol 74xx:74LS373 -> Motherboard-rescue:74LS373-74xx
- U27: symbol 74xx:74LS670 -> Motherboard-rescue:74LS670-74xx
Changed lines of the file:
@@
 $EndDescr
 $Comp
-L Interface:8237 U23
+L Motherboard-rescue:8237-Interface U23
 U 1 1 5C10FC71
 P 3375 3275
@@
 $EndComp
 $Comp
-L 74xx:74LS244 U25
+L Motherboard-rescue:74LS244-74xx U25
 U 1 1 5C11001A
 P 5500 5300
@@
 $EndComp
 $Comp
-L power:GND #PWR033
+L Motherboard-rescue:GND-power #PWR033
 U 1 1 5C1104E2
 P 3375 4875
@@
 $EndComp
 $Comp
-L power:GND #PWR035
+L Motherboard-rescue:GND-power #PWR035
 U 1 1 5C110528
 P 4700 5300
@@
 $EndComp
 $Comp
-L power:+5V #PWR037
+L Motherboard-rescue:+5V-power #PWR037
 U 1 1 5C11055D
 P 6300 5300
@@
 $EndComp
 $Comp
-L power:+5V #PWR034
+L Motherboard-rescue:+5V-power #PWR034
 U 1 1 5C1105CA
 P 3425 1675
@@
 Connection ~ 3425 1675
 $Comp
-L Device:R R5
+L Motherboard-rescue:R-Device R5
 U 1 1 5C121A87
 P 5350 3200
@@
 	5350 3375 5350 3350
 $Comp
-L power:+5V #PWR036
+L Motherboard-rescue:+5V-power #PWR036
 U 1 1 5C122765
 P 5350 3050
@@
 $EndComp
 $Comp
-L 74xx:74LS04 U24
+L Motherboard-rescue:74LS04-74xx U24
 U 2 1 5C122876
 P 5800 3375
@@
 TC
 $Comp
-L 74xx:74LS373 U26
+L Motherboard-rescue:74LS373-74xx U26
 U 1 1 5C123B44
 P 8525 5300
@@
 $EndComp
 $Comp
-L power:GND #PWR038
+L Motherboard-rescue:GND-power #PWR038
 U 1 1 5C123B4A
 P 7725 5300
@@
 $EndComp
 $Comp
-L power:+5V #PWR039
+L Motherboard-rescue:+5V-power #PWR039
 U 1 1 5C123B50
 P 9325 5300
@@
 	8025 4400 8025 4800
 $Comp
-L 74xx:74LS670 U27
+L Motherboard-rescue:74LS670-74xx U27
 U 1 1 5C12C9DA
 P 8700 2450
@@
 XD7
 $Comp
-L power:GND #PWR?
+L Motherboard-rescue:GND-power #PWR098
 U 1 1 5D4B52C2
 P 8700 3350
-F 0 "#PWR?" H 8700 3100 50  0001 C CNN
+F 0 "#PWR098" H 8700 3100 50  0001 C CNN
 F 1 "GND" H 8705 3177 50  0000 C CNN
 F 2 "" H 8700 3350 50  0001 C CNN
@@
 $EndComp
 $Comp
-L power:+5V #PWR?
+L Motherboard-rescue:+5V-power #PWR097
 U 1 1 5D4B569A
 P 8700 1650
-F 0 "#PWR?" H 8700 1500 50  0001 C CNN
+F 0 "#PWR097" H 8700 1500 50  0001 C CNN
 F 1 "+5V" V 8715 1778 50  0000 L CNN
 F 2 "" H 8700 1650 50  0001 C CNN
