File: Motherboard/DivClock.sch (KiCad schematic (older format))
At the start: 15 parts, among them SW1 TURBO, SW2 FREEZE, U15 74LS257, U5 ATF750LVC, U9 40106, Y1 14.31818 MHz, Y2 24.000 MHz

Commit message: Large Sync
Parts:
- C1, C2, C3, C4: symbol Device:C -> Motherboard-rescue:C-Device
- R1, R2, R3, R4: symbol Device:R -> Motherboard-rescue:R-Device
- SW1, SW2: symbol Switch:SW_SPST -> Motherboard-rescue:SW_SPST-Switch
- U15: symbol 74xx:74LS257 -> Motherboard-rescue:74LS257-74xx
- U9: symbol 4xxx_IEEE:40106 -> Motherboard-rescue:40106-4xxx_IEEE
- Y1, Y2: symbol Device:Crystal -> Motherboard-rescue:Crystal-Device
Connections:
- net +5V: now also SW2.2 (B); no longer R4.1
- net GND: now also R4.1; no longer SW2.2 (B)
- no-connect marks 9 -> 16
Changed lines of the file:
@@
 $EndDescr
 $Comp
-L Device:Crystal Y1
+L Motherboard-rescue:Crystal-Device Y1
 U 1 1 5BFC00B2
 P 2375 2225
@@
 $EndComp
 $Comp
-L 4xxx_IEEE:40106 U9
+L Motherboard-rescue:40106-4xxx_IEEE U9
 U 1 1 5BFC0147
 P 2400 1450
+AR Path="/5BFC0147" Ref="U9"  Part="1"
+AR Path="/5C104845/5BFC0147" Ref="U9"  Part="1"
 F 0 "U9" H 2575 1575 50  0000 L CNN
 F 1 "40106" H 2575 1325 50  0000 L CNN
@@
 $EndComp
 $Comp
-L Device:R R1
+L Motherboard-rescue:R-Device R1
 U 1 1 5BFC026F
 P 2400 975
@@
 $EndComp
 $Comp
-L Device:C C3
+L Motherboard-rescue:C-Device C3
 U 1 1 5BFC036F
 P 2900 2400
@@
 $EndComp
 $Comp
-L power:GND #PWR016
+L Motherboard-rescue:GND-power #PWR016
 U 1 1 5BFC03E5
 P 2900 2550
@@
 $EndComp
 $Comp
-L Device:Crystal Y2
+L Motherboard-rescue:Crystal-Device Y2
 U 1 1 5BFC2C74
 P 2375 4475
@@
 $EndComp
 $Comp
-L 4xxx_IEEE:40106 U9
+L Motherboard-rescue:40106-4xxx_IEEE U9
 U 3 1 5BFC2C7A
 P 2400 3700
+AR Path="/5BFC2C7A" Ref="U9"  Part="3"
+AR Path="/5C104845/5BFC2C7A" Ref="U9"  Part="3"
 F 0 "U9" H 2500 3850 50  0000 L CNN
 F 1 "40106" H 2450 3550 50  0000 L CNN
@@
 $EndComp
 $Comp
-L Device:R R2
+L Motherboard-rescue:R-Device R2
 U 1 1 5BFC2C80
 P 2400 3225
@@
 $EndComp
 $Comp
-L 4xxx_IEEE:40106 U9
+L Motherboard-rescue:40106-4xxx_IEEE U9
 U 4 1 5BFC2C9E
 P 3475 3700
+AR Path="/5BFC2C9E" Ref="U9"  Part="4"
+AR Path="/5C104845/5BFC2C9E" Ref="U9"  Part="4"
 F 0 "U9" H 3575 3850 50  0000 L CNN
 F 1 "40106" H 3525 3550 50  0000 L CNN
@@
 $EndComp
 $Comp
-L 74xx:74LS257 U15
+L Motherboard-rescue:74LS257-74xx U15
 U 1 1 5BFC38B1
 P 6125 3025
@@
 Connection ~ 4900 3625
 Wire Wire Line
-	5225 3550 5225 3725
-Connection ~ 5225 3725
-Wire Wire Line
 	3975 3700 3975 2575
 Wire Wire Line
@@
 	2850 1450 2900 1450
 $Comp
-L Device:C C1
+L Motherboard-rescue:C-Device C1
 U 1 1 5C115714
 P 1900 2400
@@
 $EndComp
 $Comp
-L power:GND #PWR014
+L Motherboard-rescue:GND-power #PWR014
 U 1 1 5C11571A
 P 1900 2550
@@
 $EndComp
 $Comp
-L 4xxx_IEEE:40106 U9
+L Motherboard-rescue:40106-4xxx_IEEE U9
 U 2 1 5C118563
 P 3475 1450
+AR Path="/5C118563" Ref="U9"  Part="2"
+AR Path="/5C104845/5C118563" Ref="U9"  Part="2"
 F 0 "U9" H 3650 1575 50  0000 L CNN
 F 1 "40106" H 3650 1325 50  0000 L CNN
@@
 	3925 3700 3975 3700
 $Comp
-L Device:C C2
+L Motherboard-rescue:C-Device C2
 U 1 1 5C12ACF7
 P 1900 4650
@@
 $EndComp
 $Comp
-L power:GND #PWR015
+L Motherboard-rescue:GND-power #PWR015
 U 1 1 5C12ACFD
 P 1900 4800
@@
 $EndComp
 $Comp
-L Device:C C4
+L Motherboard-rescue:C-Device C4
 U 1 1 5C12D628
 P 2900 4650
@@
 $EndComp
 $Comp
-L power:GND #PWR017
+L Motherboard-rescue:GND-power #PWR017
 U 1 1 5C12D62E
 P 2900 4800
@@
 $EndComp
 $Comp
-L power:+5V #PWR018
+L Motherboard-rescue:+5V-power #PWR018
 U 1 1 5C1308AD
 P 4900 3250
@@
 $EndComp
 $Comp
-L power:+5V #PWR022
+L Motherboard-rescue:+5V-power #PWR022
 U 1 1 5C130932
-P 5225 3250
-F 0 "#PWR022" H 5225 3100 50  0001 C CNN
-F 1 "+5V" H 5240 3423 50  0000 C CNN
-F 2 "" H 5225 3250 50  0001 C CNN
-F 3 "" H 5225 3250 50  0001 C CNN
-	1    5225 3250
-	1    0    0    -1
-$EndComp
-$Comp
-L Device:R R3
+P 5225 4600
+F 0 "#PWR022" H 5225 4450 50  0001 C CNN
+F 1 "+5V" H 5240 4773 50  0000 C CNN
+F 2 "" H 5225 4600 50  0001 C CNN
+F 3 "" H 5225 4600 50  0001 C CNN
+	1    5225 4600
+	-1   0    0    1
+$EndComp
+$Comp
+L Motherboard-rescue:R-Device R3
 U 1 1 5C130A0B
 P 4900 3400
@@
 $EndComp
 $Comp
-L Device:R R4
-U 1 1 5C130A93
-P 5225 3400
-F 0 "R4" H 5295 3446 50  0000 L CNN
-F 1 "10k" H 5295 3355 50  0000 L CNN
-F 2 "Resistors_THT:R_Axial_DIN0204_L3.6mm_D1.6mm_P5.08mm_Horizontal" V 5155 3400 50  0001 C CNN
-F 3 "~" H 5225 3400 50  0001 C CNN
-	1    5225 3400
-	1    0    0    -1
-$EndComp
-$Comp
-L Switch:SW_SPST SW1
+L Motherboard-rescue:SW_SPST-Switch SW1
 U 1 1 5C131152
 P 4900 4400
@@
 $EndComp
 $Comp
-L Switch:SW_SPST SW2
+L Motherboard-rescue:SW_SPST-Switch SW2
 U 1 1 5C131309
 P 5225 4400
@@
 $EndComp
 $Comp
-L power:GND #PWR019
+L Motherboard-rescue:GND-power #PWR019
 U 1 1 5C131628
 P 4900 4600
@@
 $EndComp
 $Comp
-L power:GND #PWR023
+L Motherboard-rescue:GND-power #PWR023
 U 1 1 5C1316AD
-P 5225 4600
-F 0 "#PWR023" H 5225 4350 50  0001 C CNN
-F 1 "GND" H 5230 4427 50  0000 C CNN
-F 2 "" H 5225 4600 50  0001 C CNN
-F 3 "" H 5225 4600 50  0001 C CNN
-	1    5225 4600
-	1    0    0    -1
+P 5225 3250
+F 0 "#PWR023" H 5225 3000 50  0001 C CNN
+F 1 "GND" H 5230 3077 50  0000 C CNN
+F 2 "" H 5225 3250 50  0001 C CNN
+F 3 "" H 5225 3250 50  0001 C CNN
+	1    5225 3250
+	-1   0    0    1
 $EndComp
 Wire Wire Line
@@
 	5375 2525 5625 2525
 $Comp
-L power:+5V #PWR024
+L Motherboard-rescue:+5V-power #PWR024
 U 1 1 5C14A009
 P 6125 2125
@@
 $EndComp
 $Comp
-L power:GND #PWR025
+L Motherboard-rescue:GND-power #PWR025
 U 1 1 5C14A19D
 P 6125 4025
@@
 READY
 Wire Wire Line
-	5225 3725 5225 4200
-Wire Wire Line
 	4900 3625 4900 4200
 $Comp
@@
 	7825 3325 8200 3325
 $Comp
-L power:+5V #PWR0138
+L Motherboard-rescue:+5V-power #PWR0138
 U 1 1 5C56888A
 P 2400 3550
@@
 $EndComp
 $Comp
-L power:GND #PWR0139
+L Motherboard-rescue:GND-power #PWR0139
 U 1 1 5C56893F
 P 2400 3850
@@
 $EndComp
 $Comp
-L power:GND #PWR0140
+L Motherboard-rescue:GND-power #PWR0140
 U 1 1 5C5689CA
 P 3475 3850
@@
 $EndComp
 $Comp
-L power:+5V #PWR0141
+L Motherboard-rescue:+5V-power #PWR0141
 U 1 1 5C568BBA
 P 3475 3550
@@
 $EndComp
 $Comp
-L power:+5V #PWR0142
+L Motherboard-rescue:+5V-power #PWR0142
 U 1 1 5C56974B
 P 2400 1300
@@
 $EndComp
 $Comp
-L power:+5V #PWR0143
+L Motherboard-rescue:+5V-power #PWR0143
 U 1 1 5C5697D6
 P 3475 1300
@@
 $EndComp
 $Comp
-L power:GND #PWR0144
+L Motherboard-rescue:GND-power #PWR0144
 U 1 1 5C569868
 P 2400 1600
@@
 $EndComp
 $Comp
-L power:GND #PWR0145
+L Motherboard-rescue:GND-power #PWR0145
 U 1 1 5C5698F3
 P 3475 1600
@@
 $EndComp
 $Comp
-L power:GND #PWR0146
+L Motherboard-rescue:GND-power #PWR0146
 U 1 1 5C582F09
 P 8200 3525
@@
 $EndComp
 $Comp
-L power:+5V #PWR0147
+L Motherboard-rescue:+5V-power #PWR0147
 U 1 1 5C583152
 P 9200 2425
@@
 Text HLabel 9200 3025 2    50   Output ~ 0
 ~RESET
+NoConn ~ 9200 2525
+NoConn ~ 9200 2625
+NoConn ~ 9200 2725
+NoConn ~ 9200 2825
+NoConn ~ 9200 2925
+NoConn ~ 9200 3525
+NoConn ~ 8200 3425
+Wire Wire Line
+	5225 3550 5225 3725
+Connection ~ 5225 3725
+Wire Wire Line
+	5225 3725 5225 4200
+$Comp
+L Motherboard-rescue:R-Device R4
+U 1 1 5C130A93
+P 5225 3400
+F 0 "R4" H 5295 3446 50  0000 L CNN
+F 1 "10k" H 5295 3355 50  0000 L CNN
+F 2 "Resistors_THT:R_Axial_DIN0204_L3.6mm_D1.6mm_P5.08mm_Horizontal" V 5155 3400 50  0001 C CNN
+F 3 "~" H 5225 3400 50  0001 C CNN
+	1    5225 3400
+	1    0    0    -1
+$EndComp
 $EndSCHEMATC
