File: Motherboard/FDC-Serial.sch (KiCad schematic (older format))
At the start: 17 parts, among them J10 Conn_02x17_Odd_Even, J11 USB_B, J12 DB9_Male, J13 5749266-1, J14 5749266-1, J15 DB25_Female, U10 GD75232N, U6 FDC37B787-NS, U8 FT231XS, Y3 32.768kHz

Commit message: LARGE sync
Parts:
- U8: symbol Interface_USB:FT231XS -> Motherboard-rescue:FT231XS-Interface_USB
Connections:
- net labels added: D0, D1, D2, D3, D4, D5, D6, D7, D[0...7], RESET_DRV
- net labels removed: XD0, XD1, XD2, XD3, XD4, XD5, XD6, XD7, XD[0...7]
- no-connect marks 11 -> 15
Changed lines of the file:
@@
 EESchema Schematic File Version 4
 LIBS:Motherboard-cache
-EELAYER 26 0
+EELAYER 29 0
 EELAYER END
 $Descr A3 16535 11693
@@
 $EndDescr
 $Comp
-L Interface_USB:FT231XS U8
+L Motherboard-rescue:FT231XS-Interface_USB U8
 U 1 1 5C634F5B
 P 10125 2425
@@
 	5750 7650 5450 7650
 Text Label 5450 7650 0    50   ~ 0
-XD[0...7]
+D[0...7]
 Text HLabel 5450 7650 0    50   Input ~ 0
-XD[0...7]
+D[0...7]
 Text Label 5850 7825 0    50   ~ 0
-XD0
+D0
 Text Label 5850 7925 0    50   ~ 0
-XD1
+D1
 Text Label 5850 8025 0    50   ~ 0
-XD2
+D2
 Text Label 5850 8125 0    50   ~ 0
-XD3
+D3
 Text Label 5850 8325 0    50   ~ 0
-XD4
+D4
 Text Label 5850 8425 0    50   ~ 0
-XD5
+D5
 Text Label 5850 8525 0    50   ~ 0
-XD6
+D6
 Text Label 5850 8625 0    50   ~ 0
-XD7
+D7
 NoConn ~ 8925 8825
 Text HLabel 6050 7625 0    50   Input ~ 0
@@
 Wire Wire Line
 	9025 7625 8925 7625
+Text HLabel 6125 8725 0    50   Input ~ 0
+RESET_DRV
+NoConn ~ 8925 7525
+NoConn ~ 8925 7425
+NoConn ~ 8925 7325
+NoConn ~ 8925 7225
 Wire Bus Line
 	5750 7650 5750 8525
