File: Motherboard/FDC-Serial.sch (KiCad schematic (older format))
At the start: 17 parts, among them J10 Conn_02x17_Odd_Even, J11 USB_B, J12 DB9_Male, J13 5749266-1, J14 5749266-1, J15 DB25_Female, U10 GD75232N, U6 FDC37B787-NS, U8 FT231XS, Y3 32.768kHz

Commit message: A LOT of work
Connections:
- net IRQ14: now reaches U6.39 (PCI_CLK/IRQ14/GP50)
- net IRQ15: now reaches U6.40 (SER_IRQ/IRQ15)
- net IRQ8: now reaches U6.89 (RD6/IRQ8/GP66)
- net IRQ10: now reaches U6.90 (RD7/IRQ10/GP67)
- net IRQ11: now reaches U6.91 (nROMCS/IRQ11/GP53/EETI)
- net IRQ12: now reaches U6.92 (nROMOE/IRQ12/GP54/EETI)
- no-connect marks 15 -> 9
Changed lines of the file:
@@
 EESchema Schematic File Version 4
 LIBS:Motherboard-cache
-EELAYER 29 0
+EELAYER 30 0
 EELAYER END
 $Descr A3 16535 11693
 encoding utf-8
-Sheet 9 10
+Sheet 10 10
 Title ""
 Date ""
@@
 Text HLabel 6025 9725 0    50   Input ~ 0
 TC
-NoConn ~ 6125 7325
-NoConn ~ 6125 7425
 Wire Wire Line
 	6025 8825 6125 8825
@@
 Text HLabel 6125 8725 0    50   Input ~ 0
 RESET_DRV
-NoConn ~ 8925 7525
-NoConn ~ 8925 7425
-NoConn ~ 8925 7325
-NoConn ~ 8925 7225
+Text HLabel 6125 7325 0    50   Output ~ 0
+IRQ14
+Text HLabel 6125 7425 0    50   Output ~ 0
+IRQ15
+Text HLabel 9025 7525 2    50   Output ~ 0
+IRQ8
+Text HLabel 9025 7425 2    50   Output ~ 0
+IRQ10
+Text HLabel 9025 7325 2    50   Output ~ 0
+IRQ11
+Text HLabel 9025 7225 2    50   Output ~ 0
+IRQ12
+Wire Wire Line
+	8925 7525 9025 7525
+Wire Wire Line
+	9025 7425 8925 7425
+Wire Wire Line
+	8925 7325 9025 7325
+Wire Wire Line
+	9025 7225 8925 7225
 Wire Bus Line
 	5750 7650 5750 8525
