File: Motherboard/FDC-Serial.sch (KiCad schematic (older format))
At the start: 17 parts, among them J10 Conn_02x17_Odd_Even, J11 USB_B, J12 DB9_Male, J13 5749266-1, J14 5749266-1, J15 DB25_Female, U10 GD75232N, U6 FDC37B787-NS, U8 FT231XS, Y3 32.768kHz

Commit message: Large Sync
Parts:
- BT1: symbol Device:Battery_Cell -> Motherboard-rescue:Battery_Cell-Device
- C10, C11, C12, C13: symbol Device:C_Small -> Motherboard-rescue:C_Small-Device
- J10: symbol Connector_Generic:Conn_02x17_Odd_Even -> Motherboard-rescue:Conn_02x17_Odd_Even-Connector_Generic
- J11: symbol Connector:USB_B -> Motherboard-rescue:USB_B-Connector
- J12: symbol Connector:DB9_Male -> Motherboard-rescue:DB9_Male-Connector
- J13, J14: symbol Connector:Mini-DIN-6 -> Motherboard-rescue:Mini-DIN-6-Connector
- J15: symbol Connector:DB25_Female -> Motherboard-rescue:DB25_Female-Connector
- R12, R13: symbol Device:R_Small -> Motherboard-rescue:R_Small-Device
- U10: symbol Interface_UART:GD75232N -> Motherboard-rescue:GD75232N-Interface_UART
- Y3: symbol Device:Crystal -> Motherboard-rescue:Crystal-Device
Connections:
- net IRQ10: no longer names the net of U6.90 (RD7/IRQ10/GP67)
- net IRQ11: no longer names the net of U6.91 (nROMCS/IRQ11/GP53/EETI)
- net IRQ12: no longer names the net of U6.92 (nROMOE/IRQ12/GP54/EETI)
- net IRQ14: no longer names the net of U6.39 (PCI_CLK/IRQ14/GP50)
- net IRQ15: no longer names the net of U6.40 (SER_IRQ/IRQ15)
- net IRQ8: no longer names the net of U6.89 (RD6/IRQ8/GP66)
- no-connect marks 9 -> 24
Changed lines of the file:
@@
 $EndComp
 $Comp
-L Connector:DB25_Female J15
+L Motherboard-rescue:DB25_Female-Connector J15
 U 1 1 5C671BA1
 P 11400 6325
@@
 $EndComp
 $Comp
-L Connector:Mini-DIN-6 J13
+L Motherboard-rescue:Mini-DIN-6-Connector J13
 U 1 1 5C672258
 P 10725 8650
@@
 $EndComp
 $Comp
-L Device:Battery_Cell BT1
+L Motherboard-rescue:Battery_Cell-Device BT1
 U 1 1 5C67246D
 P 9000 10100
@@
 	9000 9825 9000 9900
 $Comp
-L power:GND #PWR0172
+L Motherboard-rescue:GND-power #PWR0172
 U 1 1 5C672545
 P 9000 10200
@@
 $EndComp
 $Comp
-L Connector_Generic:Conn_02x17_Odd_Even J10
+L Motherboard-rescue:Conn_02x17_Odd_Even-Connector_Generic J10
 U 1 1 5C672A5F
 P 4875 4325
@@
 $EndComp
 $Comp
-L power:GND #PWR0173
+L Motherboard-rescue:GND-power #PWR0173
 U 1 1 5C672BF5
 P 4675 5225
@@
 $EndComp
 $Comp
-L Connector:Mini-DIN-6 J14
+L Motherboard-rescue:Mini-DIN-6-Connector J14
 U 1 1 5C67380E
 P 10725 9725
@@
 	10725 9425 10725 9175
 $Comp
-L power:GND #PWR0174
+L Motherboard-rescue:GND-power #PWR0174
 U 1 1 5C6755BC
 P 10725 9175
@@
 	10725 9175 10725 8950
 $Comp
-L power:+5V #PWR0175
+L Motherboard-rescue:+5V-power #PWR0175
 U 1 1 5C6757CF
 P 10725 10025
@@
 $EndComp
 $Comp
-L power:+5V #PWR0176
+L Motherboard-rescue:+5V-power #PWR0176
 U 1 1 5C67592C
 P 10725 8350
@@
 NoConn ~ 10825 10025
 $Comp
-L power:GND #PWR0177
+L Motherboard-rescue:GND-power #PWR0177
 U 1 1 5C6769C1
 P 8925 8925
@@
 $EndComp
 $Comp
-L Device:Crystal Y3
+L Motherboard-rescue:Crystal-Device Y3
 U 1 1 5C676BCD
 P 9275 9625
@@
 	8925 9725 9100 9725
 $Comp
-L power:+5V #PWR0178
+L Motherboard-rescue:+5V-power #PWR0178
 U 1 1 5C677D3D
 P 8925 7125
@@
 $EndComp
 $Comp
-L power:GND #PWR0179
+L Motherboard-rescue:GND-power #PWR0179
 U 1 1 5C677E2E
 P 8925 6025
@@
 $EndComp
 $Comp
-L power:+5V #PWR0180
+L Motherboard-rescue:+5V-power #PWR0180
 U 1 1 5C677EE3
 P 8925 4325
@@
 $EndComp
 $Comp
-L power:+5V #PWR0181
+L Motherboard-rescue:+5V-power #PWR0181
 U 1 1 5C678289
 P 6125 9625
@@
 $EndComp
 $Comp
-L power:GND #PWR0182
+L Motherboard-rescue:GND-power #PWR0182
 U 1 1 5C678370
 P 6125 4125
@@
 $EndComp
 $Comp
-L power:GND #PWR0183
+L Motherboard-rescue:GND-power #PWR0183
 U 1 1 5C6784A0
 P 6125 8225
@@
 	8925 9425 9325 9425
 $Comp
-L power:GND #PWR0184
+L Motherboard-rescue:GND-power #PWR0184
 U 1 1 5C678D5B
 P 8925 9625
@@
 ISA-BUS
 $Comp
-L Device:C_Small C10
+L Motherboard-rescue:C_Small-Device C10
 U 1 1 5C67F9D8
 P 9725 9475
@@
 $EndComp
 $Comp
-L Device:C_Small C11
+L Motherboard-rescue:C_Small-Device C11
 U 1 1 5C67FA1C
 P 9725 9775
@@
 Connection ~ 9275 9775
 $Comp
-L power:GND #PWR0185
+L Motherboard-rescue:GND-power #PWR0185
 U 1 1 5C6814B2
 P 9825 9475
@@
 $EndComp
 $Comp
-L power:GND #PWR0186
+L Motherboard-rescue:GND-power #PWR0186
 U 1 1 5C68151C
 P 9825 9775
@@
 NoConn ~ 8925 8725
 $Comp
-L Connector:USB_B J11
+L Motherboard-rescue:USB_B-Connector J11
 U 1 1 5C69AAEA
 P 11175 1125
@@
 	9225 2325 9225 2425
 $Comp
-L power:GND #PWR0187
+L Motherboard-rescue:GND-power #PWR0187
 U 1 1 5C6A0705
 P 9225 2425
@@
 	11275 725  11225 725
 $Comp
-L power:GND #PWR0188
+L Motherboard-rescue:GND-power #PWR0188
 U 1 1 5C6A19BA
 P 11225 725
@@
 	10325 3625 10325 3125
 $Comp
-L power:GND #PWR0189
+L Motherboard-rescue:GND-power #PWR0189
 U 1 1 5C6C208B
 P 13725 3950
@@
 $EndComp
 $Comp
-L Connector:DB9_Male J12
+L Motherboard-rescue:DB9_Male-Connector J12
 U 1 1 5C67181B
 P 14025 4350
@@
 	9800 7525 11100 7525
 $Comp
-L power:GND #PWR0190
+L Motherboard-rescue:GND-power #PWR0190
 U 1 1 5C7227A0
 P 11100 5225
@@
 $EndComp
 $Comp
-L power:GND #PWR0191
+L Motherboard-rescue:GND-power #PWR0191
 U 1 1 5C7227F6
 P 11100 5425
@@
 $EndComp
 $Comp
-L power:GND #PWR0192
+L Motherboard-rescue:GND-power #PWR0192
 U 1 1 5C722868
 P 11100 5625
@@
 $EndComp
 $Comp
-L power:GND #PWR0193
+L Motherboard-rescue:GND-power #PWR0193
 U 1 1 5C7229A8
 P 11100 5825
@@
 $EndComp
 $Comp
-L power:GND #PWR0194
+L Motherboard-rescue:GND-power #PWR0194
 U 1 1 5C7229FE
 P 11100 6025
@@
 $EndComp
 $Comp
-L power:GND #PWR0195
+L Motherboard-rescue:GND-power #PWR0195
 U 1 1 5C722A85
 P 11100 6225
@@
 $EndComp
 $Comp
-L power:GND #PWR0196
+L Motherboard-rescue:GND-power #PWR0196
 U 1 1 5C722ADB
 P 11100 6425
@@
 $EndComp
 $Comp
-L power:GND #PWR0197
+L Motherboard-rescue:GND-power #PWR0197
 U 1 1 5C722B31
 P 11100 6625
@@
 	5175 3525 6125 3525
 $Comp
-L power:+5V #PWR0198
+L Motherboard-rescue:+5V-power #PWR0198
 U 1 1 5C847208
 P 11050 2300
@@
 	11050 2325 11050 2300
 $Comp
-L Device:C_Small C12
+L Motherboard-rescue:C_Small-Device C12
 U 1 1 5C85E897
 P 10125 1275
@@
 	10325 1125 10875 1125
 $Comp
-L Device:C_Small C13
+L Motherboard-rescue:C_Small-Device C13
 U 1 1 5C8CB776
 P 10125 1425
@@
 	10025 1275 10025 1350
 $Comp
-L power:GND #PWR0199
+L Motherboard-rescue:GND-power #PWR0199
 U 1 1 5C902BB9
 P 10025 1350
@@
 	8925 1575 8925 3250
 $Comp
-L Device:R_Small R12
+L Motherboard-rescue:R_Small-Device R12
 U 1 1 5C9265E7
 P 9200 3250
@@
 $EndComp
 $Comp
-L Device:R_Small R13
+L Motherboard-rescue:R_Small-Device R13
 U 1 1 5C9268FC
 P 9525 3400
@@
 $EndComp
 $Comp
-L power:GND #PWR0200
+L Motherboard-rescue:GND-power #PWR0200
 U 1 1 5C92695D
 P 9525 3500
@@
 Connection ~ 9525 3250
 $Comp
-L Interface_UART:GD75232N U10
+L Motherboard-rescue:GD75232N-Interface_UART U10
 U 1 1 5C97A1F6
 P 12650 4450
@@
 $EndComp
 $Comp
-L power:GND #PWR0201
+L Motherboard-rescue:GND-power #PWR0201
 U 1 1 5C9977B4
 P 12550 5150
@@
 $EndComp
 $Comp
-L power:+5V #PWR0202
+L Motherboard-rescue:+5V-power #PWR0202
 U 1 1 5C9978EB
 P 12550 3750
@@
 $EndComp
 $Comp
-L power:+12V #PWR0203
+L Motherboard-rescue:+12V-power #PWR0203
 U 1 1 5C9979D4
 P 12750 3750
@@
 $EndComp
 $Comp
-L power:-12V #PWR0204
+L Motherboard-rescue:-12V-power #PWR0204
 U 1 1 5C997A7D
 P 12750 5150
@@
 Text HLabel 6125 8725 0    50   Input ~ 0
 RESET_DRV
-Text HLabel 6125 7325 0    50   Output ~ 0
-IRQ14
-Text HLabel 6125 7425 0    50   Output ~ 0
-IRQ15
-Text HLabel 9025 7525 2    50   Output ~ 0
-IRQ8
-Text HLabel 9025 7425 2    50   Output ~ 0
-IRQ10
-Text HLabel 9025 7325 2    50   Output ~ 0
-IRQ11
-Text HLabel 9025 7225 2    50   Output ~ 0
-IRQ12
-Wire Wire Line
-	8925 7525 9025 7525
-Wire Wire Line
-	9025 7425 8925 7425
-Wire Wire Line
-	8925 7325 9025 7325
-Wire Wire Line
-	9025 7225 8925 7225
+NoConn ~ 8925 7225
+NoConn ~ 8925 7325
+NoConn ~ 8925 7425
+NoConn ~ 8925 7525
+NoConn ~ 8925 8225
+NoConn ~ 8925 8325
+NoConn ~ 8925 8425
+NoConn ~ 8925 8525
+NoConn ~ 8925 8625
+NoConn ~ 6125 5225
+NoConn ~ 6125 5325
+NoConn ~ 6125 5425
+NoConn ~ 6125 5525
+NoConn ~ 6125 7325
+NoConn ~ 6125 7425
 Wire Bus Line
 	5750 7650 5750 8525
