File: Motherboard/MIDI.sch (KiCad schematic (older format))
At the start: 24 parts, among them J9 AudioJack3_SwitchTR, U12 ATF750LVC-fdc, U13 ATmega328-PU, U14 SN76489A-ALT, U16 LM386, U17 MAX538BEPA+, U20 LM386, U21 LM386, U35 74LS245

Commit message: end of day commit, routed major parts of the motherboard
Parts:
- U14: symbol TI_Sound:SN76489A-ALT -> Motherboard-rescue:SN76489A-ALT-TI_Sound
Changed lines of the file:
@@
 EESchema Schematic File Version 4
 LIBS:Motherboard-cache
-EELAYER 29 0
+EELAYER 26 0
 EELAYER END
 $Descr A4 11693 8268
@@
 $EndComp
 $Comp
-L TI_Sound:SN76489A-ALT U14
+L Motherboard-rescue:SN76489A-ALT-TI_Sound U14
 U 1 1 5C81A05B
 P 4925 1450
