File: Motherboard/MIDI.sch (KiCad schematic (older format))
At the start: 24 parts, among them J9 AudioJack3_SwitchTR, U12 ATF750LVC-fdc, U13 ATmega328-PU, U14 SN76489A-ALT, U16 LM386, U17 MAX538BEPA+, U20 LM386, U21 LM386, U35 74LS245

Commit message: Fixed schematics after merge
Parts:
- U13: symbol MCU_Microchip_ATmega:ATmega328-PU -> Motherboard-rescue:ATmega328-PU-MCU_Microchip_ATmega
Changed lines of the file:
@@
 EESchema Schematic File Version 4
-LIBS:Motherboard-cache
 EELAYER 30 0
 EELAYER END
@@
 $EndDescr
 $Comp
-L MCU_Microchip_ATmega:ATmega328-PU U13
+L Motherboard-rescue:ATmega328-PU-MCU_Microchip_ATmega U13
 U 1 1 5C7F04CC
 P 2950 4770

Commit message: Large Sync
Parts:
- C14, C16, C17, C19: symbol Device:C -> Motherboard-rescue:C-Device
- C15, C18, C20: symbol Device:CP -> Motherboard-rescue:CP-Device
- LS1: symbol Device:Speaker -> Motherboard-rescue:Speaker-Device
- R14, R15, R16: symbol Device:R -> Motherboard-rescue:R-Device
- RN3: symbol Device:R_Network03 -> Motherboard-rescue:R_Network03-Device
- RV1, RV2, RV3: symbol Device:R_POT -> Motherboard-rescue:R_POT-Device
- U14: symbol TI_Sound:SN76489A-ALT -> Motherboard-rescue:SN76489A-ALT-TI_Sound
- U16, U20, U21: symbol Amplifier_Audio:LM386 -> Motherboard-rescue:LM386-Amplifier_Audio
- U35: symbol 74xx:74LS245 -> Motherboard-rescue:74LS245-74xx
Changed lines of the file:
@@
 DACCS
 $Comp
-L power:+5V #PWR048
+L Motherboard-rescue:+5V-power #PWR048
 U 1 1 5C7F0AAC
 P 7650 3775
@@
 $EndComp
 $Comp
-L power:+3V3 #PWR049
+L Motherboard-rescue:+3V3-power #PWR049
 U 1 1 5C7F0B44
 P 7650 4200
@@
 Connection ~ 9350 2300
 $Comp
-L power:GND #PWR066
+L Motherboard-rescue:GND-power #PWR066
 U 1 1 5C7F186E
 P 9575 2500
@@
 $EndComp
 $Comp
-L Device:Speaker LS1
+L Motherboard-rescue:Speaker-Device LS1
 U 1 1 5C7F19D3
 P 9350 1475
@@
 Connection ~ 9450 2100
 $Comp
-L power:GND #PWR055
+L Motherboard-rescue:GND-power #PWR055
 U 1 1 5C7F1FEF
 P 9350 1675
@@
 	8275 4100 8275 4125
 $Comp
-L power:GND #PWR050
+L Motherboard-rescue:GND-power #PWR050
 U 1 1 5C7F4DE2
 P 7650 4300
@@
 $EndComp
 $Comp
-L Device:C C16
+L Motherboard-rescue:C-Device C16
 U 1 1 5C7F507D
 P 7925 3875
@@
 	7650 3875 7650 4000
 $Comp
-L power:GND #PWR051
+L Motherboard-rescue:GND-power #PWR051
 U 1 1 5C7F56DD
 P 8075 3875
@@
 $EndComp
 $Comp
-L power:+5V #PWR029
+L Motherboard-rescue:+5V-power #PWR029
 U 1 1 5C7F5A92
 P 2950 3220
@@
 	2950 3220 3050 3220
 $Comp
-L power:GND #PWR030
+L Motherboard-rescue:GND-power #PWR030
 U 1 1 5C7F6872
 P 2950 6270
@@
 $EndComp
 $Comp
-L power:GND #PWR028
+L Motherboard-rescue:GND-power #PWR028
 U 1 1 5C7F69D9
 P 2250 2325
@@
 $EndComp
 $Comp
-L power:+5V #PWR040
+L Motherboard-rescue:+5V-power #PWR040
 U 1 1 5C7F6A91
 P 3250 1225
@@
 ~~4MHZ
 $Comp
-L power:GND #PWR042
+L Motherboard-rescue:GND-power #PWR042
 U 1 1 5C81991F
 P 4925 2100
@@
 $EndComp
 $Comp
-L power:+5V #PWR041
+L Motherboard-rescue:+5V-power #PWR041
 U 1 1 5C819972
 P 4925 800
@@
 $EndComp
 $Comp
-L TI_Sound:SN76489A-ALT U14
+L Motherboard-rescue:SN76489A-ALT-TI_Sound U14
 U 1 1 5C81A05B
 P 4925 1450
@@
 TANDY
 $Comp
-L Amplifier_Audio:LM386 U16
+L Motherboard-rescue:LM386-Amplifier_Audio U16
 U 1 1 5C826135
 P 6375 1925
@@
 	6075 2225 6075 2025
 $Comp
-L power:+5V #PWR045
+L Motherboard-rescue:+5V-power #PWR045
 U 1 1 5C82613D
 P 6275 1625
@@
 NoConn ~ 6475 2225
 $Comp
-L Device:CP C15
+L Motherboard-rescue:CP-Device C15
 U 1 1 5C826146
 P 7175 1925
@@
 	6675 1925 6850 1925
 $Comp
-L Device:C C14
+L Motherboard-rescue:C-Device C14
 U 1 1 5C82614D
 P 6850 2125
@@
 	6850 1925 7025 1925
 $Comp
-L power:GND #PWR046
+L Motherboard-rescue:GND-power #PWR046
 U 1 1 5C826156
 P 6850 2575
@@
 $EndComp
 $Comp
-L Device:R R14
+L Motherboard-rescue:R-Device R14
 U 1 1 5C82615C
 P 6850 2425
@@
 $EndComp
 $Comp
-L power:GND #PWR044
+L Motherboard-rescue:GND-power #PWR044
 U 1 1 5C826164
 P 6075 2225
@@
 Connection ~ 6075 2225
 $Comp
-L Device:R_POT RV1
+L Motherboard-rescue:R_POT-Device RV1
 U 1 1 5C82616B
 P 5725 1825
@@
 	5725 1650 5725 1675
 $Comp
-L power:GND #PWR043
+L Motherboard-rescue:GND-power #PWR043
 U 1 1 5C826174
 P 5725 1975
@@
 SPEAKER
 $Comp
-L Device:R_Network03 RN3
+L Motherboard-rescue:R_Network03-Device RN3
 U 1 1 5CDDDDDA
 P 8925 2400
@@
 SPKR
 $Comp
-L Amplifier_Audio:LM386 U20
+L Motherboard-rescue:LM386-Amplifier_Audio U20
 U 1 1 5CDF7EAD
 P 4975 2850
@@
 	4675 3150 4675 2950
 $Comp
-L power:+5V #PWR054
+L Motherboard-rescue:+5V-power #PWR054
 U 1 1 5CDF7EB5
 P 4875 2550
@@
 NoConn ~ 5075 3150
 $Comp
-L Device:CP C18
+L Motherboard-rescue:CP-Device C18
 U 1 1 5CDF7EBE
 P 5775 2850
@@
 	5275 2850 5450 2850
 $Comp
-L Device:C C17
+L Motherboard-rescue:C-Device C17
 U 1 1 5CDF7EC5
 P 5450 3050
@@
 	5450 2850 5625 2850
 $Comp
-L power:GND #PWR064
+L Motherboard-rescue:GND-power #PWR064
 U 1 1 5CDF7ECE
 P 5450 3500
@@
 $EndComp
 $Comp
-L Device:R R15
+L Motherboard-rescue:R-Device R15
 U 1 1 5CDF7ED4
 P 5450 3350
@@
 $EndComp
 $Comp
-L power:GND #PWR053
+L Motherboard-rescue:GND-power #PWR053
 U 1 1 5CDF7EDA
 P 4675 3150
@@
 Connection ~ 4675 3150
 $Comp
-L Device:R_POT RV2
+L Motherboard-rescue:R_POT-Device RV2
 U 1 1 5CDF7EE1
 P 4325 2750
@@
 	4325 2575 4325 2600
 $Comp
-L power:GND #PWR052
+L Motherboard-rescue:GND-power #PWR052
 U 1 1 5CDF7EE9
 P 4325 2900
@@
 	4000 2575 4325 2575
 $Comp
-L Amplifier_Audio:LM386 U21
+L Motherboard-rescue:LM386-Amplifier_Audio U21
 U 1 1 5CE00BE1
 P 8925 4375
@@
 	8625 4675 8625 4475
 $Comp
-L power:+5V #PWR069
+L Motherboard-rescue:+5V-power #PWR069
 U 1 1 5CE00BE9
 P 8825 4075
@@
 NoConn ~ 9025 4675
 $Comp
-L Device:CP C20
+L Motherboard-rescue:CP-Device C20
 U 1 1 5CE00BF2
 P 9725 4375
@@
 	9225 4375 9400 4375
 $Comp
-L Device:C C19
+L Motherboard-rescue:C-Device C19
 U 1 1 5CE00BF9
 P 9400 4575
@@
 	9400 4375 9575 4375
 $Comp
-L power:GND #PWR070
+L Motherboard-rescue:GND-power #PWR070
 U 1 1 5CE00C02
 P 9400 5025
@@
 $EndComp
 $Comp
-L Device:R R16
+L Motherboard-rescue:R-Device R16
 U 1 1 5CE00C08
 P 9400 4875
@@
 $EndComp
 $Comp
-L power:GND #PWR068
+L Motherboard-rescue:GND-power #PWR068
 U 1 1 5CE00C0E
 P 8625 4675
@@
 Connection ~ 8625 4675
 $Comp
-L Device:R_POT RV3
+L Motherboard-rescue:R_POT-Device RV3
 U 1 1 5CE00C15
 P 8275 4275
@@
 	8425 4275 8625 4275
 $Comp
-L power:GND #PWR067
+L Motherboard-rescue:GND-power #PWR067
 U 1 1 5CE00C1D
 P 8275 4425
@@
 ~IOR
 $Comp
-L 74xx:74LS245 U35
+L Motherboard-rescue:74LS245-74xx U35
 U 1 1 5CE4E451
 P 4225 5770
@@
 ~IOW
 $Comp
-L power:GND #PWR0164
+L Motherboard-rescue:GND-power #PWR0164
 U 1 1 5CE7F569
 P 4225 6570
@@
 $EndComp
 $Comp
-L power:+5V #PWR0208
+L Motherboard-rescue:+5V-power #PWR0208
 U 1 1 5CE7F5DA
 P 4225 4970
