File: Motherboard/Motherboard.sch (KiCad schematic (older format))
At the start: 4 parts, among them U1 82C54_PLCC, U11 8087, U2 8088, U3 8259

Commit message: LARGE sync
Parts:
- added R17, R18, R19: 4k7, Resistor_THT:R_Axial_DIN0204_L3.6mm_D1.6mm_P5.08mm_Vertical, symbol Device:R_Small
- added U18: ATF750LVC-fdc, Housings_DIP:DIP-24_W7.62mm_Socket, symbol Motherboard-rescue:ATF750LVC-fdc
- added U19: 74LS32, symbol 74xx:74LS32
- added U22: 8259, Housings_DIP:DIP-28_W7.62mm_Socket, symbol Interface:8259
- added U37: 74LS74, Package_DIP:DIP-14_W7.62mm_Socket, symbol 74xx:74LS74
- added U4: 74LS137, symbol 74xx:74LS137
Connections:
- net D0 is gone; now on net XD0: U3.11 (D0)
- net D1 is gone; now on net XD1: U3.10 (D1)
- net D2 is gone; now on net XD2: U3.9 (D2)
- net D3 is gone; now on net XD3: U3.8 (D3)
- net D4 is gone; now on net XD4: U3.7 (D4)
- net D5 is gone; now on net XD5: U3.6 (D5)
- net D6 is gone; now on net XD6: U3.5 (D6)
- net D7 is gone; now on net XD7: U3.4 (D7)
- net HRQ is gone; now on net PU: U2.31 (~RQ~/~GT0~)
- net +5V: now also U1.13 (G0), U1.17 (G1), U1.28 (VCC), U11.34 (~BHE~/S7), U3.28 (VCC), R17.1, R18.1, R19.1, U18.24 (VCC), U19.14 (VCC), U37.10 (~S), U37.14 (VCC), U37.2 (D), U37.4 (~S), U4.16 (VCC)
- net DRQ0: now also U37.5 (Q)
- net GND: now also U1.14 (GND), U3.14 (GND), U18.12 (GND), U19.7 (GND), U22.14 (GND), U22.16 (~SP~/~EN~), U37.7 (GND), U4.8 (GND)
- net HLDA: now also U11.31 (~RQ~/~GT0~), R19.2
- net ~AEN: now also U4.6 (G1)
- net ~DACK0BRD: now also U37.1 (~R)
- net ~INTA: now also U22.26 (~INTA~)
- net NMI: now reaches U2.17 (NMI)
- net INTR: now reaches U2.18 (INTR)
- net INTR: now also U3.17 (INT)
- net BSY: now reaches U2.23 (~TEST~)
- net BSY: now also U11.23 (BUSY), R18.2
- net QS1: now reaches U2.24 (QS1)
- net QS1: now also U11.24 (QS1)
- net QS0: now reaches U2.25 (QS0)
- net QS0: now also U11.25 (QS0)
- net ~LOCK: now reaches U2.29 (~LOCK~)
- net ~INTRCS: now reaches U3.1 (~CS~)
- net ~INTRCS: now also U4.14 (Y1)
- net at U3.12 (CAS0): now also U22.12 (CAS0)
- net at U3.13 (CAS1): now also U22.13 (CAS1)
- net at U3.15 (CAS2): now also U22.15 (CAS2)
- net PU: now reaches U3.16 (~SP~/~EN~)
- net PU: now also U11.33 (~RQ~/~GT1~), R17.2
- net IRQ0: now reaches U3.18 (IR0)
- net IRQ0: now also U1.12 (OUT0)
- net ~XIOR: now reaches U3.2 (~RD~)
- net ~XIOR: now also U1.26 (~RD~), U18.13 (IN), U22.2 (~RD~)
- net SIRQ: now reaches U3.20 (IR2)
- net SIRQ: now also U22.17 (INT)
- net XA0: now reaches U3.27 (A0)
- net XA0: now also U1.22 (A0), U18.2 (IN), U22.27 (A0)
- net ~XIOW: now reaches U3.3 (~WR~)
- net ~XIOW: now also U1.27 (~WR~), U18.1 (CLK/IN), U19.1, U19.4, U22.3 (~WR~)
- net at U1.10 (CLK0): now also U1.18 (CLK1), U1.21 (CLK2), U37.9 (Q)
- net at U1.16 (OUT1): now also U37.3 (C)
- net at U1.19 (G2): now also U18.23 (I/O)
- net XD7: now reaches U1.2 (D7)
- net XD7: now also U18.11 (IN), U22.4 (D7)
- net SPEAKER: now reaches U1.20 (OUT2)
- net XA1: now reaches U1.23 (A1)
- net XA1: now also U18.3 (IN)
- net XD6: now reaches U1.3 (D6)
- net XD6: now also U18.10 (I/O), U22.5 (D6)
- net XD5: now reaches U1.4 (D5)
- net XD5: now also U18.9 (I/O), U22.6 (D5)
- net XD4: now reaches U1.5 (D4)
- net XD4: now also U18.8 (IN), U22.7 (D4)
- net XD3: now reaches U1.6 (D3)
- net XD3: now also U18.7 (IN), U22.8 (D3)
- net XD2: now reaches U1.7 (D2)
- net XD2: now also U18.6 (IN), U22.9 (D2)
- net XD1: now reaches U1.8 (D1)
- net XD1: now also U18.5 (IN), U22.10 (D1)
- net XD0: now reaches U1.9 (D0)
- net XD0: now also U18.4 (IN), U22.11 (D0)
- new net: U37.12 (D), U37.8 (~Q)
- new net: U19.5, U4.11 (Y4)
- new net ENB_IO_CK: U18.21 (I/O)
- new net IRQ10: U22.20 (IR2)
- new net IRQ11: U22.21 (IR3)
- new net IRQ12: U22.22 (IR4)
- new net IRQ13: U22.23 (IR5)
- new net IRQ14: U22.24 (IR6)
- new net IRQ15: U22.25 (IR7)
- new net IRQ8: U22.18 (IR0)
- new net IRQ9: U22.19 (IR1)
- new net PCLK: U37.11 (C)
- new net PPICS: U18.14 (I/O)
- new net SPKR_DATA: U18.22 (I/O)
- new net XA5: U4.3 (A2)
- new net XA6: U4.2 (A1)
- new net XA7: U4.1 (A0)
- new net XA8: U4.5 (~G2)
- new net XA9: U4.4 (~GL)
- new net ~DMACS: U4.15 (Y0)
- new net ~INTR2CS: U19.2, U4.10 (Y5)
- new net ~INTRCS2: U22.1 (~CS~)
- new net ~PPICS: U4.12 (Y3)
- new net ~RESET: U37.13 (~R)
- new net ~TCCS: U4.13 (Y2)
- new net ~WRTDMAPGREG: U19.6
- new net ~WRTNMIREG: U19.3
- no-connect marks 0 -> 5
Other:
- note added: "IRQ2 = IRQ9"
- note added: "Lista ut NMI Addr...\nAT använder PROM för avkodning"
- moved on the sheet: U1, U3
