File: Motherboard/Motherboard.sch (KiCad schematic (older format))
At the start: 12 parts, among them U1 82C54_PLCC, U11 8087, U18 ATF750LVC-fdc, U19 74LS32, U2 8088, U22 8259, U3 8259, U37 74LS74, U4 74LS137

Commit message: Large Sync
Parts:
- removed unit 5 of U19
- removed U22: 8259, Housings_DIP:DIP-28_W7.62mm_Socket, symbol Motherboard-rescue:8259-Interface
- R17, R18, R19: symbol Device:R_Small -> Motherboard-rescue:R_Small-Device
- U1: symbol Timer:82C54_PLCC -> Motherboard-rescue:82C54_PLCC-Timer
- U11: symbol MCU_Intel:8087 -> Motherboard-rescue:8087-MCU_Intel
- U19: symbol 74xx:74LS32 -> Motherboard-rescue:74LS32-74xx
- U2: symbol MCU_Intel:8088_Max_Mode -> Motherboard-rescue:8088_Max_Mode-MCU_Intel
- U37: symbol 74xx:74LS74 -> Motherboard-rescue:74LS74-74xx
- U4: symbol 74xx:74LS137 -> Motherboard-rescue:74LS137-74xx
Connections:
- net SIRQ is gone; now on net IRQ2: U3.20 (IR2)
- net XA5: now also U4.1 (A0); no longer U4.3 (A2)
- net XA7: now also U4.3 (A2); no longer U4.1 (A0)
- net ~INTR2CS: no longer names the net of U19.2, U4.10 (Y5)
- no-connect marks 5 -> 8
