File: Motherboard/PSU.sch (KiCad schematic (older format))
At the start: 11 parts, among them J4 ATX24, J8 3.3V_HEADER, SW3 SW_SPST_LED, SW4 RESET, U38 L79L05_TO92

Commit message: Large Sync
Parts:
- C21, C22: symbol Device:CP -> Motherboard-rescue:CP-Device
- D1: symbol Diode:1N4001 -> Motherboard-rescue:1N4001-Diode
- J8: symbol Connector_Generic:Conn_02x03_Odd_Even -> Motherboard-rescue:Conn_02x03_Odd_Even-Connector_Generic
- R6, R7, R8: symbol Device:R -> Motherboard-rescue:R-Device
- SW3: symbol Switch:SW_SPST_LED -> Motherboard-rescue:SW_SPST_LED-Switch
- SW4: symbol Switch:SW_Push -> Motherboard-rescue:SW_Push-Switch
- U38: symbol Regulator_Linear:L79L05_TO92 -> Motherboard-rescue:L79L05_TO92-Regulator_Linear
Changed lines of the file:
@@
 $EndComp
 $Comp
-L Switch:SW_SPST_LED SW3
+L Motherboard-rescue:SW_SPST_LED-Switch SW3
 U 1 1 5C30AF4E
 P 3675 2250
@@
 	3575 2450 3625 2450
 $Comp
-L power:GND #PWR0101
+L Motherboard-rescue:GND-power #PWR0101
 U 1 1 5C30B19D
 P 3625 2450
@@
 	3625 2450 3675 2450
 $Comp
-L power:+3V3 #PWR0102
+L Motherboard-rescue:+3V3-power #PWR0102
 U 1 1 5C30B28F
 P 2275 1200
@@
 POK
 $Comp
-L power:+3V3 #PWR0103
+L Motherboard-rescue:+3V3-power #PWR0103
 U 1 1 5C30B891
 P 1625 2775
@@
 	1625 2475 1925 2475
 $Comp
-L power:GND #PWR0104
+L Motherboard-rescue:GND-power #PWR0104
 U 1 1 5C30D498
 P 2750 2175
@@
 $EndComp
 $Comp
-L power:+5V #PWR0105
+L Motherboard-rescue:+5V-power #PWR0105
 U 1 1 5C30D4D2
 P 2750 2575
@@
 $EndComp
 $Comp
-L power:+5V #PWR0106
+L Motherboard-rescue:+5V-power #PWR0106
 U 1 1 5C30D539
 P 1600 2075
@@
 GND
 $Comp
-L power:-12V #PWR0107
+L Motherboard-rescue:-12V-power #PWR0107
 U 1 1 5C30E6AA
 P 2850 1650
@@
 GND
 $Comp
-L power:GND #PWR0108
+L Motherboard-rescue:GND-power #PWR0108
 U 1 1 5C30ED86
 P 2650 3350
@@
 	2650 3250 2650 3350
 $Comp
-L Device:R R6
+L Motherboard-rescue:R-Device R6
 U 1 1 5C30F4E0
 P 3425 1975
@@
 	2625 1975 3275 1975
 $Comp
-L Switch:SW_Push SW4
+L Motherboard-rescue:SW_Push-Switch SW4
 U 1 1 5C317854
 P 5100 1950
@@
 Connection ~ 5100 1750
 $Comp
-L Device:R R8
+L Motherboard-rescue:R-Device R8
 U 1 1 5C322C7C
 P 5100 2300
@@
 $EndComp
 $Comp
-L Device:R R7
+L Motherboard-rescue:R-Device R7
 U 1 1 5C322F17
 P 3675 1825
@@
 	3675 1575 3675 1675
 $Comp
-L power:GND #PWR0109
+L Motherboard-rescue:GND-power #PWR0109
 U 1 1 5C3237F3
 P 5100 2450
@@
 	2625 2375 2750 2375
 $Comp
-L power:-5V #PWR0126
+L Motherboard-rescue:-5V-power #PWR0126
 U 1 1 5C3282DF
 P 2750 2375
@@
 If present on\nATX supply
 $Comp
-L power:+12V #PWR0127
+L Motherboard-rescue:+12V-power #PWR0127
 U 1 1 5C329C6E
 P 1850 2625
@@
 	1850 2625 1850 2675
 $Comp
-L Connector_Generic:Conn_02x03_Odd_Even J8
+L Motherboard-rescue:Conn_02x03_Odd_Even-Connector_Generic J8
 U 1 1 5C5AECD2
 P 1350 1050
@@
 	1150 1050 1150 1150
 $Comp
-L power:GND #PWR05
+L Motherboard-rescue:GND-power #PWR05
 U 1 1 5C5B02E8
 P 1150 1150
@@
 Connection ~ 1150 1150
 $Comp
-L Regulator_Linear:L79L05_TO92 U38
+L Motherboard-rescue:L79L05_TO92-Regulator_Linear U38
 U 1 1 5C9522CD
 P 3680 3490
@@
 $EndComp
 $Comp
-L Device:CP C21
+L Motherboard-rescue:CP-Device C21
 U 1 1 5C95256B
 P 3150 3300
@@
 $EndComp
 $Comp
-L Device:CP C22
+L Motherboard-rescue:CP-Device C22
 U 1 1 5C9526F7
 P 4290 3300
@@
 $EndComp
 $Comp
-L Diode:1N4001 D1
+L Motherboard-rescue:1N4001-Diode D1
 U 1 1 5C9527BC
 P 3680 3840
@@
 	3680 3150 4290 3150
 $Comp
-L power:GND #PWR083
+L Motherboard-rescue:GND-power #PWR083
 U 1 1 5C95F2A2
 P 3680 3150
@@
 Connection ~ 3150 3490
 $Comp
-L power:-12V #PWR082
+L Motherboard-rescue:-12V-power #PWR082
 U 1 1 5C960419
 P 2890 3290
@@
 	4640 3490 4640 3290
 $Comp
-L power:-5V #PWR084
+L Motherboard-rescue:-5V-power #PWR084
 U 1 1 5C961532
 P 4640 3290
