File: Motherboard/IO-Decoder.sch (KiCad schematic (older format))
At the start: 20 parts, among them U28 8288, U29 74LS245, U30 74LS04, U31 74LS573, U32 74LS244, U33 74LS573, U40 74LS27, U41 74LS04, U42 AS6C8008, U43 74LS244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

Commit message: A LOT of work
Connections:
- net ~IORC renamed ~IOR
- net ~MRDC renamed ~MEMR
Changed lines of the file:
@@
 EESchema Schematic File Version 4
 LIBS:Motherboard-cache
-EELAYER 29 0
+EELAYER 30 0
 EELAYER END
 $Descr A3 16535 11693
@@
 	2625 1600 3000 1600
 Text HLabel 3675 1700 2    50   Output ~ 0
-~MRDC
+~MEMR
 Text HLabel 3675 1800 2    50   Output ~ 0
-~IORC
+~IOR
 Text HLabel 3675 1900 2    50   Input ~ 0
 ~INTA
