File: Motherboard/IO-Decoder.sch (KiCad schematic (older format))
At the start: 20 parts, among them U28 8288, U29 74LS245, U30 74LS04, U31 74LS573, U32 74LS244, U33 74LS573, U40 74LS27, U41 74LS04, U42 AS6C8008, U43 74LS244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

Commit message: Fixed schematics after merge
Parts:
- U42: symbol Motherboard-rescue:AS6C8008-RAM -> RAM:AS6C8008
Changed lines of the file:
@@
 EESchema Schematic File Version 4
-LIBS:Motherboard-cache
 EELAYER 30 0
 EELAYER END
@@
 $EndComp
 $Comp
-L Motherboard-rescue:AS6C8008-RAM U42
+L RAM:AS6C8008 U42
 U 1 1 5CA57105
 P 5155 9710

Commit message: Large Sync
Parts:
- RN1: symbol Device:R_Network05 -> Motherboard-rescue:R_Network05-Device
- RN2: symbol Device:R_Network04 -> Motherboard-rescue:R_Network04-Device
- U28: symbol Interface:8288 -> Motherboard-rescue:8288-Interface
- U29, U46, U47: symbol 74xx:74LS245 -> Motherboard-rescue:74LS245-74xx
- U30, U41: symbol 74xx:74LS04 -> Motherboard-rescue:74LS04-74xx
- U31, U33: symbol 74xx:74LS573 -> Motherboard-rescue:74LS573-74xx
- U32, U43, U44, U45: symbol 74xx:74LS244 -> Motherboard-rescue:74LS244-74xx
- U40: symbol 74xx:74LS27 -> Motherboard-rescue:74LS27-74xx
- U42: symbol RAM:AS6C8008 -> Motherboard-rescue:AS6C8008-RAM
- U48: symbol Memory_Flash:SST39SF010 -> Motherboard-rescue:SST39SF010-Memory_Flash
- U49: symbol 74xx:74LS243 -> Motherboard-rescue:74LS243-74xx
- U50: symbol 74xx:7400 -> Motherboard-rescue:7400-74xx
- U52: symbol 74xx:74LS32 -> Motherboard-rescue:74LS32-74xx
Changed lines of the file:
@@
 AD[0...19]
 $Comp
-L Interface:8288 U28
+L Motherboard-rescue:8288-Interface U28
 U 1 1 5C32B2F4
 P 1925 1900
@@
 $EndComp
 $Comp
-L 74xx:74LS245 U29
+L Motherboard-rescue:74LS245-74xx U29
 U 1 1 5C32B3C4
 P 1975 4925
@@
 $EndComp
 $Comp
-L 74xx:74LS244 U32
+L Motherboard-rescue:74LS244-74xx U32
 U 1 1 5C32B65A
 P 5400 4500
@@
 	1075 2400 1225 2400
 $Comp
-L power:GND #PWR0128
+L Motherboard-rescue:GND-power #PWR0128
 U 1 1 5C32E57E
 P 675 2350
@@
 	675  2300 1225 2300
 $Comp
-L power:+5V #PWR0129
+L Motherboard-rescue:+5V-power #PWR0129
 U 1 1 5C32E776
 P 1925 1000
@@
 $EndComp
 $Comp
-L power:GND #PWR0130
+L Motherboard-rescue:GND-power #PWR0130
 U 1 1 5C32E81E
 P 1925 2800
@@
 NoConn ~ 2625 2400
 $Comp
-L Device:R_Network05 RN1
+L Motherboard-rescue:R_Network05-Device RN1
 U 1 1 5C32EDA5
 P 3000 975
@@
 	3200 1800 3675 1800
 $Comp
-L power:+5V #PWR0131
+L Motherboard-rescue:+5V-power #PWR0131
 U 1 1 5C33048A
 P 2800 775
@@
 $EndComp
 $Comp
-L 74xx:74LS04 U30
+L Motherboard-rescue:74LS04-74xx U30
 U 1 1 5C330D78
 P 2750 2925
@@
 	2750 2500 2750 2625
 $Comp
-L power:+5V #PWR0132
+L Motherboard-rescue:+5V-power #PWR0132
 U 1 1 5C331F2B
 P 1975 4125
@@
 $EndComp
 $Comp
-L power:GND #PWR0133
+L Motherboard-rescue:GND-power #PWR0133
 U 1 1 5C331FAF
 P 1975 5725
@@
 AENBRD
 $Comp
-L power:GND #PWR0134
+L Motherboard-rescue:GND-power #PWR0134
 U 1 1 5C3CDBF7
 P 5400 7325
@@
 $EndComp
 $Comp
-L power:GND #PWR0135
+L Motherboard-rescue:GND-power #PWR0135
 U 1 1 5C3CDC97
 P 5400 5300
@@
 $EndComp
 $Comp
-L power:GND #PWR0136
+L Motherboard-rescue:GND-power #PWR0136
 U 1 1 5C3CDD0D
 P 5350 2850
@@
 $EndSheet
 $Comp
-L 74xx:74LS573 U33
+L Motherboard-rescue:74LS573-74xx U33
 U 1 1 5C352412
 P 5400 6525
@@
 $EndComp
 $Comp
-L 74xx:74LS573 U31
+L Motherboard-rescue:74LS573-74xx U31
 U 1 1 5C35252C
 P 5350 2050
@@
 XCLK
 $Comp
-L 74xx:74LS244 U43
+L Motherboard-rescue:74LS244-74xx U43
 U 1 1 5C4C44F2
 P 10350 2000
@@
 $EndComp
 $Comp
-L 74xx:74LS244 U44
+L Motherboard-rescue:74LS244-74xx U44
 U 1 1 5C4C45B6
 P 10350 3950
@@
 $EndComp
 $Comp
-L 74xx:74LS244 U45
+L Motherboard-rescue:74LS244-74xx U45
 U 1 1 5C4C4634
 P 10375 5850
@@
 $EndComp
 $Comp
-L 74xx:74LS245 U46
+L Motherboard-rescue:74LS245-74xx U46
 U 1 1 5C4C4857
 P 10375 7700
@@
 ~MEMW
 $Comp
-L 74xx:74LS243 U49
+L Motherboard-rescue:74LS243-74xx U49
 U 1 1 5C59AF38
 P 13775 1950
@@
 $EndComp
 $Comp
-L Device:R_Network04 RN2
+L Motherboard-rescue:R_Network04-Device RN2
 U 1 1 5C59B3EE
 P 14825 1300
@@
 $EndComp
 $Comp
-L power:+5V #PWR062
+L Motherboard-rescue:+5V-power #PWR062
 U 1 1 5C59B44A
 P 14625 1100
@@
 	9850 4450 9850 4525
 $Comp
-L power:GND #PWR056
+L Motherboard-rescue:GND-power #PWR056
 U 1 1 5C70F34B
 P 9850 4525
@@
 $EndComp
 $Comp
-L power:GND #PWR057
+L Motherboard-rescue:GND-power #PWR057
 U 1 1 5C70F43F
 P 9875 6425
@@
 ~XMEMW
 $Comp
-L 74xx:74LS27 U40
+L Motherboard-rescue:74LS27-74xx U40
 U 1 1 5C742C51
 P 9730 9755
@@
 $EndComp
 $Comp
-L 74xx:74LS27 U40
+L Motherboard-rescue:74LS27-74xx U40
 U 2 1 5C742DA7
 P 9830 8930
@@
 	9730 9455 9730 9230
 $Comp
-L 74xx:74LS04 U41
+L Motherboard-rescue:74LS04-74xx U41
 U 1 1 5C74FFCA
 P 10305 9705
@@
 ~XIOR
 $Comp
-L Memory_Flash:SST39SF010 U48
+L Motherboard-rescue:SST39SF010-Memory_Flash U48
 U 1 1 5C83E2EF
 P 13750 5300
@@
 	13150 5600 12950 5600
 $Comp
-L power:GND #PWR058
+L Motherboard-rescue:GND-power #PWR058
 U 1 1 5C9964D6
 P 13150 5700
@@
 $EndComp
 $Comp
-L power:GND #PWR059
+L Motherboard-rescue:GND-power #PWR059
 U 1 1 5C9965D0
 P 13150 6100
@@
 $EndComp
 $Comp
-L power:GND #PWR061
+L Motherboard-rescue:GND-power #PWR061
 U 1 1 5C996D4B
 P 13750 6500
@@
 $EndComp
 $Comp
-L power:+5V #PWR060
+L Motherboard-rescue:+5V-power #PWR060
 U 1 1 5C996E70
 P 13750 4000
@@
 ROMADDR
 $Comp
-L power:+5V #PWR092
+L Motherboard-rescue:+5V-power #PWR092
 U 1 1 5D019148
 P 13775 1350
@@
 $EndComp
 $Comp
-L power:GND #PWR093
+L Motherboard-rescue:GND-power #PWR093
 U 1 1 5D0191B5
 P 13775 2550
@@
 $EndComp
 $Comp
-L power:+5V #PWR090
+L Motherboard-rescue:+5V-power #PWR090
 U 1 1 5D0193CB
 P 10350 1200
@@
 $EndComp
 $Comp
-L power:GND #PWR091
+L Motherboard-rescue:GND-power #PWR091
 U 1 1 5D01945A
 P 10350 2800
@@
 $EndComp
 $Comp
-L RAM:AS6C8008 U42
+L Motherboard-rescue:AS6C8008-RAM U42
 U 1 1 5CA57105
 P 5155 9710
@@
 	5790 10560 5755 10560
 $Comp
-L power:GND #PWR086
+L Motherboard-rescue:GND-power #PWR086
 U 1 1 5CAD2034
 P 5790 10610
@@
 	5790 10610 5790 10560
 $Comp
-L power:+5V #PWR087
+L Motherboard-rescue:+5V-power #PWR087
 U 1 1 5CAD228F
 P 5800 10360
@@
 XA[0...19]
 $Comp
-L 74xx:74LS245 U47
+L Motherboard-rescue:74LS245-74xx U47
 U 1 1 5CA70F64
 P 6775 8960
@@
 	5755 9460 6275 9460
 $Comp
-L power:+5V #PWR089
+L Motherboard-rescue:+5V-power #PWR089
 U 1 1 5CC1818D
 P 6775 9760
@@
 $EndComp
 $Comp
-L power:GND #PWR088
+L Motherboard-rescue:GND-power #PWR088
 U 1 1 5CC1844E
 P 6775 8160
@@
 ~XMEMR
 $Comp
-L power:+5V #PWR085
+L Motherboard-rescue:+5V-power #PWR085
 U 1 1 5CDBABE0
 P 5755 9910
@@
 	9830 8100 9830 8630
 $Comp
-L 74xx:74LS32 U52
+L Motherboard-rescue:74LS32-74xx U52
 U 1 1 5CEAACFF
 P 7490 7420
@@
 	7490 7720 7490 7725
 $Comp
-L 74xx:7400 U50
+L Motherboard-rescue:7400-74xx U50
 U 1 1 5D040E8B
 P 7390 8025
