File: Motherboard/IO_SigDecoder.sch (KiCad schematic (older format))
At the start: 12 parts, among them SW5 SW_DIP_x01, U30 74LS04, U34 74LS04, U36 74LS00, U4 CD40147, U51 ATF750LVC, U57 DS1100Z-100+ (TTLDL-20)

Commit message: LARGE sync
Parts:
- removed U4 (x2): CD40147, Housings_DIP:DIP-16_W7.62mm_Socket, symbol Motherboard-rescue:CD40147-CD40147
- removed U57 (x2): DS1100Z-100+ (TTLDL-20), Housings_SOIC:SOIC-8_3.9x4.9mm_Pitch1.27mm, symbol Motherboard-rescue:DS1100Z-100+-DS1100Z-100+
- R9: footprint (none) -> Resistors_THT:R_Axial_DIN0204_L3.6mm_D1.6mm_P2.54mm_Vertical
Other:
- note removed: "U44 in techref"
Changed lines of the file:
@@
 EESchema Schematic File Version 4
 LIBS:Motherboard-cache
-EELAYER 26 0
+EELAYER 29 0
 EELAYER END
 $Descr A3 16535 11693
@@
 ~CS7
 $Comp
-L Motherboard-rescue:DS1100Z-100+-DS1100Z-100+ U57
-U 1 1 5C9BD2D6
-P 5650 1750
-F 0 "U57" H 5650 2265 50  0000 C CNN
-F 1 "DS1100Z-100+ (TTLDL-20)" H 5650 2174 50  0000 C CNN
-F 2 "Housings_SOIC:SOIC-8_3.9x4.9mm_Pitch1.27mm" H 5650 1750 50  0001 C CNN
-F 3 "DOCUMENTATION" H 5650 1750 50  0001 C CNN
-	1    5650 1750
-	1    0    0    -1
-$EndComp
-$Comp
-L Motherboard-rescue:CD40147-CD40147 U4
-U 1 1 5CA70B41
-P 5975 3500
-AR Path="/5CA70B41" Ref="U4"  Part="1"
-AR Path="/5C32B2C3/5C3CEA0C/5CA70B41" Ref="U4"  Part="1"
-F 0 "U4" H 5975 4115 50  0000 C CNN
-F 1 "CD40147" H 5975 4024 50  0000 C CNN
-F 2 "Housings_DIP:DIP-16_W7.62mm_Socket" H 5975 3500 50  0001 C CNN
-F 3 "DOCUMENTATION" H 5975 3500 50  0001 C CNN
-	1    5975 3500
-	1    0    0    -1
-$EndComp
-Text Notes 5775 3000 2    50   ~ 0
-U44 in techref
-$Comp
 L power:+5V #PWR0137
 U 1 1 5CFED197
@@
 F 0 "R9" H 2409 2121 50  0000 L CNN
 F 1 "1k" H 2409 2030 50  0000 L CNN
-F 2 "" H 2350 2075 50  0001 C CNN
+F 2 "Resistors_THT:R_Axial_DIN0204_L3.6mm_D1.6mm_P2.54mm_Vertical" H 2350 2075 50  0001 C CNN
 F 3 "~" H 2350 2075 50  0001 C CNN
 	1    2350 2075
@@
 Wire Wire Line
 	2675 2575 2850 2575
-$Comp
-L power:GND #PWR0208
-U 1 1 5CFF0678
-P 2850 2675
-F 0 "#PWR0208" H 2850 2425 50  0001 C CNN
-F 1 "GND" H 2855 2502 50  0000 C CNN
-F 2 "" H 2850 2675 50  0001 C CNN
-F 3 "" H 2850 2675 50  0001 C CNN
-	1    2850 2675
-L Motherboard-rescue:DS1100Z-100+-DS1100Z-100+ U57
-U 1 1 5C9BD2D6
-P 8325 2750
-F 0 "U57" H 8325 3265 50  0000 C CNN
-F 1 "DS1100Z-100+ (TTLDL-20)" H 8325 3174 50  0000 C CNN
-F 2 "Housings_SOIC:SOIC-8_3.9x4.9mm_Pitch1.27mm" H 8325 2750 50  0001 C CNN
-F 3 "DOCUMENTATION" H 8325 2750 50  0001 C CNN
-	1    8325 2750
-	1    0    0    -1
-$EndComp
-$Comp
-L power:+5V #PWR0209
-U 1 1 5CFF0744
-P 3850 1575
-F 0 "#PWR0209" H 3850 1425 50  0001 C CNN
-F 1 "+5V" H 3865 1748 50  0000 C CNN
-F 2 "" H 3850 1575 50  0001 C CNN
-F 3 "" H 3850 1575 50  0001 C CNN
-	1    3850 1575
-L Motherboard-rescue:CD40147-CD40147 U4
-U 1 1 5CA70B41
-P 6775 6400
-F 0 "U4" H 6775 7015 50  0000 C CNN
-F 1 "CD40147" H 6775 6924 50  0000 C CNN
-F 2 "Housings_DIP:DIP-16_W7.62mm_Socket" H 6775 6400 50  0001 C CNN
-F 3 "DOCUMENTATION" H 6775 6400 50  0001 C CNN
-	1    6775 6400
-	1    0    0    -1
-$EndComp
 Wire Wire Line
 	3850 2175 4075 2175

Commit message: A LOT of work
Connections:
- net +5V: now also U51.24 (VCC)
- net GND: now also U51.12 (GND)
- net IOCHCK renamed IOCHCK_I
- net IOCHCK_I: no longer U51.23 (I/O)
- new net IOCHCK_O: U51.23 (I/O)
Changed lines of the file:
@@
 EESchema Schematic File Version 4
 LIBS:Motherboard-cache
-EELAYER 29 0
+EELAYER 30 0
 EELAYER END
 $Descr A3 16535 11693
@@
 ~ENABLEIOCK'
 Text HLabel 2275 1975 0    50   Input ~ 0
-IOCHCK
+IOCHCK_I
 $Comp
 L 74xx:74LS00 U36
@@
 $EndComp
 Text HLabel 3850 1675 2    50   Output ~ 0
-IOCHCK
+IOCHCK_O
 Text HLabel 2850 2075 0    50   Input ~ 0
 ~PCK
@@
 Wire Bus Line
 	1400 675  1400 1225
+$Comp
+L power:GND #PWR?
+U 1 1 5EB4770B
+P 2850 2675
+F 0 "#PWR?" H 2850 2425 50  0001 C CNN
+F 1 "GND" H 2855 2502 50  0000 C CNN
+F 2 "" H 2850 2675 50  0001 C CNN
+F 3 "" H 2850 2675 50  0001 C CNN
+	1    2850 2675
+	1    0    0    -1
+$EndComp
+$Comp
+L power:+5V #PWR?
+U 1 1 5EB47B98
+P 3850 1575
+F 0 "#PWR?" H 3850 1425 50  0001 C CNN
+F 1 "+5V" H 3865 1748 50  0000 C CNN
+F 2 "" H 3850 1575 50  0001 C CNN
+F 3 "" H 3850 1575 50  0001 C CNN
+	1    3850 1575
+	1    0    0    -1
+$EndComp
 $EndSCHEMATC

Commit message: Large Sync
Parts:
- R10, R11: symbol Device:R -> Motherboard-rescue:R-Device
- R9: symbol Device:R_Small -> Motherboard-rescue:R_Small-Device
- SW5: symbol Switch:SW_DIP_x01 -> Motherboard-rescue:SW_DIP_x01-Switch
- U30, U34: symbol 74xx:74LS04 -> Motherboard-rescue:74LS04-74xx
- U36: symbol 74xx:74LS00 -> Motherboard-rescue:74LS00-74xx
Changed lines of the file:
@@
 CLK33
 $Comp
-L 74xx:74LS04 U34
+L Motherboard-rescue:74LS04-74xx U34
 U 1 1 5C3CEA6F
 P 2675 4150
@@
 	2175 4150 2375 4150
 $Comp
-L 74xx:74LS04 U30
+L Motherboard-rescue:74LS04-74xx U30
 U 2 1 5C3CEB4A
 P 2675 3750
@@
 	2175 3750 2375 3750
 $Comp
-L Device:R R10
+L Motherboard-rescue:R-Device R10
 U 1 1 5C3CEC19
 P 3175 3750
@@
 IOCHCK_I
 $Comp
-L 74xx:74LS00 U36
+L Motherboard-rescue:74LS00-74xx U36
 U 2 1 5C3CF7E9
 P 3825 3950
@@
 XA15
 $Comp
-L Device:R R11
+L Motherboard-rescue:R-Device R11
 U 1 1 5C9B19FC
 P 2675 2725
@@
 	2675 2575 2575 2575
 $Comp
-L Switch:SW_DIP_x01 SW5
+L Motherboard-rescue:SW_DIP_x01-Switch SW5
 U 1 1 5C9B21CC
 P 2275 2575
@@
 $EndComp
 $Comp
-L power:GND #PWR063
+L Motherboard-rescue:GND-power #PWR063
 U 1 1 5C9B2325
 P 1975 2575
@@
 $EndComp
 $Comp
-L power:+5V #PWR065
+L Motherboard-rescue:+5V-power #PWR065
 U 1 1 5C9B2372
 P 2675 2875
@@
 ~CS7
 $Comp
-L power:+5V #PWR0137
+L Motherboard-rescue:+5V-power #PWR0137
 U 1 1 5CFED197
 P 2350 2175
@@
 $EndComp
 $Comp
-L Device:R_Small R9
+L Motherboard-rescue:R_Small-Device R9
 U 1 1 5CFED308
 P 2350 2075
@@
 Wire Wire Line
 	1500 1225 1700 1225
-Wire Bus Line
-	1400 675  1400 1225
-$Comp
-L power:GND #PWR?
+$Comp
+L Motherboard-rescue:GND-power #PWR099
 U 1 1 5EB4770B
 P 2850 2675
-F 0 "#PWR?" H 2850 2425 50  0001 C CNN
+F 0 "#PWR099" H 2850 2425 50  0001 C CNN
 F 1 "GND" H 2855 2502 50  0000 C CNN
 F 2 "" H 2850 2675 50  0001 C CNN
@@
 $EndComp
 $Comp
-L power:+5V #PWR?
+L Motherboard-rescue:+5V-power #PWR0100
 U 1 1 5EB47B98
 P 3850 1575
-F 0 "#PWR?" H 3850 1425 50  0001 C CNN
+F 0 "#PWR0100" H 3850 1425 50  0001 C CNN
 F 1 "+5V" H 3865 1748 50  0000 C CNN
 F 2 "" H 3850 1575 50  0001 C CNN
@@
 	1    0    0    -1
 $EndComp
+Wire Bus Line
+	1400 675  1400 1225
 $EndSCHEMATC
