File: FDC/FDC.sch (KiCad schematic (older format))
At the start: 38 parts, among them J1 Bus_ISA_8bit, J2 Floppy IDC, SW1 DSEL, U1 74LS08, U13 74LS08, U16 74LS175, U17 MC3487N, U19 74LS74, U2 74LS32, U21 74LS161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

Commit message: Fixed missing +5V on FDC
Parts:
- U6: symbol fdc:uPD765BC -> FDC-rescue:uPD765BC-fdc
Connections:
- net +5V: now also U23.16 (VCC), U24.16 (VCC)
Changed lines of the file:
@@
 $EndComp
 $Comp
-L fdc:uPD765BC U6
+L FDC-rescue:uPD765BC-fdc U6
 U 1 1 5C3633C4
 P 5225 1925
@@
 	0    1    1    0
 $EndComp
+Text Label 6175 1525 2    50   ~ 0
+WPT
 Wire Bus Line
 	4375 1325 4375 2025
@@
 Wire Bus Line
 	3350 1275 3350 2225
-Text Label 6175 1525 2    50   ~ 0
-WPT
+$Comp
+L power:+5V #PWR?
+U 1 1 5C52E833
+P 12100 4225
+F 0 "#PWR?" H 12100 4075 50  0001 C CNN
+F 1 "+5V" V 12115 4353 50  0000 L CNN
+F 2 "" H 12100 4225 50  0001 C CNN
+F 3 "" H 12100 4225 50  0001 C CNN
+	1    12100 4225
+	0    1    1    0
+$EndComp
+$Comp
+L power:+5V #PWR?
+U 1 1 5C52E945
+P 13825 4450
+F 0 "#PWR?" H 13825 4300 50  0001 C CNN
+F 1 "+5V" V 13840 4578 50  0000 L CNN
+F 2 "" H 13825 4450 50  0001 C CNN
+F 3 "" H 13825 4450 50  0001 C CNN
+	1    13825 4450
+	0    1    1    0
+$EndComp
 $EndSCHEMATC

Commit message: Added missing HD/DD /REDWC option
Parts:
- added R7: 4k7, Resistors_THT:R_Axial_DIN0204_L3.6mm_D1.6mm_P2.54mm_Vertical, symbol Device:R
- SW1: footprint Housings_DIP:DIP-4_W7.62mm -> Housings_DIP:DIP-8_W7.62mm; symbol Switch:SW_DIP_x02 -> Switch:SW_DIP_x04
Connections:
- net +5V: now also U6.40 (VCC), R7.2
- net 1MHZ: now also SW1.6; no longer SW1.4
- net 2MHZ: now also SW1.5; no longer SW1.3
- net GND: now also SW1.2, U6.20 (GND)
- net INDEX: now also U6.17 (INDEX)
- net LCT_DIR: now also U6.38 (LCT/DIR)
- net ~REDWC: now also SW1.7, R7.1
- new net: SW1.3, SW1.4, U6.21 (WCLK)
- now unconnected: SW1.1
- no-connect marks 8 -> 27
Changed lines of the file:
@@
 8MHZ
 $Comp
-L Switch:SW_DIP_x02 SW1
+L Switch:SW_DIP_x04 SW1
 U 1 1 5C6B5C02
-P 5875 3600
-F 0 "SW1" V 5829 3830 50  0000 L CNN
-F 1 "DSEL" V 5920 3830 50  0000 L CNN
-F 2 "Housings_DIP:DIP-4_W7.62mm" H 5875 3600 50  0001 C CNN
-F 3 "" H 5875 3600 50  0001 C CNN
-	1    5875 3600
+P 5975 3600
+F 0 "SW1" V 5929 3830 50  0000 L CNN
+F 1 "DSEL" V 6020 3830 50  0000 L CNN
+F 2 "Housings_DIP:DIP-8_W7.62mm" H 5975 3600 50  0001 C CNN
+F 3 "" H 5975 3600 50  0001 C CNN
+	1    5975 3600
 	0    1    1    0
 $EndComp
@@
 	5925 3300 5975 3300
 Connection ~ 5925 3300
-Wire Wire Line
-	5875 3900 5875 4125
 Wire Wire Line
 	5975 3900 5975 4125
@@
 Text Label 6175 1525 2    50   ~ 0
 WPT
+$Comp
+L power:+5V #PWR0113
+U 1 1 5C52E833
+P 12100 4225
+F 0 "#PWR0113" H 12100 4075 50  0001 C CNN
+F 1 "+5V" V 12115 4353 50  0000 L CNN
+F 2 "" H 12100 4225 50  0001 C CNN
+F 3 "" H 12100 4225 50  0001 C CNN
+	1    12100 4225
+	0    1    1    0
+$EndComp
+$Comp
+L power:+5V #PWR0114
+U 1 1 5C52E945
+P 13825 4450
+F 0 "#PWR0114" H 13825 4300 50  0001 C CNN
+F 1 "+5V" V 13840 4578 50  0000 L CNN
+F 2 "" H 13825 4450 50  0001 C CNN
+F 3 "" H 13825 4450 50  0001 C CNN
+	1    13825 4450
+	0    1    1    0
+$EndComp
+$Comp
+L power:GND #PWR0115
+U 1 1 5C5E09FE
+P 4525 2825
+F 0 "#PWR0115" H 4525 2575 50  0001 C CNN
+F 1 "GND" H 4530 2652 50  0000 C CNN
+F 2 "" H 4525 2825 50  0001 C CNN
+F 3 "" H 4525 2825 50  0001 C CNN
+	1    4525 2825
+	1    0    0    -1
+$EndComp
+$Comp
+L power:+5V #PWR0116
+U 1 1 5C5E0D6B
+P 5925 925
+F 0 "#PWR0116" H 5925 775 50  0001 C CNN
+F 1 "+5V" H 5940 1098 50  0000 C CNN
+F 2 "" H 5925 925 50  0001 C CNN
+F 3 "" H 5925 925 50  0001 C CNN
+	1    5925 925
+	1    0    0    -1
+$EndComp
+Wire Wire Line
+	4525 2525 4225 2525
+Text Label 4225 2525 0    50   ~ 0
+INDEX
+NoConn ~ 5925 1425
+Wire Wire Line
+	5925 1125 6250 1125
+Text Label 6250 1125 2    50   ~ 0
+LCT_DIR
+NoConn ~ 5925 1325
+NoConn ~ 11525 1575
+NoConn ~ 11525 1775
+NoConn ~ 11525 1975
+NoConn ~ 11525 2175
+NoConn ~ 11600 4525
+NoConn ~ 12600 4525
+NoConn ~ 12600 4625
+NoConn ~ 12600 4825
+NoConn ~ 12600 5025
+NoConn ~ 12600 5225
+NoConn ~ 13825 7425
+NoConn ~ 13825 7525
+NoConn ~ 13825 7625
+NoConn ~ 13825 7725
+NoConn ~ 14825 7925
+$Comp
+L power:GND #PWR0117
+U 1 1 5C8B7957
+P 6075 3300
+F 0 "#PWR0117" H 6075 3050 50  0001 C CNN
+F 1 "GND" H 6080 3127 50  0000 C CNN
+F 2 "" H 6075 3300 50  0001 C CNN
+F 3 "" H 6075 3300 50  0001 C CNN
+	1    6075 3300
+	-1   0    0    1
+$EndComp
+Wire Wire Line
+	6075 3900 6075 4300
+Wire Wire Line
+	6075 4300 6375 4300
+$Comp
+L Device:R R7
+U 1 1 5C8DDDD9
+P 6075 4450
+F 0 "R7" V 5868 4450 50  0000 C CNN
+F 1 "4k7" V 5959 4450 50  0000 C CNN
+F 2 "Resistors_THT:R_Axial_DIN0204_L3.6mm_D1.6mm_P2.54mm_Vertical" V 6005 4450 50  0001 C CNN
+F 3 "~" H 6075 4450 50  0001 C CNN
+	1    6075 4450
+	1    0    0    -1
+$EndComp
+$Comp
+L power:+5V #PWR0118
+U 1 1 5C8DDF3F
+P 6075 4600
+F 0 "#PWR0118" H 6075 4450 50  0001 C CNN
+F 1 "+5V" H 6090 4773 50  0000 C CNN
+F 2 "" H 6075 4600 50  0001 C CNN
+F 3 "" H 6075 4600 50  0001 C CNN
+	1    6075 4600
+	0    -1   -1   0
+$EndComp
+Text Label 6375 4300 2    50   ~ 0
+~REDWC
+NoConn ~ 6175 3300
+NoConn ~ 6175 3900
+Connection ~ 6075 4300
+Wire Wire Line
+	5875 3900 5875 4125
 Wire Bus Line
 	4375 1325 4375 2025
@@
 Wire Bus Line
 	3350 1275 3350 2225
-$Comp
-L power:+5V #PWR?
-U 1 1 5C52E833
-P 12100 4225
-F 0 "#PWR?" H 12100 4075 50  0001 C CNN
-F 1 "+5V" V 12115 4353 50  0000 L CNN
-F 2 "" H 12100 4225 50  0001 C CNN
-F 3 "" H 12100 4225 50  0001 C CNN
-	1    12100 4225
-	0    1    1    0
-$EndComp
-$Comp
-L power:+5V #PWR?
-U 1 1 5C52E945
-P 13825 4450
-F 0 "#PWR?" H 13825 4300 50  0001 C CNN
-F 1 "+5V" V 13840 4578 50  0000 L CNN
-F 2 "" H 13825 4450 50  0001 C CNN
-F 3 "" H 13825 4450 50  0001 C CNN
-	1    13825 4450
-	0    1    1    0
-$EndComp
 $EndSCHEMATC

Commit message: Large sync
Parts:
- added SW2: DSEL, Housings_DIP:DIP-8_W7.62mm, symbol Switch:SW_DIP_x04
Connections:
- new net PLL/1MHZ: SW2.4
- new net PLL/2MHZ: SW2.3
- new net PLL/PLLCLK: SW2.5, SW2.6
- no-connect marks 27 -> 31
Changed lines of the file:
@@
 F3 "MFM" I L 6525 2400 50
 F4 "DIN" I L 6525 2650 50
-F5 "DOUT" O R 7225 2650 50
+F5 "DOUT" O R 7225 2675 50
 F6 "DATA_WINDOW" O R 7225 2775 50
+F7 "2MHZ" O R 7225 2350 50
+F8 "1MHZ" O R 7225 2450 50
+F9 "PLLCLK" I R 7225 2600 50
 $EndSheet
 Wire Wire Line
@@
 	5925 2525 6525 2525
 Wire Wire Line
-	7225 2650 7500 2650
-Wire Wire Line
-	7500 2650 7500 3200
+	7225 2675 7500 2675
 Wire Wire Line
 	7500 3200 6175 3200
@@
 Wire Wire Line
 	5875 3900 5875 4125
+Wire Wire Line
+	7225 2450 7375 2450
+Wire Wire Line
+	7225 2350 7375 2350
+Wire Wire Line
+	7500 2675 7500 3200
+Wire Wire Line
+	7225 2600 7975 2600
+$Comp
+L Switch:SW_DIP_x04 SW2
+U 1 1 5C6D1D58
+P 7675 2350
+F 0 "SW2" V 7629 2580 50  0000 L CNN
+F 1 "DSEL" V 7720 2580 50  0000 L CNN
+F 2 "Housings_DIP:DIP-8_W7.62mm" H 7675 2350 50  0001 C CNN
+F 3 "" H 7675 2350 50  0001 C CNN
+	1    7675 2350
+	1    0    0    -1
+$EndComp
+Wire Wire Line
+	7975 2350 7975 2450
+Wire Wire Line
+	7975 2450 7975 2600
+Connection ~ 7975 2450
+NoConn ~ 7375 2250
+NoConn ~ 7375 2150
+NoConn ~ 7975 2150
+NoConn ~ 7975 2250
 Wire Bus Line
 	4375 1325 4375 2025
