File: FDC/PLL.sch (KiCad schematic (older format))
At the start: 22 parts, among them Q1 2N2219, Q2 2N3905, U10 74LS161, U11 74LS10, U12 74LS74, U14 74LS157, U15 74LS74, U18 74LS74, U20 74LS629, U9 74LS161

Commit message: Large sync
Parts:
- R1: value R_Small -> 2k2
- R2: value R_Small -> 1k
- R5: value R -> 1k
Connections:
- net 1MHZ: no longer U12.11 (C), U14.6 (I1b)
- net 2MHZ: now reaches U10.13 (Q1)
- new net PLLCLK: U12.11 (C), U14.6 (I1b)
- no-connect marks 21 -> 20
Changed lines of the file:
@@
 NoConn ~ 2250 3200
 Wire Wire Line
-	2250 3400 2800 3400
-Wire Wire Line
-	2800 3400 2800 3000
+	2250 3400 2500 3400
 Wire Wire Line
 	2800 3000 3250 3000
 Wire Wire Line
-	2800 3400 2800 4425
-Wire Wire Line
 	2800 4425 3050 4425
-Connection ~ 2800 3400
 Wire Wire Line
 	2250 3500 2700 3500
@@
 Wire Wire Line
 	2700 4325 3050 4325
-Text Label 2550 3400 0    50   ~ 0
+Text Label 2250 3400 0    50   ~ 0
 1MHZ
-Text Label 2450 3500 0    50   ~ 0
+Text Label 2375 3500 0    50   ~ 0
 500KHZ
 $Comp
@@
 P 4900 1825
 F 0 "R5" H 4970 1871 50  0000 L CNN
-F 1 "R" H 4970 1780 50  0000 L CNN
+F 1 "1k" H 4970 1780 50  0000 L CNN
 F 2 "Resistors_THT:R_Axial_DIN0204_L3.6mm_D1.6mm_P1.90mm_Vertical" V 4830 1825 50  0001 C CNN
 F 3 "~" H 4900 1825 50  0001 C CNN
@@
 P 4175 3100
 F 0 "R1" V 3979 3100 50  0000 C CNN
-F 1 "R_Small" V 4070 3100 50  0000 C CNN
+F 1 "2k2" V 4070 3100 50  0000 C CNN
 F 2 "Resistors_THT:R_Axial_DIN0204_L3.6mm_D1.6mm_P1.90mm_Vertical" H 4175 3100 50  0001 C CNN
 F 3 "~" H 4175 3100 50  0001 C CNN
@@
 P 4325 3250
 F 0 "R2" H 4384 3296 50  0000 L CNN
-F 1 "R_Small" H 4384 3205 50  0000 L CNN
+F 1 "1k" H 4384 3205 50  0000 L CNN
 F 2 "Resistors_THT:R_Axial_DIN0204_L3.6mm_D1.6mm_P1.90mm_Vertical" H 4325 3250 50  0001 C CNN
 F 3 "~" H 4325 3250 50  0001 C CNN
@@
 	9450 1700 9450 1800
 Connection ~ 8700 2800
-NoConn ~ 2250 3300
 $Comp
 L Device:R_POT_TRIM RV7
@@
 $EndComp
 Connection ~ 5275 1450
+Text HLabel 2375 2750 1    50   Output ~ 0
+2MHZ
+Text HLabel 2500 2750 1    50   Output ~ 0
+1MHZ
+Text HLabel 2800 2750 1    50   Input ~ 0
+PLLCLK
+Wire Wire Line
+	2800 2750 2800 3000
+Connection ~ 2800 3000
+Wire Wire Line
+	2250 3300 2375 3300
+Wire Wire Line
+	2375 3300 2375 2750
+Wire Wire Line
+	2500 2750 2500 3400
+Wire Wire Line
+	2800 3000 2800 4425
 $EndSCHEMATC
